File: HARDWARE/KICAD/MCU.kicad_sch (KiCad schematic)
At the start: 49 parts, among them Q1 2N7002K, Q2 2N7002K, U4 STM32F411RET6, Y1 12MHz 18pF, Y2 32.768kHz 12.5pF

Commit message: Refactoring.
Other:
- company: (none) -> Mechatronix Lab
- title: (none) -> EMBARCADOS - CURSO PCB
Changed lines of the file:
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@@
 	(generator_version "8.0")
 	(paper "A4")
+	(title_block
+		(title "EMBARCADOS - CURSO PCB")
+		(date "2024-11-11")
+		(rev "00")
+		(company "Mechatronix Lab")
+		(comment 1 "Eng. André A. M. Araújo")
+	)
 	(junction
 		(at 53.34 43.18)

Commit message: Added ANALOG and INTERFACE sheets.
Parts:
- removed R19: 1K 1%, EMBARCADOS - CURSO PCB:R_0603_1608Metric, symbol EMBARCADOS - CURSO PCB:RES 0603 1K 1% VISHAY CRCW06031K00FK
- removed TP2: PC0, symbol EMBARCADOS - CURSO PCB:AUX TEST POINT
- removed TP3: PC1, symbol EMBARCADOS - CURSO PCB:AUX TEST POINT
- removed TP4: PC2, symbol EMBARCADOS - CURSO PCB:AUX TEST POINT
- removed TP5: PC3, symbol EMBARCADOS - CURSO PCB:AUX TEST POINT
- added R19: 51R 1%, EMBARCADOS - CURSO PCB:R_0603_1608Metric, symbol EMBARCADOS - CURSO PCB:RES 0603 51R 1% VISHAY CRCW060351R0FK
- C12, C13, C20: symbol EMBARCADOS - CURSO PCB:CAP 0805 10uH 16V AVX KGM21AR71C106K -> EMBARCADOS - CURSO PCB:CAP 0805 10uF 16V AVX KGM21AR71C106K
Connections:
- net MCU PC9: now also R19.1
- net PWM BUZZER: now also R19.2
- net MCU PC0 renamed PC0
- net MCU PC1 renamed PC1
- net MCU PC2 renamed PC2
- net MCU PC3 renamed PC3

Commit message: Refactoring.
Changed lines of the file:
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@@
 	(wire
 		(pts
-			(xy 73.66 55.88) (xy 73.66 68.58)
+			(xy 74.93 55.88) (xy 74.93 68.58)
 		)
 		(stroke
@@
 	(wire
 		(pts
-			(xy 168.91 39.37) (xy 168.91 60.96)
+			(xy 168.91 40.64) (xy 168.91 60.96)
 		)
 		(stroke
@@
 	(wire
 		(pts
-			(xy 120.65 91.44) (xy 120.65 44.45)
+			(xy 120.65 91.44) (xy 120.65 45.72)
 		)
 		(stroke
@@
 	(wire
 		(pts
-			(xy 125.73 53.34) (xy 125.73 60.96)
+			(xy 125.73 50.8) (xy 125.73 60.96)
 		)
 		(stroke
@@
 	(wire
 		(pts
-			(xy 115.57 39.37) (xy 115.57 109.22)
+			(xy 115.57 40.64) (xy 115.57 109.22)
 		)
 		(stroke
@@
 	(wire
 		(pts
-			(xy 73.66 68.58) (xy 128.27 68.58)
+			(xy 74.93 68.58) (xy 128.27 68.58)
 		)
 		(stroke
@@
 	(wire
 		(pts
-			(xy 73.66 55.88) (xy 53.34 55.88)
+			(xy 74.93 55.88) (xy 53.34 55.88)
 		)
 		(stroke
@@
 	(symbol
 		(lib_id "EMBARCADOS - CURSO PCB:+5V")
-		(at 120.65 44.45 0)
+		(at 120.65 45.72 0)
 		(unit 1)
 		(exclude_from_sim no)
@@
 		(dnp no)
 		(property "Reference" "#PWR034"
-			(at 120.65 48.26 0)
+			(at 120.65 49.53 0)
 			(effects
 				(font
@@
 		)
 		(property "Value" "+3.3VA"
-			(at 120.65 40.64 0)
+			(at 120.65 41.91 0)
 			(effects
 				(font
@@
 		)
 		(property "Footprint" ""
-			(at 120.65 44.45 0)
+			(at 120.65 45.72 0)
 			(effects
 				(font
@@
 		)
 		(property "Datasheet" ""
-			(at 120.65 44.45 0)
+			(at 120.65 45.72 0)
 			(effects
 				(font
@@
 		)
 		(property "Description" "Power symbol creates a global label with name \"+5V\""
-			(at 120.65 44.45 0)
+			(at 120.65 45.72 0)
 			(effects
 				(font
@@
 		)
 		(property "MPN" ""
-			(at 120.65 44.45 0)
+			(at 120.65 45.72 0)
 			(effects
 				(font
@@
 		)
 		(property "Manufacturer" ""
-			(at 120.65 44.45 0)
+			(at 120.65 45.72 0)
 			(effects
 				(font
@@
 		)
 		(property "3D Model" ""
-			(at 120.65 44.45 0)
+			(at 120.65 45.72 0)
 			(effects
 				(font
@@
 		)
 		(property "Notes" ""
-			(at 120.65 44.45 0)
+			(at 120.65 45.72 0)
 			(effects
 				(font
@@
 		)
 		(property "LCSC Part # " ""
-			(at 120.65 44.45 0)
+			(at 120.65 45.72 0)
 			(effects
 				(font
@@
 		)
 		(property "LCSC MPN " ""
-			(at 120.65 44.45 0)
+			(at 120.65 45.72 0)
 			(effects
 				(font
@@
 		)
 		(property "LCSC MANUFACTURER " ""
-			(at 120.65 44.45 0)
+			(at 120.65 45.72 0)
 			(effects
 				(font
@@
 	(symbol
 		(lib_id "EMBARCADOS - CURSO PCB:+5V")
-		(at 115.57 39.37 0)
+		(at 115.57 40.64 0)
 		(unit 1)
 		(exclude_from_sim no)
@@
 		(dnp no)
 		(property "Reference" "#PWR031"
-			(at 115.57 43.18 0)
+			(at 115.57 44.45 0)
 			(effects
 				(font
@@
 		)
 		(property "Value" "+3.3V"
-			(at 115.57 35.56 0)
+			(at 115.57 36.83 0)
 			(effects
 				(font
@@
 		)
 		(property "Footprint" ""
-			(at 115.57 39.37 0)
+			(at 115.57 40.64 0)
 			(effects
 				(font
@@
 		)
 		(property "Datasheet" ""
-			(at 115.57 39.37 0)
+			(at 115.57 40.64 0)
 			(effects
 				(font
@@
 		)
 		(property "Description" "Power symbol creates a global label with name \"+5V\""
-			(at 115.57 39.37 0)
+			(at 115.57 40.64 0)
 			(effects
 				(font
@@
 		)
 		(property "MPN" ""
-			(at 115.57 39.37 0)
+			(at 115.57 40.64 0)
 			(effects
 				(font
@@
 		)
 		(property "Manufacturer" ""
-			(at 115.57 39.37 0)
+			(at 115.57 40.64 0)
 			(effects
 				(font
@@
 		)
 		(property "3D Model" ""
-			(at 115.57 39.37 0)
+			(at 115.57 40.64 0)
 			(effects
 				(font
@@
 		)
 		(property "Notes" ""
-			(at 115.57 39.37 0)
+			(at 115.57 40.64 0)
 			(effects
 				(font
@@
 		)
 		(property "LCSC Part # " ""
-			(at 115.57 39.37 0)
+			(at 115.57 40.64 0)
 			(effects
 				(font
@@
 		)
 		(property "LCSC MPN " ""
-			(at 115.57 39.37 0)
+			(at 115.57 40.64 0)
 			(effects
 				(font
@@
 		)
 		(property "LCSC MANUFACTURER " ""
-			(at 115.57 39.37 0)
+			(at 115.57 40.64 0)
 			(effects
 				(font
@@
 	(symbol
 		(lib_id "EMBARCADOS - CURSO PCB:+5V")
-		(at 168.91 39.37 0)
+		(at 168.91 40.64 0)
 		(unit 1)
 		(exclude_from_sim no)
@@
 		(dnp no)
 		(property "Reference" "#PWR035"
-			(at 168.91 43.18 0)
+			(at 168.91 44.45 0)
 			(effects
 				(font
@@
 		)
 		(property "Value" "+3.3V"
-			(at 168.91 35.56 0)
+			(at 168.91 36.83 0)
 			(effects
 				(font
@@
 		)
 		(property "Footprint" ""
-			(at 168.91 39.37 0)
+			(at 168.91 40.64 0)
 			(effects
 				(font
@@
 		)
 		(property "Datasheet" ""
-			(at 168.91 39.37 0)
+			(at 168.91 40.64 0)
 			(effects
 				(font
@@
 		)
 		(property "Description" "Power symbol creates a global label with name \"+5V\""
-			(at 168.91 39.37 0)
+			(at 168.91 40.64 0)
 			(effects
 				(font
@@
 		)
 		(property "MPN" ""
-			(at 168.91 39.37 0)
+			(at 168.91 40.64 0)
 			(effects
 				(font
@@
 		)
 		(property "Manufacturer" ""
-			(at 168.91 39.37 0)
+			(at 168.91 40.64 0)
 			(effects
 				(font
@@
 		)
 		(property "3D Model" ""
-			(at 168.91 39.37 0)
+			(at 168.91 40.64 0)
 			(effects
 				(font
@@
 		)
 		(property "Notes" ""
-			(at 168.91 39.37 0)
+			(at 168.91 40.64 0)
 			(effects
 				(font
@@
 		)
 		(property "LCSC Part # " ""
-			(at 168.91 39.37 0)
+			(at 168.91 40.64 0)
 			(effects
 				(font
@@
 		)
 		(property "LCSC MPN " ""
-			(at 168.91 39.37 0)
+			(at 168.91 40.64 0)
 			(effects
 				(font
@@
 		)
 		(property "LCSC MANUFACTURER " ""
-			(at 168.91 39.37 0)
+			(at 168.91 40.64 0)
 			(effects
 				(font
@@
 	(symbol
 		(lib_id "EMBARCADOS - CURSO PCB:+5V")
-		(at 125.73 53.34 0)
+		(at 125.73 50.8 0)
 		(unit 1)
 		(exclude_from_sim no)
@@
 		(dnp no)
 		(property "Reference" "#PWR029"
-			(at 125.73 57.15 0)
+			(at 125.73 54.61 0)
 			(effects
 				(font
@@
 		)
 		(property "Value" "+3VBAT"
-			(at 125.73 45.72 0)
+			(at 125.73 46.99 0)
 			(effects
 				(font
@@
 		)
 		(property "Footprint" ""
-			(at 125.73 53.34 0)
+			(at 125.73 50.8 0)
 			(effects
 				(font
@@
 		)
 		(property "Datasheet" ""
-			(at 125.73 53.34 0)
+			(at 125.73 50.8 0)
 			(effects
 				(font
@@
 		)
 		(property "Description" "Power symbol creates a global label with name \"+5V\""
-			(at 125.73 53.34 0)
+			(at 125.73 50.8 0)
 			(effects
 				(font
@@
 		)
 		(property "MPN" ""
-			(at 125.73 53.34 0)
+			(at 125.73 50.8 0)
 			(effects
 				(font
@@
 		)
 		(property "Manufacturer" ""
-			(at 125.73 53.34 0)
+			(at 125.73 50.8 0)
 			(effects
 				(font
@@
 		)
 		(property "3D Model" ""
-			(at 125.73 53.34 0)
+			(at 125.73 50.8 0)
 			(effects
 				(font
@@
 		)
 		(property "Notes" ""
-			(at 125.73 53.34 0)
+			(at 125.73 50.8 0)
 			(effects
 				(font
@@
 		)
 		(property "LCSC Part # " ""
-			(at 125.73 53.34 0)
+			(at 125.73 50.8 0)
 			(effects
 				(font
@@
 		)
 		(property "LCSC MPN " ""
-			(at 125.73 53.34 0)
+			(at 125.73 50.8 0)
 			(effects
 				(font
@@
 		)
 		(property "LCSC MANUFACTURER " ""
-			(at 125.73 53.34 0)
+			(at 125.73 50.8 0)
 			(effects
 				(font

Commit message: Finished schematic.
Parts:
- added C44: 100nF 50V, EMBARCADOS - CURSO PCB:C_0603_1608Metric, symbol EMBARCADOS - CURSO PCB:CAP 0603 100nF 50V AVX KGM15BR71H104K
Connections:
- net GND: now also C44.1
- net NRST: now also C44.2

Commit message: Starting PCB layout.
Parts:
- TP1, TP10, TP11, TP6, TP7, TP8, TP9: footprint (none) -> EMBARCADOS - CURSO PCB:TestPoint_Keystone_5000-5004_Miniature
Changed lines of the file:
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@@
 			)
 		)
-		(property "Footprint" ""
+		(property "Footprint" "EMBARCADOS - CURSO PCB:TestPoint_Keystone_5000-5004_Miniature"
 			(at 113.03 58.42 0)
 			(effects
@@
 			)
 		)
-		(property "Footprint" ""
+		(property "Footprint" "EMBARCADOS - CURSO PCB:TestPoint_Keystone_5000-5004_Miniature"
 			(at 179.07 96.52 0)
 			(effects
@@
 			)
 		)
-		(property "Footprint" ""
+		(property "Footprint" "EMBARCADOS - CURSO PCB:TestPoint_Keystone_5000-5004_Miniature"
 			(at 179.07 91.44 0)
 			(effects
@@
 			)
 		)
-		(property "Footprint" ""
+		(property "Footprint" "EMBARCADOS - CURSO PCB:TestPoint_Keystone_5000-5004_Miniature"
 			(at 113.03 129.54 0)
 			(effects
@@
 			)
 		)
-		(property "Footprint" ""
+		(property "Footprint" "EMBARCADOS - CURSO PCB:TestPoint_Keystone_5000-5004_Miniature"
 			(at 179.07 93.98 0)
 			(effects
@@
 			)
 		)
-		(property "Footprint" ""
+		(property "Footprint" "EMBARCADOS - CURSO PCB:TestPoint_Keystone_5000-5004_Miniature"
 			(at 179.07 86.36 0)
 			(effects
@@
 			)
 		)
-		(property "Footprint" ""
+		(property "Footprint" "EMBARCADOS - CURSO PCB:TestPoint_Keystone_5000-5004_Miniature"
 			(at 179.07 83.82 0)
 			(effects

Commit message: Recorded Class 08.07 Part 5.
Parts:
- removed TP1: PC13, EMBARCADOS - CURSO PCB:TestPoint_Keystone_5000-5004_Miniature, symbol EMBARCADOS - CURSO PCB:AUX TEST POINT
- removed TP10: PC12, EMBARCADOS - CURSO PCB:TestPoint_Keystone_5000-5004_Miniature, symbol EMBARCADOS - CURSO PCB:AUX TEST POINT
- removed TP11: PC11, EMBARCADOS - CURSO PCB:TestPoint_Keystone_5000-5004_Miniature, symbol EMBARCADOS - CURSO PCB:AUX TEST POINT
- removed TP6: PB10, EMBARCADOS - CURSO PCB:TestPoint_Keystone_5000-5004_Miniature, symbol EMBARCADOS - CURSO PCB:AUX TEST POINT
- removed TP7: PB5, EMBARCADOS - CURSO PCB:TestPoint_Keystone_5000-5004_Miniature, symbol EMBARCADOS - CURSO PCB:AUX TEST POINT
- removed TP8: PB4, EMBARCADOS - CURSO PCB:TestPoint_Keystone_5000-5004_Miniature, symbol EMBARCADOS - CURSO PCB:AUX TEST POINT
- removed TP9: PD2, EMBARCADOS - CURSO PCB:TestPoint_Keystone_5000-5004_Miniature, symbol EMBARCADOS - CURSO PCB:AUX TEST POINT
- renumbered C17 to C16, C16 to C17, C11 to C18, C15 to C24, C18 to C26, C10 to C27, C44 to C28, C19 to C32, C14 to C33, C13 to C34, C9 to C40, C12 to C41, C21 to C42, C8 to C43, C20 to C44, C23 to C7, C22 to C8, FB2 to FB4, Q1 to Q3, R23 to R14, R21 to R17, R22 to R18, R24 to R19, R15 to R22, R14 to R23, R13 to R25, R20 to R26, R9 to R32, R19 to R33, R18 to R34, R17 to R35, R16 to R36, R10 to R37, R11 to R42, R12 to R45, U4 to U7, Y2 to Y1, Y1 to Y2
Connections:
- net MCU PB10: no longer names the net of U7.29 (PB10)
- net MCU PB4: no longer names the net of U7.56 (PB4)
- net MCU PB5: no longer names the net of U7.57 (PB5)
- net MCU PC11: no longer names the net of U7.52 (PC11)
- net MCU PC12: no longer names the net of U7.53 (PC12)
- net MCU PC13: no longer names the net of U7.2 (PC13)
- net MCU PD2: no longer names the net of U7.54 (PD2)
- no-connect marks 0 -> 7

Commit message: Finished PCB Layout.
Parts:
- renumbered R17 to R15, R18 to R16
Changed lines of the file:
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@@
 		(on_board yes)
 		(dnp no)
-		(property "Reference" "R17"
+		(property "Reference" "R15"
 			(at 199.39 48.26 90)
 			(effects
@@
 			(project ""
 				(path "/d5268f1b-b782-4609-86ee-ff462c2ec1ad/c29651ae-6018-447b-aeb5-0320701650ee"
-					(reference "R17")
+					(reference "R15")
 					(unit 1)
 				)
@@
 		(on_board yes)
 		(dnp no)
-		(property "Reference" "R18"
+		(property "Reference" "R16"
 			(at 201.93 48.26 90)
 			(effects
@@
 			(project "EMBARCADOS - CURSO PCB"
 				(path "/d5268f1b-b782-4609-86ee-ff462c2ec1ad/c29651ae-6018-447b-aeb5-0320701650ee"
-					(reference "R18")
+					(reference "R16")
 					(unit 1)
 				)
