File: HARDWARE/KICAD/MCU.kicad_sch (KiCad schematic)
At the start: 39 parts, among them Q2 2N7002K, Q3 2N7002K, U7 STM32F411RET6, Y1 32.768kHz 12.5pF, Y2 12MHz 18pF

Commit message: Finished overall project review for PCB fabrication at JLCPCB.
Parts:
- C16, C17, C26, C32: LCSC Part # C1634 -> (none); LCSC Part #  (none) -> C1634
- C18, C24, C27, C28, C33, C40, C42, C43, C7, C8: LCSC Part # C14663 -> (none); LCSC Part #  (none) -> C14663
- C34, C41, C44: LCSC Part # C15850 -> (none); LCSC Part #  (none) -> C15850
- Y2: LCSC Part # C6071564 -> (none)
Changed lines of the file:
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@@
 			)
 		)
-		(property "LCSC Part #" "C14663 "
-			(at 76.2 83.566 0)
+		(property "LCSC MPN " "CC0603KRX7R9BB104 "
+			(at 75.692 87.884 0)
 			(effects
 				(font
@@
 			)
 		)
-		(property "LCSC MPN " "CC0603KRX7R9BB104 "
-			(at 75.692 87.884 0)
+		(property "LCSC MANUFACTURER " "YAGEO "
+			(at 75.946 85.598 0)
 			(effects
 				(font
@@
 			)
 		)
-		(property "LCSC MANUFACTURER " "YAGEO "
-			(at 75.946 85.598 0)
+		(property "LCSC Part # " "C14663 "
+			(at 76.2 83.566 0)
 			(effects
 				(font
@@
 			)
 		)
-		(property "LCSC Part #" "C1634 "
-			(at 59.944 83.82 0)
+		(property "LCSC MPN " "CL10C100JB8NNNC "
+			(at 55.626 83.312 0)
 			(effects
 				(font
@@
 			)
 		)
-		(property "LCSC MPN " "CL10C100JB8NNNC "
-			(at 55.626 83.312 0)
+		(property "LCSC MANUFACTURER " "SAMSUNG "
+			(at 57.912 83.566 0)
 			(effects
 				(font
@@
 			)
 		)
-		(property "LCSC MANUFACTURER " "SAMSUNG "
-			(at 57.912 83.566 0)
+		(property "LCSC Part # " "C1634 "
+			(at 59.944 83.82 0)
 			(effects
 				(font
@@
 			)
 		)
-		(property "LCSC Part #" "C14663 "
-			(at 43.18 162.306 0)
+		(property "LCSC MPN " "CC0603KRX7R9BB104 "
+			(at 42.672 166.624 0)
 			(effects
 				(font
@@
 			)
 		)
-		(property "LCSC MPN " "CC0603KRX7R9BB104 "
-			(at 42.672 166.624 0)
+		(property "LCSC MANUFACTURER " "YAGEO "
+			(at 42.926 164.338 0)
 			(effects
 				(font
@@
 			)
 		)
-		(property "LCSC MANUFACTURER " "YAGEO "
-			(at 42.926 164.338 0)
+		(property "LCSC Part # " "C14663 "
+			(at 43.18 162.306 0)
 			(effects
 				(font
@@
 			)
 		)
-		(property "LCSC Part #" "C6071564 "
-			(at 71.374 77.47 0)
-			(effects
-				(font
-					(size 1.27 1.27)
-				)
-				(hide yes)
-			)
-		)
 		(property "LCSC MPN " "3225 12M 18PF 20PPM "
 			(at 71.374 77.47 0)
@@
 			)
 		)
-		(property "LCSC Part #" "C14663 "
-			(at 219.456 26.67 0)
+		(property "LCSC MPN " "CC0603KRX7R9BB104 "
+			(at 223.774 26.162 0)
 			(effects
 				(font
@@
 			)
 		)
-		(property "LCSC MPN " "CC0603KRX7R9BB104 "
-			(at 223.774 26.162 0)
+		(property "LCSC MANUFACTURER " "YAGEO "
+			(at 221.488 26.416 0)
 			(effects
 				(font
@@
 			)
 		)
-		(property "LCSC MANUFACTURER " "YAGEO "
-			(at 221.488 26.416 0)
+		(property "LCSC Part # " "C14663 "
+			(at 219.456 26.67 0)
 			(effects
 				(font
@@
 			)
 		)
-		(property "LCSC Part #" "C15850 "
-			(at 146.05 193.294 0)
+		(property "LCSC MPN " "CL21A106KAYNNNE "
+			(at 146.558 188.976 0)
 			(effects
 				(font
@@
 			)
 		)
-		(property "LCSC MPN " "CL21A106KAYNNNE "
-			(at 146.558 188.976 0)
+		(property "LCSC MANUFACTURER " "SAMSUNG "
+			(at 146.304 191.262 0)
 			(effects
 				(font
@@
 			)
 		)
-		(property "LCSC MANUFACTURER " "SAMSUNG "
-			(at 146.304 191.262 0)
+		(property "LCSC Part # " "C15850 "
+			(at 146.05 193.294 0)
 			(effects
 				(font
@@
 			)
 		)
-		(property "LCSC Part #" "C14663 "
-			(at 104.14 162.306 0)
+		(property "LCSC MPN " "CC0603KRX7R9BB104 "
+			(at 103.632 166.624 0)
 			(effects
 				(font
@@
 			)
 		)
-		(property "LCSC MPN " "CC0603KRX7R9BB104 "
-			(at 103.632 166.624 0)
+		(property "LCSC MANUFACTURER " "YAGEO "
+			(at 103.886 164.338 0)
 			(effects
 				(font
@@
 			)
 		)
-		(property "LCSC MANUFACTURER " "YAGEO "
-			(at 103.886 164.338 0)
+		(property "LCSC Part # " "C14663 "
+			(at 104.14 162.306 0)
 			(effects
 				(font
@@
 			)
 		)
-		(property "LCSC Part #" "C14663 "
-			(at 209.804 26.67 0)
+		(property "LCSC MPN " "CC0603KRX7R9BB104 "
+			(at 205.486 26.162 0)
 			(effects
 				(font
@@
 			)
 		)
-		(property "LCSC MPN " "CC0603KRX7R9BB104 "
-			(at 205.486 26.162 0)
+		(property "LCSC MANUFACTURER " "YAGEO "
+			(at 207.772 26.416 0)
 			(effects
 				(font
@@
 			)
 		)
-		(property "LCSC MANUFACTURER " "YAGEO "
-			(at 207.772 26.416 0)
+		(property "LCSC Part # " "C14663 "
+			(at 209.804 26.67 0)
 			(effects
 				(font
@@
 			)
 		)
-		(property "LCSC Part #" "C14663 "
-			(at 120.65 162.306 0)
+		(property "LCSC MPN " "CC0603KRX7R9BB104 "
+			(at 120.142 166.624 0)
 			(effects
 				(font
@@
 			)
 		)
-		(property "LCSC MPN " "CC0603KRX7R9BB104 "
-			(at 120.142 166.624 0)
+		(property "LCSC MANUFACTURER " "YAGEO "
+			(at 120.396 164.338 0)
 			(effects
 				(font
@@
 			)
 		)
-		(property "LCSC MANUFACTURER " "YAGEO "
-			(at 120.396 164.338 0)
+		(property "LCSC Part # " "C14663 "
+			(at 120.65 162.306 0)
 			(effects
 				(font
@@
 			)
 		)
-		(property "LCSC Part #" "C1634 "
-			(at 59.944 55.88 0)
+		(property "LCSC MPN " "CL10C100JB8NNNC "
+			(at 55.626 55.372 0)
 			(effects
 				(font
@@
 			)
 		)
-		(property "LCSC MPN " "CL10C100JB8NNNC "
-			(at 55.626 55.372 0)
+		(property "LCSC MANUFACTURER " "SAMSUNG "
+			(at 57.912 55.626 0)
 			(effects
 				(font
@@
 			)
 		)
-		(property "LCSC MANUFACTURER " "SAMSUNG "
-			(at 57.912 55.626 0)
+		(property "LCSC Part # " "C1634 "
+			(at 59.944 55.88 0)
 			(effects
 				(font
@@
 			)
 		)
-		(property "LCSC Part #" "C14663 "
-			(at 60.96 162.306 0)
+		(property "LCSC MPN " "CC0603KRX7R9BB104 "
+			(at 60.452 166.624 0)
 			(effects
 				(font
@@
 			)
 		)
-		(property "LCSC MPN " "CC0603KRX7R9BB104 "
-			(at 60.452 166.624 0)
+		(property "LCSC MANUFACTURER " "YAGEO "
+			(at 60.706 164.338 0)
 			(effects
 				(font
@@
 			)
 		)
-		(property "LCSC MANUFACTURER " "YAGEO "
-			(at 60.706 164.338 0)
+		(property "LCSC Part # " "C14663 "
+			(at 60.96 162.306 0)
 			(effects
 				(font
@@
 			)
 		)
-		(property "LCSC Part #" "C15850 "
-			(at 95.25 193.294 0)
+		(property "LCSC MPN " "CL21A106KAYNNNE "
+			(at 95.758 188.976 0)
 			(effects
 				(font
@@
 			)
 		)
-		(property "LCSC MPN " "CL21A106KAYNNNE "
-			(at 95.758 188.976 0)
+		(property "LCSC MANUFACTURER " "SAMSUNG "
+			(at 95.504 191.262 0)
 			(effects
 				(font
@@
 			)
 		)
-		(property "LCSC MANUFACTURER " "SAMSUNG "
-			(at 95.504 191.262 0)
+		(property "LCSC Part # " "C15850 "
+			(at 95.25 193.294 0)
 			(effects
 				(font
@@
 			)
 		)
-		(property "LCSC Part #" "C15850 "
-			(at 69.85 193.294 0)
+		(property "LCSC MPN " "CL21A106KAYNNNE "
+			(at 70.358 188.976 0)
 			(effects
 				(font
@@
 			)
 		)
-		(property "LCSC MPN " "CL21A106KAYNNNE "
-			(at 70.358 188.976 0)
+		(property "LCSC MANUFACTURER " "SAMSUNG "
+			(at 70.104 191.262 0)
 			(effects
 				(font
@@
 			)
 		)
-		(property "LCSC MANUFACTURER " "SAMSUNG "
-			(at 70.104 191.262 0)
+		(property "LCSC Part # " "C15850 "
+			(at 69.85 193.294 0)
 			(effects
 				(font
@@
 			)
 		)
-		(property "LCSC Part #" "C14663 "
-			(at 154.94 162.306 0)
+		(property "LCSC MPN " "CC0603KRX7R9BB104 "
+			(at 154.432 166.624 0)
 			(effects
 				(font
@@
 			)
 		)
-		(property "LCSC MPN " "CC0603KRX7R9BB104 "
-			(at 154.432 166.624 0)
+		(property "LCSC MANUFACTURER " "YAGEO "
+			(at 154.686 164.338 0)
 			(effects
 				(font
@@
 			)
 		)
-		(property "LCSC MANUFACTURER " "YAGEO "
-			(at 154.686 164.338 0)
+		(property "LCSC Part # " "C14663 "
+			(at 154.94 162.306 0)
 			(effects
 				(font
@@
 			)
 		)
-		(property "LCSC Part #" "C14663 "
-			(at 34.29 162.306 0)
+		(property "LCSC MPN " "CC0603KRX7R9BB104 "
+			(at 33.782 166.624 0)
 			(effects
 				(font
@@
 			)
 		)
-		(property "LCSC MPN " "CC0603KRX7R9BB104 "
-			(at 33.782 166.624 0)
+		(property "LCSC MANUFACTURER " "YAGEO "
+			(at 34.036 164.338 0)
 			(effects
 				(font
@@
 			)
 		)
-		(property "LCSC MANUFACTURER " "YAGEO "
-			(at 34.036 164.338 0)
+		(property "LCSC Part # " "C14663 "
+			(at 34.29 162.306 0)
 			(effects
 				(font
@@
 			)
 		)
-		(property "LCSC Part #" "C14663 "
-			(at 52.07 162.306 0)
+		(property "LCSC MPN " "CC0603KRX7R9BB104 "
+			(at 51.562 166.624 0)
 			(effects
 				(font
@@
 			)
 		)
-		(property "LCSC MPN " "CC0603KRX7R9BB104 "
-			(at 51.562 166.624 0)
+		(property "LCSC MANUFACTURER " "YAGEO "
+			(at 51.816 164.338 0)
 			(effects
 				(font
@@
 			)
 		)
-		(property "LCSC MANUFACTURER " "YAGEO "
-			(at 51.816 164.338 0)
+		(property "LCSC Part # " "C14663 "
+			(at 52.07 162.306 0)
 			(effects
 				(font
@@
 			)
 		)
-		(property "LCSC Part #" "C1634 "
-			(at 59.944 43.18 0)
+		(property "LCSC MPN " "CL10C100JB8NNNC "
+			(at 55.626 42.672 0)
 			(effects
 				(font
@@
 			)
 		)
-		(property "LCSC MPN " "CL10C100JB8NNNC "
-			(at 55.626 42.672 0)
+		(property "LCSC MANUFACTURER " "SAMSUNG "
+			(at 57.912 42.926 0)
 			(effects
 				(font
@@
 			)
 		)
-		(property "LCSC MANUFACTURER " "SAMSUNG "
-			(at 57.912 42.926 0)
+		(property "LCSC Part # " "C1634 "
+			(at 59.944 43.18 0)
 			(effects
 				(font
@@
 			)
 		)
-		(property "LCSC Part #" "C1634 "
-			(at 59.944 71.12 0)
+		(property "LCSC MPN " "CL10C100JB8NNNC "
+			(at 55.626 70.612 0)
 			(effects
 				(font
@@
 			)
 		)
-		(property "LCSC MPN " "CL10C100JB8NNNC "
-			(at 55.626 70.612 0)
+		(property "LCSC MANUFACTURER " "SAMSUNG "
+			(at 57.912 70.866 0)
 			(effects
 				(font
@@
 			)
 		)
-		(property "LCSC MANUFACTURER " "SAMSUNG "
-			(at 57.912 70.866 0)
+		(property "LCSC Part # " "C1634 "
+			(at 59.944 71.12 0)
 			(effects
 				(font
