File: HARDWARE/KICAD/EMBARCADOS - CURSO PCB.kicad_sch (KiCad schematic)
At the start: 14 parts, among them J1 DC BARREL JACK, U1 AP3012

Commit message: Finished 1st pass of the power circuits. 3 classes recorded.
Parts:
- removed R1: 10K 1%, EMBARCADOS - CURSO PCB:R_0603_1608Metric, symbol EMBARCADOS - CURSO PCB:RES 0603 10K 1% VISHAY CRCW060310K0FK
- added C3, C4, C5, C6: 10µF 16V, EMBARCADOS - CURSO PCB:C_0805_2012Metric, symbol EMBARCADOS - CURSO PCB:CAP 0805 10uH 16V AVX KGM21AR71C106K
- added R1: 47K 1%, EMBARCADOS - CURSO PCB:R_0603_1608Metric, symbol EMBARCADOS - CURSO PCB:RES 0603 47K 1% VISHAY CRCW060347K0FK
- added U2: LD1117S33TR, EMBARCADOS - CURSO PCB:SOT-223-3_TabPin2, symbol EMBARCADOS - CURSO PCB:IC DC-DC LDO LD1117S33TR SOT223
- added U3: LD1117S50TR, EMBARCADOS - CURSO PCB:SOT-223-3_TabPin2, symbol EMBARCADOS - CURSO PCB:IC DC-DC LDO LD1117S50TR SOT223
- JP1: value SolderJumper_2_Open -> BOOST IN
- JP2: value SolderJumper_2_Open -> BOOST OUT
Connections:
- net +VBOOST: now also C6.1, U3.3 (VI)
- net +VSEL: now also C3.1, U2.3 (VI)
- net GND: now also C3.2, C4.2, C5.2, C6.2, U2.1 (GND), U3.1 (GND)
- net BOOST IN: now reaches C1.1, JP1.2 (B), L1.1, R3.1, U1.5 (IN)
- net BOOST OUT: now reaches C2.1, D3.1 (K), JP2.1 (A)
- net BOOST OUT: now also R1.1
- net BOOST SW: now reaches D3.2 (A), L1.2, U1.1 (SW)
- net BOOST FB: now reaches R2.1, U1.3 (FB)
- net BOOST FB: now also R1.2
- net BOOST ~{SHDN}: now reaches R3.2, U1.4 (~{SHDN})
- new net +3.3V: C4.1, U2.2 (VO)
- new net +5V: C5.1, U3.2 (VO)
Other:
- note added: "BOOST OUT = 1.25 * (1 + R1/R2)"
- note removed: "VERIFICAR VALORES R1 E R2"
- moved on the sheet: C1, C2, D3, JP2, L1, R2, R3, U1

Commit message: Re-recorded class 07.03 due to audio error.
Parts:
- added C7: 10µF 16V, EMBARCADOS - CURSO PCB:C_0805_2012Metric, symbol EMBARCADOS - CURSO PCB:CAP 0805 10uH 16V AVX KGM21AR71C106K
- added FB1: 600R 800mA, EMBARCADOS - CURSO PCB:L_0603_1608Metric, symbol EMBARCADOS - CURSO PCB:FB 0603 600R 800mA WÜRTH ELEKTRONIK 742792651
- added LED1, LED2, LED3, LED4, LED5: RED, EMBARCADOS - CURSO PCB:LED_0603_1608Metric, symbol EMBARCADOS - CURSO PCB:LED 0603 RED WÜRTH ELEKTRONIK 150060SS55040
- added R4, R5, R6, R7, R8: 10K 1%, EMBARCADOS - CURSO PCB:R_0603_1608Metric, symbol EMBARCADOS - CURSO PCB:RES 0603 10K 1% VISHAY CRCW060310K0FK
Connections:
- net +3.3V: now also LED5.2 (A)
- net +5V: now also C6.1, FB1.1, LED4.2 (A); no longer C5.1
- net +VBOOST: now also C5.1, LED3.2 (A); no longer C6.1
- net +VEXT: now also LED1.2 (A)
- net GND: now also C7.2, R4.1, R5.1, R6.1, R7.1, R8.1
- new net: LED4.1 (K), R7.2
- new net: LED5.1 (K), R8.2
- new net: LED2.1 (K), R5.2
- new net: LED3.1 (K), R6.2
- new net: LED1.1 (K), R4.2
- new net +5VA: C7.1, FB1.2
Other:
- note added: "INCLUIR TEST POINTS"

Commit message: Added POWER and MCU sheets. Added MCU, decoupling capacitors and crystals.
Parts:
- removed BT1: CR2032, EMBARCADOS - CURSO PCB:BatteryHolder_Keystone_1060_1x2032, symbol EMBARCADOS - CURSO PCB:BATTERY HOLDER CR2032
- removed C1, C2, C3, C4, C5, C6, C7: 10µF 16V, EMBARCADOS - CURSO PCB:C_0805_2012Metric, symbol EMBARCADOS - CURSO PCB:CAP 0805 10uH 16V AVX KGM21AR71C106K
- removed D1, D2, D3: 1N5819HW, EMBARCADOS - CURSO PCB:D_SOD-123, symbol EMBARCADOS - CURSO PCB:DIODE SCHOTTKY 1N5819WS SOD-123 DIODES INC
- removed FB1: 600R 800mA, EMBARCADOS - CURSO PCB:L_0603_1608Metric, symbol EMBARCADOS - CURSO PCB:FB 0603 600R 800mA WÜRTH ELEKTRONIK 742792651
- removed J1: DC BARREL JACK, EMBARCADOS - CURSO PCB:BarrelJack_GCT_DCJ200-10-A_Horizontal, symbol EMBARCADOS - CURSO PCB:CONN DC BARREL JACK WÜRTH ELEKTRONIK 694108301002
- removed JP1: BOOST IN, EMBARCADOS - CURSO PCB:SolderJumper-2_P1.3mm_Open_RoundedPad1.0x1.5mm, symbol EMBARCADOS - CURSO PCB:AUX JUMPER SOLDER OPEN
- removed JP2: BOOST OUT, EMBARCADOS - CURSO PCB:SolderJumper-2_P1.3mm_Open_RoundedPad1.0x1.5mm, symbol EMBARCADOS - CURSO PCB:AUX JUMPER SOLDER OPEN
- removed L1: 10µH 650mA, EMBARCADOS - CURSO PCB:WE-LQS SMT Semi-Shielded Power Inductor, symbol EMBARCADOS - CURSO PCB:IND 2.5x2.0 10µH 650mA WÜRTH ELEKTRONIK 74404024100
- removed LED1, LED2, LED3, LED4, LED5: RED, EMBARCADOS - CURSO PCB:LED_0603_1608Metric, symbol EMBARCADOS - CURSO PCB:LED 0603 RED WÜRTH ELEKTRONIK 150060SS55040
- removed R1: 47K 1%, EMBARCADOS - CURSO PCB:R_0603_1608Metric, symbol EMBARCADOS - CURSO PCB:RES 0603 47K 1% VISHAY CRCW060347K0FK
- removed R2, R3, R4, R5, R6, R7, R8: 10K 1%, EMBARCADOS - CURSO PCB:R_0603_1608Metric, symbol EMBARCADOS - CURSO PCB:RES 0603 10K 1% VISHAY CRCW060310K0FK
- removed U1: AP3012, EMBARCADOS - CURSO PCB:SOT-23-5, symbol EMBARCADOS - CURSO PCB:IC DC-DC BOOST AP3012 DIODES
- removed U2: LD1117S33TR, EMBARCADOS - CURSO PCB:SOT-223-3_TabPin2, symbol EMBARCADOS - CURSO PCB:IC DC-DC LDO LD1117S33TR SOT223
- removed U3: LD1117S50TR, EMBARCADOS - CURSO PCB:SOT-223-3_TabPin2, symbol EMBARCADOS - CURSO PCB:IC DC-DC LDO LD1117S50TR SOT223
Connections:
- no-connect marks 1 -> 0
Other:
- added sheet MCU (MCU.kicad_sch)
- added sheet POWER (POWER.kicad_sch)
- note removed: "BOOST OUT = 1.25 * (1 + R1/R2)"
- note removed: "INCLUIR TEST POINTS"

Commit message: Recorded IO sheet class.
Other:
- added sheet IO (IO.kicad_sch)
Changed lines of the file:
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@@
+	)
+	(sheet
+		(at 160.02 25.4)
+		(size 41.91 30.48)
+		(fields_autoplaced yes)
+		(stroke
+			(width 0.1524)
+			(type solid)
+		)
+		(fill
+			(color 0 0 0 0.0000)
+		)
+		(property "Sheetname" "IO"
+			(at 160.02 24.6884 0)
+			(effects
+				(font
+					(size 1.27 1.27)
+				)
+				(justify left bottom)
+			)
+		)
+		(property "Sheetfile" "IO.kicad_sch"
+			(at 160.02 56.4646 0)
+			(effects
+				(font
+					(size 1.27 1.27)
+				)
+				(justify left top)
+			)
+		)
+		(instances
+			(project "EMBARCADOS - CURSO PCB"
+				(path "/d5268f1b-b782-4609-86ee-ff462c2ec1ad"
+					(page "4")
+				)
+			)
+		)
 	)
 	(sheet

Commit message: Added ANALOG and INTERFACE sheets.
Other:
- added sheet ANALOG (ANALOG.kicad_sch)
- added sheet INTERFACE (INTERFACE.kicad_sch)
Changed lines of the file:
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@@
+	)
+	(sheet
+		(at 97.79 87.63)
+		(size 41.91 35.56)
+		(fields_autoplaced yes)
+		(stroke
+			(width 0.1524)
+			(type solid)
+		)
+		(fill
+			(color 0 0 0 0.0000)
+		)
+		(property "Sheetname" "INTERFACE"
+			(at 97.79 86.9184 0)
+			(effects
+				(font
+					(size 1.27 1.27)
+				)
+				(justify left bottom)
+			)
+		)
+		(property "Sheetfile" "INTERFACE.kicad_sch"
+			(at 97.79 123.7746 0)
+			(effects
+				(font
+					(size 1.27 1.27)
+				)
+				(justify left top)
+			)
+		)
+		(instances
+			(project "EMBARCADOS - CURSO PCB"
+				(path "/d5268f1b-b782-4609-86ee-ff462c2ec1ad"
+					(page "6")
+				)
+			)
+		)
+	)
+	(sheet
+		(at 33.02 93.98)
+		(size 39.37 33.02)
+		(fields_autoplaced yes)
+		(stroke
+			(width 0.1524)
+			(type solid)
+		)
+		(fill
+			(color 0 0 0 0.0000)
+		)
+		(property "Sheetname" "ANALOG"
+			(at 33.02 93.2684 0)
+			(effects
+				(font
+					(size 1.27 1.27)
+				)
+				(justify left bottom)
+			)
+		)
+		(property "Sheetfile" "ANALOG.kicad_sch"
+			(at 33.02 127.5846 0)
+			(effects
+				(font
+					(size 1.27 1.27)
+				)
+				(justify left top)
+			)
+		)
+		(instances
+			(project "EMBARCADOS - CURSO PCB"
+				(path "/d5268f1b-b782-4609-86ee-ff462c2ec1ad"
+					(page "5")
+				)
+			)
+		)
 	)
 	(sheet

Commit message: Finished schematic.
Other:
- added sheet AUXILIAR (AUXILIAR.kicad_sch)
Changed lines of the file:
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@@
 	)
 	(sheet
-		(at 33.02 25.4)
-		(size 39.37 30.48)
+		(at 38.1 25.4)
+		(size 63.5 50.8)
 		(fields_autoplaced yes)
 		(stroke
@@
 		)
 		(property "Sheetname" "POWER"
-			(at 33.02 24.6884 0)
+			(at 38.1 24.6884 0)
 			(effects
 				(font
@@
 		)
 		(property "Sheetfile" "POWER.kicad_sch"
-			(at 33.02 56.4646 0)
+			(at 38.1 76.7846 0)
 			(effects
 				(font
@@
 	)
 	(sheet
-		(at 160.02 25.4)
-		(size 41.91 30.48)
+		(at 190.5 25.4)
+		(size 63.5 50.8)
 		(fields_autoplaced yes)
 		(stroke
@@
 		)
 		(property "Sheetname" "IO"
-			(at 160.02 24.6884 0)
+			(at 190.5 24.6884 0)
 			(effects
 				(font
@@
 		)
 		(property "Sheetfile" "IO.kicad_sch"
-			(at 160.02 56.4646 0)
+			(at 190.5 76.7846 0)
 			(effects
 				(font
@@
 	)
 	(sheet
-		(at 97.79 87.63)
-		(size 41.91 35.56)
+		(at 114.3 88.9)
+		(size 63.5 50.8)
 		(fields_autoplaced yes)
 		(stroke
@@
 		)
 		(property "Sheetname" "INTERFACE"
-			(at 97.79 86.9184 0)
+			(at 114.3 88.1884 0)
 			(effects
 				(font
@@
 		)
 		(property "Sheetfile" "INTERFACE.kicad_sch"
-			(at 97.79 123.7746 0)
+			(at 114.3 140.2846 0)
 			(effects
 				(font
@@
 	)
 	(sheet
-		(at 33.02 93.98)
-		(size 39.37 33.02)
+		(at 38.1 88.9)
+		(size 63.5 50.8)
 		(fields_autoplaced yes)
 		(stroke
@@
 		)
 		(property "Sheetname" "ANALOG"
-			(at 33.02 93.2684 0)
+			(at 38.1 88.1884 0)
 			(effects
 				(font
@@
 		)
 		(property "Sheetfile" "ANALOG.kicad_sch"
-			(at 33.02 127.5846 0)
+			(at 38.1 140.2846 0)
 			(effects
 				(font
@@
 	)
 	(sheet
-		(at 97.79 25.4)
-		(size 40.64 30.48)
+		(at 114.3 25.4)
+		(size 63.5 50.8)
 		(fields_autoplaced yes)
 		(stroke
@@
 		)
 		(property "Sheetname" "MCU"
-			(at 97.79 24.6884 0)
+			(at 114.3 24.6884 0)
 			(effects
 				(font
@@
 		)
 		(property "Sheetfile" "MCU.kicad_sch"
-			(at 97.79 56.4646 0)
+			(at 114.3 76.7846 0)
 			(effects
 				(font
@@
 				)
 			)
+		)
+	)
+	(sheet
+		(at 190.5 88.9)
+		(size 63.5 50.8)
+		(fields_autoplaced yes)
+		(stroke
+			(width 0.1524)
+			(type solid)
+		)
+		(fill
+			(color 0 0 0 0.0000)
+		)
+		(property "Sheetname" "AUXILIAR"
+			(at 190.5 88.1884 0)
+			(effects
+				(font
+					(size 1.27 1.27)
+				)
+				(justify left bottom)
+			)
+		)
+		(property "Sheetfile" "AUXILIAR.kicad_sch"
+			(at 190.5 140.2846 0)
+			(effects
+				(font
+					(size 1.27 1.27)
+				)
+				(justify left top)
+			)
+		)
+		(instances
+			(project "EMBARCADOS - CURSO PCB"
+				(path "/d5268f1b-b782-4609-86ee-ff462c2ec1ad"
+					(page "7")
+				)
+			)
