File: HARDWARE/KICAD/EMBARCADOS - CURSO PCB.kicad_sch (KiCad schematic)
At the start: 0 parts

Commit message: Revision 02: fixed minor issues with D2 and U6 symbols/footprints. Generated new gerber and Drill files. Generated new PDF files of schematic and layout.
Changed lines of the file:
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@@
 	(title_block
 		(title "EMBARCADOS - CURSO PCB")
-		(date "2025-01-05")
-		(rev "01")
+		(date "2025-02-09")
+		(rev "02")
 		(company "Mechatronix Lab")
 		(comment 1 "Eng. André A. M. Araújo")
 	)
+	(text_box "Revision Log:\nRev: 00 - Initial Release\nRev: 01 - Improved images on silkscreen\nRev: 02 - Corrected minor issues on D2 and U6 symbols/footprints"
+		(exclude_from_sim no)
+		(at 177.8 154.94 0)
+		(size 106.68 10.16)
+		(stroke
+			(width 0)
+			(type default)
+		)
+		(fill
+			(type none)
+		)
+		(effects
+			(font
+				(size 1.27 1.27)
+			)
+			(justify left top)
+		)
+	)
 	(sheet
