File: HARDWARE/KICAD/EMBARCADOS - CURSO PCB.kicad_pcb (KiCad board)
At the start: 4 copper layers, 100 x 90 mm, 178 parts, among them J1 3V-7V, J2 Conn_01x20_Socket, J3 Conn_01x20_Socket, J4 USB_C_Receptacle_USB2.0_16P, J5 Micro_SD_Card_Det1, J6 CONN 02x05 ODD EVEN, Q1 2N7002K, Q2 2N7002K, Q3 2N7002K, SW1 UP, SW2 DOWN, SW3 LEFT, SW4 RIGHT, SW5 CENTER, SW6 BUTTON 1, SW7 BUTTON 2, SW8 ~{RST}, SW9 BOOT, U1 LD1117S33TR, U2 AP3012, U3 LD1117S50TR, U4 STM32F411RET6, U5 USBLC6-2SC6, U6 LMV324, U7 ADS1115, U8 OLED 1.3" 128x64, Y1 12MHz 18pF, Y2 32.768kHz 12.5pF

Commit message: Recorded Class 08.06 Part 1.
Parts:
- J2, J3: value Conn_01x20_Socket -> Conn_02x20_Odd_Even; footprint EMBARCADOS - CURSO PCB:PinSocket_1x20_P2.54mm_Horizontal -> EMBARCADOS - CURSO PCB:PinSocket_2x20_P2.54mm_Horizontal
- moved J3 95.0 mm to (125.8, 140.4), turned to 90 degrees
- moved J2 94.2 mm to (173.2, 59.6), turned to -90 degrees
- moved R9 3.95 mm to (135.8, 99.8)
- moved C18 3.86 mm to (137.2, 97.2), turned to 90 degrees
- moved C19 3.76 mm to (131.5, 97.2), turned to -90 degrees
- moved LED4 3.00 mm to (121.5, 75.0)
- moved R4 2.50 mm to (121.5, 78.0)
- moved C44 2.36 mm to (141.5, 99.8), turned to 0 degrees
- moved LED5 2.25 mm to (169.5, 75.8)
- moved R5 2.00 mm to (169.5, 79.0)
- moved R33 1.94 mm to (165.5, 64.2)
- moved R32 1.94 mm to (168.0, 64.2)
- moved R34 1.94 mm to (163.0, 64.2)
- moved R35 1.94 mm to (160.5, 64.2)
- moved R36 1.94 mm to (155.0, 63.7)
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Connections:
- J2 pad 1: PA0 -> +3.3V
- J2 pad 10: SPI MISO -> GND
- J2 pad 11: SPI MOSI -> /IO/NRST CONN
- J2 pad 12: SPI SCK -> GND
- J2 pad 13: SPI NSS -> DEBUG TX
- J2 pad 14: PWM RED -> GND
- J2 pad 15: PWM GREEN -> /IO/RX CONN
- J2 pad 16: PWM BLUE -> GND
- J2 pad 17: PWM BUZZER -> I2C SDA 3.3V
- J2 pad 18: USB OTG ID -> GND
- J2 pad 19: GND -> I2C SCL 3.3V
- J2 pad 2: PA1 -> GND
- J2 pad 20: +3.3V -> GND
- J2 pad 3: PA2 -> GND
- J2 pad 4: PA3 -> GND
- J2 pad 5: PA4 -> /IO/SWDIO CONN
- J2 pad 6: PA5 -> GND
- J2 pad 7: PA6 -> /IO/SWCLK CONN
- J2 pad 8: PA7 -> GND
- J2 pad 9: GND -> /IO/SWO CONN
- J3 pad 1: +3.3V -> PA0
- J3 pad 10: I2C SCL 3.3V -> GND
- J3 pad 11: PC3 -> PA5
- J3 pad 12: PC2 -> GND
- J3 pad 13: PC1 -> PA6
- J3 pad 14: PC0 -> GND
- J3 pad 15: GND -> PA7
- J3 pad 16: I2C SDA 5V -> GND
- J3 pad 17: I2C SCL 5V -> GND
- J3 pad 18: NEOPIXEL DIN -> GND
- J3 pad 19: NEOPIXEL DOUT -> SPI MISO
- J3 pad 20: +5V -> GND
- J3 pad 3: /IO/SWDIO CONN -> PA1
- J3 pad 4: /IO/SWCLK CONN -> GND
- J3 pad 5: /IO/SWO CONN -> PA2
- J3 pad 6: /IO/NRST CONN -> GND
- J3 pad 7: DEBUG TX -> PA3
- J3 pad 8: /IO/RX CONN -> GND
- J3 pad 9: I2C SDA 3.3V -> PA4
- L2 pad 1: unconnected-(L2-Pad1) -> /IO/USB DATA FLT +
- L2 pad 2: unconnected-(L2-Pad2) -> USB D+
- L2 pad 3: unconnected-(L2-Pad3) -> USB D-
- L2 pad 4: unconnected-(L2-Pad4) -> /IO/USB DATA FLT -
Routing:
- net GND: track 0.00 -> 42.4 mm
- net +3.3V: track 0.00 -> 27.7 mm
- net +5V: track 0.00 -> 13.5 mm
- net /MCU/LSE OUT: track 0.00 -> 10.0 mm
- net /MCU/HSE IN: track 0.00 -> 9.63 mm
- net /MCU/MCU PB12: track 0.00 -> 9.35 mm
- net DEBUG RX: track 0.00 -> 8.70 mm
- net /MCU/LSE IN: track 0.00 -> 8.67 mm
- net /POWER/BOOST FB: track 0.00 -> 8.54 mm
- net /POWER/BOOST IN: track 0.00 -> 8.38 mm
- net /MCU/HSE OUT: track 0.00 -> 8.16 mm
- net /MCU/MCU PB13: track 0.00 -> 8.06 mm
- net +VBOOST: track 0.00 -> 8.03 mm
- net /MCU/MCU PB15: track 0.00 -> 7.85 mm
- net /MCU/MCU PC6: track 0.00 -> 7.43 mm
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
Commit message: Recorded Class 08.06 Part 2.
Parts:
- moved TP3 19.6 mm to (177.2, 89.8)
- moved R30 13.1 mm to (182.0, 116.8), turned to 0 degrees
- moved R2 13.0 mm to (178.0, 86.5), turned to 90 degrees
- moved LED2 11.3 mm to (179.8, 84.2), turned to 0 degrees
- moved R29 10.8 mm to (182.0, 115.2), turned to 0 degrees
- moved TP2 8.00 mm to (188.5, 82.0)
- moved LED1 7.46 mm to (183.8, 84.2)
- moved D2 7.16 mm to (180.5, 81.0), turned to -90 degrees
- moved R1 6.08 mm to (185.0, 82.0), turned to -90 degrees
- moved TP4 5.59 mm to (175.0, 82.5)
- moved D1 4.03 mm to (183.0, 81.0), turned to -90 degrees
- moved TP15 3.47 mm to (171.5, 82.2)
- moved R27 2.71 mm to (182.2, 107.5), turned to 0 degrees
- moved R28 2.47 mm to (179.8, 107.8)
- moved C27 2.37 mm to (182.2, 105.2)
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Routing:
- net SPI MISO: track 0.00 -> 30.7 mm
- net USB D-: track 0.00 -> 28.0 mm
- net USB D+: track 0.00 -> 28.0 mm
- net SPI NSS: track 0.00 -> 25.0 mm, vias 0 -> 2
- net SPI SCK: track 0.00 -> 23.6 mm
- net SPI MOSI: track 0.00 -> 23.5 mm
- net +VBUS: track 0.00 -> 18.5 mm
- net PWM BLUE: track 0.00 -> 18.5 mm
- net +VEXT: track 0.00 -> 17.2 mm
- net PWM GREEN: track 0.00 -> 10.8 mm
- net PWM RED: track 0.00 -> 10.6 mm
- net +VSEL: track 2.52 -> 11.6 mm
- net +VBUSF: track 0.00 -> 7.21 mm
- net /IO/USB DATA+: track 0.00 -> 6.44 mm
- net /IO/USB DATA-: track 0.00 -> 5.70 mm
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
Commit message: Recorded Class 08.06 Part 3.
Parts:
- moved R55 9.66 mm to (164.5, 80.0)
- moved SW9 9.66 mm to (164.5, 75.5)
- moved C7 6.29 mm to (124.0, 78.7)
- moved FB1 6.29 mm to (125.0, 75.7)
- moved C4 5.56 mm to (127.5, 73.0)
- moved C5 5.56 mm to (124.0, 73.0)
- moved LED4 5.56 mm to (121.2, 69.5)
- moved R4 5.56 mm to (121.2, 72.5)
- moved TP12 5.56 mm to (118.8, 69.0)
- moved U3 5.56 mm to (125.8, 67.5)
- moved C45 5.55 mm to (133.2, 67.0), turned to 180 degrees
- moved R54 4.95 mm to (159.0, 80.0), turned to 180 degrees
- moved SW8 4.95 mm to (159.0, 75.5)
- moved C43 3.78 mm to (147.5, 82.2)
- moved R20 2.75 mm to (153.0, 91.8)
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Routing:
- net BUTTON CENTER: track 0.00 -> 61.4 mm
- net I2C SCL 5V: track 0.00 -> 58.5 mm
- net I2C SDA 5V: track 0.00 -> 58.5 mm
- net BUTTON LEFT: track 0.00 -> 52.4 mm
- net I2C SCL 3.3V: track 0.00 -> 51.4 mm
- net NEOPIXEL DIN: track 0.00 -> 49.8 mm, vias 0 -> 2
- net USB OTG ID: track 0.00 -> 49.1 mm, vias 0 -> 2
- net I2C SDA 3.3V: track 0.00 -> 48.6 mm
- net SPI SCK: track 23.6 -> 72.0 mm, vias 0 -> 1
- net BUTTON DOWN: track 0.00 -> 44.4 mm
- net BUTTON 2: track 0.00 -> 43.8 mm, vias 0 -> 2
- net SPI MOSI: track 23.5 -> 67.0 mm, vias 0 -> 1
- net SWDIO: track 0.00 -> 40.7 mm
- net BUTTON UP: track 0.00 -> 39.1 mm
- net SPI MISO: track 30.7 -> 69.5 mm, vias 0 -> 1
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
Commit message: Recorded Class 08.06 Part 4.
Parts:
- moved C38 6.73 mm to (115.0, 94.2), turned to -90 degrees
- moved TP13 3.25 mm to (108.0, 108.8)
- moved C39 1.75 mm to (118.8, 100.0)
- moved U7 1.75 mm to (121.8, 100.0)
- moved TP15 1.58 mm to (170.0, 82.8)
- moved C40 1.50 mm to (124.5, 100.0)
- moved C29 1.03 mm to (119.5, 94.2)
- moved C31 1.03 mm to (110.5, 94.2)
- moved C32 1.03 mm to (113.5, 94.2)
- moved R39 1.03 mm to (112.0, 91.2)
- moved R40 1.03 mm to (112.0, 94.2)
- moved TP14 1.00 mm to (132.0, 104.5)
- moved C30 0.55 mm to (116.5, 94.2)
- moved R37 0.55 mm to (118.0, 91.2)
- moved R38 0.55 mm to (118.0, 94.2)
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Routing:
- net +3.3V: track 39.4 -> 263.8 mm, vias 0 -> 19
- net +VBOOST: track 8.03 -> 103.3 mm, vias 0 -> 1
- net +5VA: track 0.00 -> 62.1 mm, vias 0 -> 5
- net +3VBAT: track 0.00 -> 12.2 mm, vias 0 -> 1
- net GND: track 52.4 -> 60.0 mm, vias 22 -> 31
- net /INTERFACE/BUZZER DRAIN: track 0.00 -> 3.87 mm
- net +5V: track 16.8 -> 18.8 mm
- net I2C SCL 5V: track 58.5 -> 60.2 mm
- net I2C SDA 5V: track 58.5 -> 60.1 mm

Commit message: Recorded Class 08.06 Part 6.
Parts:
- moved Y2 3.95 mm to (135.8, 90.2)
- moved C16 3.40 mm to (137.8, 92.5)
- moved C17 2.50 mm to (135.0, 94.5)
- moved C15 2.26 mm to (140.8, 94.2)
- moved TP9 2.02 mm to (197.0, 124.8)
- moved TP1 1.68 mm to (191.5, 123.8)
- moved R2 1.58 mm to (177.5, 85.0)
- moved C35 1.50 mm to (119.0, 106.0)
- moved C8 0.75 mm to (145.8, 108.5)
Routing:
- net PWM BUZZER: track 0.00 -> 132.3 mm, vias 0 -> 3
- net PC3: track 0.00 -> 61.7 mm, vias 0 -> 2
- net PWM GREEN: track 10.8 -> 66.4 mm, vias 0 -> 1
- net +3.3V: track 263.8 -> 317.6 mm, vias 19 -> 21
- net PWM RED: track 10.6 -> 63.6 mm, vias 0 -> 1
- net PWM BLUE: track 18.5 -> 70.2 mm, vias 0 -> 1
- net PC2: track 0.00 -> 51.7 mm, vias 0 -> 2
- net PC0: track 0.00 -> 51.4 mm, vias 0 -> 2
- net PC1: track 0.00 -> 50.2 mm, vias 0 -> 2
- net BUTTON RIGHT: track 26.2 -> 74.6 mm
- net PA0: track 0.00 -> 46.8 mm, vias 0 -> 1
- net PA1: track 0.00 -> 44.9 mm, vias 0 -> 1
- net PA2: track 0.00 -> 43.3 mm, vias 0 -> 1
- net PA3: track 0.00 -> 41.3 mm, vias 0 -> 1
- net PA4: track 0.00 -> 40.2 mm, vias 0 -> 1
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
Commit message: Recorded Class 08.07 Part 1.
Routing:
- net +5V: track 23.8 -> 31.3 mm, vias 0 -> 2
- net +VBOOST: track 103.3 -> 100.3 mm
- net GND: track 61.3 -> 63.8 mm, vias 40 -> 47
- net PC0: track 51.4 -> 49.0 mm
- net PC3: track 61.7 -> 59.6 mm
- net I2C SCL 5V: track 60.2 -> 58.5 mm
- net I2C SDA 5V: track 60.1 -> 58.5 mm
- net PC2: track 51.7 -> 50.9 mm
- net I2C SCL 3.3V: track 51.4 -> 50.8 mm

Commit message: Refactoring.
Parts:
- moved TP13 20.2 mm to (105.5, 88.8)
- moved R52 9.19 mm to (178.5, 125.0), turned to -90 degrees
- moved U1 8.29 mm to (174.1, 65.7)
- moved C1 8.25 mm to (176.0, 71.2)
- moved C3 8.25 mm to (172.2, 71.2)
- moved R50 7.00 mm to (126.5, 125.0)
- moved TP22 6.93 mm to (130.0, 107.5)
- moved R51 5.70 mm to (120.0, 129.5), turned to 180 degrees
- moved C19 5.48 mm to (135.2, 101.2), turned to 0 degrees
- moved Y2 5.35 mm to (139.0, 94.5)
- moved SW6 5.00 mm to (175.0, 125.0), turned to 90 degrees
- moved SW7 5.00 mm to (185.0, 125.0), turned to -90 degrees
- moved C17 4.26 mm to (138.2, 91.8), turned to -90 degrees
- moved R53 3.81 mm to (181.5, 125.0), turned to -90 degrees
- moved C43 3.78 mm to (147.5, 86.0)
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Routing:
- net GND: track 63.8 -> 127.1 mm, vias 47 -> 90
- net BUTTON RIGHT: track 74.6 -> 40.4 mm, vias 0 -> 2
- net +3.3V: track 317.6 -> 287.2 mm, vias 21 -> 19
- net +3.3VA: track 7.02 -> 17.6 mm
- net +5VA: track 62.1 -> 55.4 mm, vias 5 -> 3
- net PWM BLUE: track 70.2 -> 63.6 mm
- net PWM GREEN: track 66.4 -> 59.9 mm
- net /MCU/LSE OUT: track 14.7 -> 8.51 mm
- net BUTTON 1: track 33.2 -> 39.1 mm
- net +VSEL: track 11.6 -> 17.4 mm
- net +3VBAT: track 12.8 -> 18.5 mm
- net /MCU/LSE IN: track 11.9 -> 6.39 mm
- net PWM RED: track 63.6 -> 58.2 mm
- net A3: track 19.0 -> 23.8 mm
- net SPI NSS: track 63.5 -> 58.9 mm
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
Commit message: Refactoring.
Parts:
- moved R5 10.7 mm to (171.5, 68.5), turned to 0 degrees
- moved LED5 8.81 mm to (174.5, 68.5), turned to 0 degrees
- moved C4 8.28 mm to (126.2, 79.2)
- moved C5 8.23 mm to (122.8, 79.2)
- moved U1 8.16 mm to (175.5, 73.8)
- moved U3 8.16 mm to (124.5, 73.8)
- moved C3 8.12 mm to (173.7, 79.2)
- moved C1 8.08 mm to (177.1, 79.2)
- moved TP12 8.01 mm to (119.8, 61.0)
- moved FB1 6.17 mm to (123.8, 81.8)
- moved C7 5.68 mm to (122.8, 84.2)
- moved TP3 5.51 mm to (177.5, 84.2)
- moved TP4 5.48 mm to (173.8, 84.2)
- moved R2 4.25 mm to (181.8, 85.0), turned to -90 degrees
- moved R4 3.96 mm to (121.5, 68.5), turned to 0 degrees
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Routing:
- net SD CARD ~{IN}: track 2.66 -> 59.6 mm, vias 0 -> 2
- net GND: track 127.1 -> 183.9 mm, vias 90 -> 129
- net NRST: track 20.5 -> 53.5 mm, vias 0 -> 4
- net +3.3V: track 287.2 -> 301.3 mm, vias 19 -> 20
- net +5V: track 26.9 -> 40.1 mm, vias 2 -> 0
- net BOOT0: track 28.4 -> 38.6 mm
- net BUTTON 1: track 39.1 -> 47.0 mm
- net BUTTON 2: track 46.1 -> 54.1 mm
- net +VBUS: track 18.5 -> 25.3 mm
- net I2C SCL 5V: track 58.5 -> 52.2 mm
- net NEOPIXEL DIN: track 49.1 -> 55.2 mm
- net PWM GREEN: track 59.9 -> 53.9 mm
- net +VEXT: track 17.2 -> 12.1 mm
- net +5VA: track 55.4 -> 51.1 mm, vias 3 -> 2
- net PWM BUZZER: track 128.3 -> 132.4 mm
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