File: HARDWARE/KICAD/EMBARCADOS - CURSO PCB.kicad_pcb (KiCad board)
At the start: 4 copper layers, 100 x 90 mm, 178 parts, among them J1 3V-7V, J2 Conn_02x20_Odd_Even, J3 Conn_02x20_Odd_Even, J4 USB_C_Receptacle_USB2.0_16P, J5 Micro_SD_Card_Det1, J6 CONN 02x05 ODD EVEN, Q1 2N7002K, Q2 2N7002K, Q3 2N7002K, SW1 UP, SW2 DOWN, SW3 LEFT, SW4 RIGHT, SW5 CENTER, SW6 BUTTON 1, SW7 BUTTON 2, SW8 ~{RST}, SW9 BOOT, U1 LD1117S33TR, U2 AP3012, U3 LD1117S50TR, U4 STM32F411RET6, U5 USBLC6-2SC6, U6 LMV324, U7 ADS1115, U8 OLED 1.3" 128x64, Y1 12MHz 18pF, Y2 32.768kHz 12.5pF

Commit message: Routing detailing before Class 08.07 Part 2.
Parts:
- moved TP15 26.2 mm to (177.8, 59.2)
- moved TP12 2.92 mm to (122.2, 59.5)
- moved TP13 1.60 mm to (104.5, 90.0)
- moved LED5 1.00 mm to (175.5, 68.5)
- moved R5 1.00 mm to (172.5, 68.5)
- moved J1 0.50 mm to (187.5, 77.5)
- moved J4 0.32 mm to (197.2, 92.5)
Routing:
- net GND: track 183.9 -> 203.0 mm, vias 129 -> 150
- net +3.3V: track 301.3 -> 306.4 mm
- net +VBOOST: track 95.9 -> 99.4 mm
- net A0: track 23.8 -> 25.7 mm
- net A3: track 23.8 -> 25.5 mm
- net PWM BUZZER: track 132.4 -> 130.9 mm
- net +5VA: track 51.1 -> 52.4 mm
- net +VBUS: track 25.3 -> 25.9 mm

Commit message: Refactoring before Class 08.07 Part 3.
Parts:
- moved TP10 18.0 mm to (184.6, 142.5)
- moved TP6 18.0 mm to (180.3, 142.5)
- moved TP1 17.7 mm to (180.3, 137.8)
- moved TP9 17.7 mm to (184.6, 137.8)
- moved TP12 5.94 mm to (120.0, 65.0)
- moved TP7 5.77 mm to (188.4, 137.8)
- moved C41 5.00 mm to (113.0, 72.5)
- moved LS1 5.00 mm to (110.0, 75.0)
- moved Q3 5.00 mm to (113.0, 75.5)
- moved R45 5.00 mm to (110.0, 75.0)
- moved R46 5.00 mm to (116.0, 75.5)
- moved FID3 5.00 mm to (104.0, 137.0)
- moved R47 5.00 mm to (115.0, 118.5)
- moved R48 5.00 mm to (115.0, 131.5)
- moved R49 5.00 mm to (108.5, 125.0)
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Routing:
- net GND: track 203.0 -> 211.5 mm, vias 150 -> 164
- net BUTTON LEFT: track 60.3 -> 67.5 mm
- net BUTTON UP: track 47.2 -> 54.0 mm
- net PWM BUZZER: track 130.9 -> 124.1 mm
- net BUTTON RIGHT: track 40.4 -> 46.9 mm
- net BUTTON CENTER: track 69.8 -> 76.2 mm
- net BUTTON DOWN: track 52.0 -> 58.5 mm
- net PA0: track 48.4 -> 42.1 mm
- net USB OTG ID: track 49.1 -> 44.0 mm
- net BUTTON 2: track 54.1 -> 59.1 mm
- net BUTTON 1: track 47.0 -> 52.0 mm
- net DEBUG RX: track 34.1 -> 29.4 mm
- net PA4: track 40.3 -> 35.7 mm
- net SPI MISO: track 69.8 -> 65.3 mm
- net PWM GREEN: track 53.9 -> 49.4 mm
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
Commit message: Refactoring before Class 08.07 Part 3.
Routing:
- net GND: track 211.5 -> 214.3 mm
Changed lines of the file:
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@@
 	)
 	(segment
+		(start 139 110)
+		(end 138.5 109.5)
+		(width 0.7)
+		(layer "F.Cu")
+		(net 1)
+	)
+	(segment
 		(start 182.5 84.175)
 		(end 183.25 84.175)
@@
 	)
 	(segment
+		(start 138.5 108.7)
+		(end 137.55 107.75)
+		(width 0.7)
+		(layer "F.Cu")
+		(net 1)
+	)
+	(segment
 		(start 134.475 99.425)
 		(end 134.4 99.35)
@@
 	)
 	(segment
+		(start 138.5 109.5)
+		(end 138.5 108.7)
+		(width 0.7)
+		(layer "F.Cu")
+		(net 1)
+	)
+	(segment
 		(start 136.025 94)
 		(end 136.025 95.25)
@@
 	)
 	(via
-		(at 138.75 109.75)
+		(at 139 110)
 		(size 0.7)
 		(drill 0.3)
@@
 	)
 	(segment
+		(start 146 109)
+		(end 146 108.5)
+		(width 0.7)
+		(layer "B.Cu")
+		(net 5)
+	)
+	(segment
+		(start 146 108.5)
+		(end 150 104.5)
+		(width 0.7)
+		(layer "B.Cu")
+		(net 5)
+	)
+	(segment
+		(start 139.5 109)
+		(end 132 109)
+		(width 0.7)
+		(layer "B.Cu")
+		(net 5)
+	)
+	(segment
 		(start 109.5 125)
 		(end 115 130.5)
@@
 	)
 	(segment
-		(start 150 105)
-		(end 150.5 105.5)
+		(start 151 105.5)
+		(end 156 105.5)
 		(width 0.7)
 		(layer "B.Cu")
@@
 	)
 	(segment
-		(start 150 104)
-		(end 150 96.25)
-		(width 0.7)
-		(layer "B.Cu")
-		(net 5)
-	)
-	(segment
 		(start 180.5 117)
 		(end 185 121.5)
@@
 	)
 	(segment
-		(start 121.5 119.5)
-		(end 121.5 123)
+		(start 137.75 81.5)
+		(end 137.75 80.25)
 		(width 0.7)
 		(layer "B.Cu")
@@
 	)
 	(segment
-		(start 137.75 81.5)
-		(end 137.75 80.25)
+		(start 140 108.5)
+		(end 146 108.5)
 		(width 0.7)
 		(layer "B.Cu")
@@
 	)
 	(segment
-		(start 139.5 109)
-		(end 146 109)
+		(start 184.25 111)
+		(end 184.25 111.05)
 		(width 0.7)
 		(layer "B.Cu")
@@
 	)
 	(segment
-		(start 150 105)
-		(end 150 104)
+		(start 146 109)
+		(end 146 109.5)
 		(width 0.7)
 		(layer "B.Cu")
@@
 	)
 	(segment
-		(start 184.25 111)
-		(end 184.25 111.05)
+		(start 121.5 119.5)
+		(end 121.5 123)
 		(width 0.7)
 		(layer "B.Cu")
@@
 	)
 	(segment
-		(start 146 109)
-		(end 146 109.5)
+		(start 145 91)
+		(end 145 91.272793)
 		(width 0.7)
 		(layer "B.Cu")
@@
 	)
 	(segment
-		(start 145 91)
-		(end 145 91.272793)
+		(start 145.65 91.9)
+		(end 150 96.25)
 		(width 0.7)
 		(layer "B.Cu")
@@
 	)
 	(segment
-		(start 145.65 91.9)
-		(end 150 96.25)
+		(start 150 104.5)
+		(end 151 105.5)
 		(width 0.7)
 		(layer "B.Cu")
@@
 	)
 	(segment
-		(start 146 109)
-		(end 150 105)
+		(start 150 104.5)
+		(end 150 96.25)
 		(width 0.7)
 		(layer "B.Cu")
@@
 	)
 	(segment
-		(start 145.627207 91.9)
-		(end 145.65 91.9)
+		(start 139.5 109)
+		(end 140 108.5)
 		(width 0.7)
 		(layer "B.Cu")
@@
 	)
 	(segment
-		(start 158.8625 94.3875)
-		(end 157.75 95.5)
+		(start 145.627207 91.9)
+		(end 145.65 91.9)
 		(width 0.7)
 		(layer "B.Cu")
@@
 	)
 	(segment
-		(start 139.5 109)
-		(end 132 109)
+		(start 158.8625 94.3875)
+		(end 157.75 95.5)
 		(width 0.7)
 		(layer "B.Cu")
@@
 	)
 	(segment
-		(start 150.5 105.5)
-		(end 156 105.5)
-		(width 0.7)
-		(layer "B.Cu")
-		(net 5)
-	)
-	(segment
 		(start 132 109)
 		(end 121.5 119.5)
@@
 	)
 	(segment
-		(start 121.25 104.75)
-		(end 121.25 102.15)
+		(start 120.275 104.975)
+		(end 121.25 104)
 		(width 0.156464)
 		(layer "F.Cu")
@@
 	(segment
 		(start 119.5 104.975)
-		(end 121.025 104.975)
+		(end 120.275 104.975)
 		(width 0.156464)
 		(layer "F.Cu")
@@
 	)
 	(segment
-		(start 121.025 104.975)
-		(end 121.25 104.75)
+		(start 121.25 104)
+		(end 121.25 102.15)
 		(width 0.156464)
 		(layer "F.Cu")

Commit message: Refactoring before Class 08.07 Part 4.
Parts:
- moved TP17 13.2 mm to (178.0, 138.0)
- moved TP19 13.1 mm to (196.0, 70.0)
- moved TP20 12.0 mm to (122.0, 138.0)
- moved TP11 11.8 mm to (184.0, 133.0)
- moved TP10 10.5 mm to (187.8, 132.5)
- moved TP6 6.77 mm to (182.0, 136.0)
- moved FID3 5.10 mm to (109.0, 136.0)
- moved TP1 4.79 mm to (180.0, 133.0)
- moved TP7 4.58 mm to (191.0, 134.0)
- moved H2 4.50 mm to (196.0, 63.5)
- moved H3 4.50 mm to (104.0, 136.5)
- moved H4 4.50 mm to (196.0, 136.5)
- moved FID1 4.12 mm to (109.0, 64.0)
- moved H1 3.64 mm to (104.0, 63.5)
- moved TP8 1.77 mm to (190.0, 138.0)
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Routing:
- net GND: track 214.3 -> 222.2 mm, vias 164 -> 172
- net BUTTON LEFT: track 67.5 -> 65.6 mm
- net +VBUS: track 25.9 -> 25.1 mm
- net PA3: track 37.4 -> 36.6 mm
- net +3.3V: track 311.3 -> 312.0 mm, vias 21 -> 23
- added copper zone on B.Cu, net +3.3V
- added copper zone on In1.Cu, net GND
- added copper zone on In2.Cu, net GND
Other:
- board size 100 x 90 mm -> 100 x 81 mm

Commit message: Recorded Class 08.07 Part 5.
Parts:
- removed the TP1 at (180.0, 133.0)
- removed the TP10 at (187.8, 132.5)
- removed the TP11 at (184.0, 133.0)
- removed the TP6 at (182.0, 136.0)
- removed the TP7 at (191.0, 134.0)
- removed the TP8 at (190.0, 138.0)
- removed the TP9 at (186.0, 137.0)
- J3: renamed from J4; value USB_C_Receptacle_USB2.0_16P -> USB
- J5: value Micro_SD_Card_Det1 -> Micro SD
- renumbered C6 to C1, C1 to C10, C42 to C11, C7 to C12, C43 to C13, C26 to C14, C24 to C15, C17 to C16, C16 to C17, C11 to C18, C31 to C19, C45 to C2, C32 to C20, C38 to C21, C30 to C22, C29 to C23, C15 to C24, C18 to C26, C10 to C27, C44 to C28, C37 to C29, C41 to C3, C39 to C30, C40 to C31, C19 to C32, C14 to C33, C13 to C34, C27 to C35, C33 to C36, C34 to C37, C36 to C38, C35 to C39, C2 to C4, C9 to C40, C12 to C41, C21 to C42, C8 to C43, C20 to C44, C28 to C45, C4 to C6, C23 to C7, C22 to C8, C3 to C9, D3 to D1, D5 to D2, D2 to D3, D1 to D4, D4 to D5, FB4 to FB2, FB2 to FB4, J2 to J1, J1 to J2, J6 to J4, J3 to J6, JP2 to JP1, JP1 to JP2, LED3 to LED1, LED4 to LED2, LED5 to LED3, LED2 to LED4, LED1 to LED5, Q3 to Q1, Q1 to Q3, R3 to R1, R5 to R10, R45 to R11, R46 to R12, R6 to R13, R23 to R14, R54 to R15, R55 to R16, R21 to R17, R22 to R18, R24 to R19, R8 to R2, R2 to R20, R1 to R21, R15 to R22, R14 to R23, R26 to R24, R13 to R25, R20 to R26, R39 to R27, R37 to R28, R40 to R29, R7 to R3, R38 to R30, R25 to R31, R9 to R32, R19 to R33, R18 to R34, R17 to R35, R16 to R36, R10 to R37, R42 to R38, R44 to R39, R36 to R4, R28 to R40, R27 to R41, R11 to R42, R41 to R43, R43 to R44, R12 to R45, R31 to R46, R29 to R47, R30 to R48, R47 to R49, R35 to R5, R49 to R50, R50 to R51, R51 to R54, R48 to R55, R34 to R6, R33 to R7, R32 to R8, R4 to R9, SW8 to SW1, SW9 to SW2, SW1 to SW3, SW3 to SW4, SW4 to SW6, SW6 to SW7, SW7 to SW8, SW2 to SW9, TP15 to TP1, TP16 to TP10, TP14 to TP11, TP22 to TP12, TP21 to TP13, TP20 to TP14, TP17 to TP15, TP18 to TP2, TP12 to TP3, TP5 to TP4, TP19 to TP5, TP4 to TP6, TP3 to TP7, TP2 to TP8, TP13 to TP9, U2 to U1, U3 to U2, U1 to U3, U5 to U4, U6 to U5, U7 to U6, U4 to U7, Y2 to Y1, Y1 to Y2
Connections:
- U7 pad 2: /MCU/MCU PC13 -> unconnected-(U7-PC13-Pad2)
- U7 pad 29: /MCU/MCU PB10 -> unconnected-(U7-PB10-Pad29)
- U7 pad 52: /MCU/MCU PC11 -> unconnected-(U7-PC11-Pad52)
- U7 pad 53: /MCU/MCU PC12 -> unconnected-(U7-PC12-Pad53)
- U7 pad 54: /MCU/MCU PD2 -> unconnected-(U7-PD2-Pad54)
- U7 pad 56: /MCU/MCU PB4 -> unconnected-(U7-PB4-Pad56)
- U7 pad 57: /MCU/MCU PB5 -> unconnected-(U7-PB5-Pad57)
Routing:
- net +5VA: track 52.4 -> 71.9 mm
- net GND: track 222.2 -> 229.6 mm, vias 172 -> 177
- net +5V: track 43.0 -> 49.4 mm
- net +3.3V: track 312.0 -> 316.2 mm
- net +VBUSF: track 8.48 -> 10.0 mm
- net +VSEL: track 17.3 -> 18.8 mm
- net BOOT0: track 38.4 -> 38.9 mm

Commit message: Refactoring.
Parts:
- J4: value CONN 02x05 ODD EVEN -> ANALOG
- moved TP1 28.2 mm to (168.0, 89.0)
- moved TP14 21.1 mm to (102.0, 131.2)
- moved TP15 21.1 mm to (198.0, 131.2)
- moved TP9 18.5 mm to (122.8, 87.0)
- moved TP2 13.5 mm to (102.0, 68.8)
- moved TP11 11.4 mm to (132.0, 92.5)
- moved TP8 10.5 mm to (198.0, 85.0)
- moved TP7 4.78 mm to (177.0, 89.0)
- moved TP3 4.37 mm to (117.8, 68.8)
- moved TP12 3.61 mm to (132.0, 104.5)
- moved FID1 3.25 mm to (107.8, 61.0)
- moved FID2 3.25 mm to (192.2, 61.0)
- moved FID3 3.25 mm to (107.8, 139.0)
- moved TP6 3.25 mm to (177.0, 84.2)
- moved TP4 2.50 mm to (187.5, 62.5)
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Routing:
- net +5VA: track 71.9 -> 53.2 mm
- net +VEXT: track 11.9 -> 24.1 mm
- net +3VBAT: track 19.0 -> 22.7 mm
- net +3.3VA: track 17.6 -> 14.3 mm
- net +VSEL: track 18.8 -> 15.9 mm
- net +5V: track 49.4 -> 50.5 mm
- net +3.3V: track 316.2 -> 317.1 mm

Commit message: Refactoring after Class 08.07 Part 5.
Parts:
- removed the U4 at (187.5, 92.5)
- added D5: USBLC6-2SC6, EMBARCADOS - CURSO PCB:SOT-23-6, F.Cu at (187.5, 92.5)
- moved R10 2.03 mm to (166.5, 68.9)
- moved R7 2.03 mm to (158.9, 68.9)
- moved R9 2.03 mm to (164.0, 68.9)
- moved R8 2.03 mm to (161.4, 68.9)
- moved R6 1.59 mm to (155.1, 68.9)
- moved FID1 0.50 mm to (107.8, 60.5)
- moved FID2 0.50 mm to (192.2, 60.5)
- moved FID3 0.50 mm to (107.8, 139.5)
- moved H1 0.50 mm to (104.0, 63.0)
- moved H2 0.50 mm to (196.0, 63.0)
- moved H3 0.50 mm to (104.0, 137.0)
- moved H4 0.50 mm to (196.0, 137.0)
- renumbered D5 to D6, D6 to D7, R8 to R10, R9 to R4, R10 to R5, R4 to R6, R5 to R7, R6 to R8, R7 to R9, TP4 to TP1, TP11 to TP10, TP10 to TP11, TP5 to TP4, TP6 to TP5, TP8 to TP6, TP9 to TP7, TP1 to TP8, TP7 to TP9, U5 to U4, U6 to U5, U8 to U6
Routing:
- net SWCLK: track 31.4 -> 28.8 mm
- net SWDIO: track 36.5 -> 33.9 mm
- net /IO/SWDIO CONN: track 3.11 -> 5.23 mm
- net /IO/SWCLK CONN: track 3.11 -> 5.23 mm
- net /IO/NRST CONN: track 3.51 -> 5.62 mm
- net /IO/SWO CONN: track 3.11 -> 5.23 mm
- net NRST: track 49.2 -> 47.2 mm
- net SWO: track 31.6 -> 29.7 mm
- net /IO/RX CONN: track 3.11 -> 4.70 mm
- net DEBUG RX: track 29.4 -> 27.8 mm
- net BUTTON 1: track 52.0 -> 53.1 mm
- net +3.3V: track 317.1 -> 318.1 mm
- net BUTTON 2: track 59.1 -> 59.8 mm
- net GND: track 229.6 -> 229.8 mm, vias 177 -> 365
Other:
- board size 100 x 81 mm -> 100 x 82 mm

Commit message: Refactoring before Class 08.07 Part 6.
Parts:
- moved C30 0.10 mm to (118.9, 100.0)
Routing:
- net GND: track 229.8 -> 229.9 mm, vias 365 -> 357
