File: HARDWARE/KICAD/EMBARCADOS - CURSO PCB.kicad_pcb (KiCad board)
At the start: 4 copper layers, 100 x 82 mm, 173 parts, among them J1 Conn_02x20_Odd_Even, J2 3V-7V, J3 USB, J4 ANALOG, J5 Micro SD, J6 Conn_02x20_Odd_Even, Q1 2N7002K, Q2 2N7002K, Q3 2N7002K, SW1 ~{RST}, SW2 BOOT, SW3 UP, SW4 LEFT, SW5 CENTER, SW6 RIGHT, SW7 BUTTON 1, SW8 BUTTON 2, SW9 DOWN, U1 AP3012, U2 LD1117S50TR, U3 LD1117S33TR, U4 LMV324, U5 ADS1115, U6 OLED 1.3" 128x64, U7 STM32F411RET6, Y1 32.768kHz 12.5pF, Y2 12MHz 18pF

Commit message: Regenerated Gerber and Drill files.
Other:
- board text added: "Green"
- board text added: "White"
- board text added: "prepreg"
- board text removed: "prepreg - 3313"

Commit message: Updated logos with higher resolution images.
Parts:
- removed the G*** at (182.3, 96.7)
- added G***: LOGO, LOGO, F.Cu at (149.8, 96.7)
- added G***: LOGO, LOGO, B.Cu at (150.5, 97.2)
Other:
- board text added: "PROJETO DE PCB PARA SISTEMAS EMBARCADOS"
- board text removed: "CURSO - PROJETO DE PCB PARA SISTEMAS EMBARCADOS"

Commit message: Added QR code for project repo on GitHub. Changed board revision to 01 2025.01.05.
Parts:
- removed the G*** at (150.5, 97.2)
- added G***: LOGO, LOGO, B.Cu at (138.8, 97.7)
- added G***: LOGO, LOGO, B.Cu at (161.5, 98.7)
Other:
- board text added: "CURSO - PROJETO DE PCB PARA SISTEMAS EMBARCADOS"
- board text added: "PORTAL EMBARCADOS Projeto de PCB para Sistemas Embarcados Rev.01 2025/01/05 Eng. André A. M. Araújo"
- board text removed: "PORTAL EMBARCADOS Projeto de PCB para Sistemas Embarcados Rev.00 2024/11/16 Eng. André A. M. Araújo"
- board text removed: "PROJETO DE PCB PARA SISTEMAS EMBARCADOS"
