File: HARDWARE/KICAD/IO.kicad_sch (KiCad schematic)
At the start: 25 parts, among them J2 Conn_02x20_Odd_Even, J3 Conn_02x20_Odd_Even, J4 USB_C_Receptacle_USB2.0_16P, J5 Micro_SD_Card_Det1, U5 USBLC6-2SC6

Commit message: Recorded Class 08.07 Part 5.
Parts:
- J3: renamed from J4; value USB_C_Receptacle_USB2.0_16P -> USB
- J5: value Micro_SD_Card_Det1 -> Micro SD
- renumbered C26 to C14, C24 to C15, C27 to C35, C28 to C45, FB4 to FB2, J2 to J1, J3 to J6, R26 to R24, R25 to R31, R36 to R4, R28 to R40, R27 to R41, R31 to R46, R29 to R47, R30 to R48, R35 to R5, R34 to R6, R33 to R7, R32 to R8, U5 to U4
Changed lines of the file:
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@@
 		(on_board yes)
 		(dnp no)
-		(property "Reference" "C28"
+		(property "Reference" "C45"
 			(at 224.79 35.56 90)
 			(effects
@@
 			(project "EMBARCADOS - CURSO PCB"
 				(path "/d5268f1b-b782-4609-86ee-ff462c2ec1ad/5c5c1b35-8adb-4bed-8f60-c08a0db2168d"
-					(reference "C28")
+					(reference "C45")
 					(unit 1)
 				)
@@
 		(on_board yes)
 		(dnp no)
-		(property "Reference" "J3"
+		(property "Reference" "J6"
 			(at 80.01 96.52 0)
 			(effects
@@
 			(project "EMBARCADOS - CURSO PCB"
 				(path "/d5268f1b-b782-4609-86ee-ff462c2ec1ad/5c5c1b35-8adb-4bed-8f60-c08a0db2168d"
-					(reference "J3")
+					(reference "J6")
 					(unit 1)
 				)
@@
 		(on_board yes)
 		(dnp no)
-		(property "Reference" "R35"
+		(property "Reference" "R5"
 			(at 166.37 114.3 90)
 			(effects
@@
 			(project "EMBARCADOS - CURSO PCB"
 				(path "/d5268f1b-b782-4609-86ee-ff462c2ec1ad/5c5c1b35-8adb-4bed-8f60-c08a0db2168d"
-					(reference "R35")
+					(reference "R5")
 					(unit 1)
 				)
@@
 		(dnp no)
 		(fields_autoplaced yes)
-		(property "Reference" "J2"
+		(property "Reference" "J1"
 			(at 199.39 96.52 0)
 			(effects
@@
 			(project ""
 				(path "/d5268f1b-b782-4609-86ee-ff462c2ec1ad/5c5c1b35-8adb-4bed-8f60-c08a0db2168d"
-					(reference "J2")
+					(reference "J1")
 					(unit 1)
 				)
@@
 		(on_board yes)
 		(dnp no)
-		(property "Reference" "R27"
+		(property "Reference" "R41"
 			(at 210.82 44.45 90)
 			(effects
@@
 			(project "EMBARCADOS - CURSO PCB"
 				(path "/d5268f1b-b782-4609-86ee-ff462c2ec1ad/5c5c1b35-8adb-4bed-8f60-c08a0db2168d"
-					(reference "R27")
+					(reference "R41")
 					(unit 1)
 				)
@@
 		(on_board yes)
 		(dnp no)
-		(property "Reference" "R31"
+		(property "Reference" "R46"
 			(at 187.96 68.58 90)
 			(effects
@@
 			(project "EMBARCADOS - CURSO PCB"
 				(path "/d5268f1b-b782-4609-86ee-ff462c2ec1ad/5c5c1b35-8adb-4bed-8f60-c08a0db2168d"
-					(reference "R31")
+					(reference "R46")
 					(unit 1)
 				)
@@
 		(on_board yes)
 		(dnp no)
-		(property "Reference" "R28"
+		(property "Reference" "R40"
 			(at 208.28 44.45 90)
 			(effects
@@
 			(project "EMBARCADOS - CURSO PCB"
 				(path "/d5268f1b-b782-4609-86ee-ff462c2ec1ad/5c5c1b35-8adb-4bed-8f60-c08a0db2168d"
-					(reference "R28")
+					(reference "R40")
 					(unit 1)
 				)
@@
 		(on_board yes)
 		(dnp no)
-		(property "Reference" "J4"
+		(property "Reference" "J3"
 			(at 39.37 38.1 0)
 			(effects
@@
 			)
 		)
-		(property "Value" "USB_C_Receptacle_USB2.0_16P"
+		(property "Value" "USB"
 			(at 58.42 38.1 0)
 			(effects
@@
 			(project ""
 				(path "/d5268f1b-b782-4609-86ee-ff462c2ec1ad/5c5c1b35-8adb-4bed-8f60-c08a0db2168d"
-					(reference "J4")
+					(reference "J3")
 					(unit 1)
 				)
@@
 		(on_board yes)
 		(dnp no)
-		(property "Reference" "R33"
+		(property "Reference" "R7"
 			(at 166.37 109.22 90)
 			(effects
@@
 			(project "EMBARCADOS - CURSO PCB"
 				(path "/d5268f1b-b782-4609-86ee-ff462c2ec1ad/5c5c1b35-8adb-4bed-8f60-c08a0db2168d"
-					(reference "R33")
+					(reference "R7")
 					(unit 1)
 				)
@@
 			)
 		)
-		(property "Value" "Micro_SD_Card_Det1"
+		(property "Value" "Micro SD"
 			(at 243.84 45.72 0)
 			(effects
@@
 		(on_board yes)
 		(dnp no)
-		(property "Reference" "C24"
+		(property "Reference" "C15"
 			(at 107.95 35.56 90)
 			(effects
@@
 			(project ""
 				(path "/d5268f1b-b782-4609-86ee-ff462c2ec1ad/5c5c1b35-8adb-4bed-8f60-c08a0db2168d"
-					(reference "C24")
+					(reference "C15")
 					(unit 1)
 				)
@@
 		(on_board yes)
 		(dnp no)
-		(property "Reference" "C27"
+		(property "Reference" "C35"
 			(at 224.79 24.13 90)
 			(effects
@@
 			(project "EMBARCADOS - CURSO PCB"
 				(path "/d5268f1b-b782-4609-86ee-ff462c2ec1ad/5c5c1b35-8adb-4bed-8f60-c08a0db2168d"
-					(reference "C27")
+					(reference "C35")
 					(unit 1)
 				)
@@
 		(on_board yes)
 		(dnp no)
-		(property "Reference" "R36"
+		(property "Reference" "R4"
 			(at 166.37 119.38 90)
 			(effects
@@
 			(project "EMBARCADOS - CURSO PCB"
 				(path "/d5268f1b-b782-4609-86ee-ff462c2ec1ad/5c5c1b35-8adb-4bed-8f60-c08a0db2168d"
-					(reference "R36")
+					(reference "R4")
 					(unit 1)
 				)
@@
 		(on_board yes)
 		(dnp no)
-		(property "Reference" "R25"
+		(property "Reference" "R31"
 			(at 60.96 45.72 90)
 			(effects
@@
 			(project ""
 				(path "/d5268f1b-b782-4609-86ee-ff462c2ec1ad/5c5c1b35-8adb-4bed-8f60-c08a0db2168d"
-					(reference "R25")
+					(reference "R31")
 					(unit 1)
 				)
@@
 		(on_board yes)
 		(dnp no)
-		(property "Reference" "C26"
+		(property "Reference" "C14"
 			(at 83.82 24.13 90)
 			(effects
@@
 			(project ""
 				(path "/d5268f1b-b782-4609-86ee-ff462c2ec1ad/5c5c1b35-8adb-4bed-8f60-c08a0db2168d"
-					(reference "C26")
+					(reference "C14")
 					(unit 1)
 				)
@@
 		(on_board yes)
 		(dnp no)
-		(property "Reference" "R32"
+		(property "Reference" "R8"
 			(at 166.37 106.68 90)
 			(effects
@@
 			(project "EMBARCADOS - CURSO PCB"
 				(path "/d5268f1b-b782-4609-86ee-ff462c2ec1ad/5c5c1b35-8adb-4bed-8f60-c08a0db2168d"
-					(reference "R32")
+					(reference "R8")
 					(unit 1)
 				)
@@
 		(on_board yes)
 		(dnp no)
-		(property "Reference" "R26"
+		(property "Reference" "R24"
 			(at 60.96 48.26 90)
 			(effects
@@
 			(project "EMBARCADOS - CURSO PCB"
 				(path "/d5268f1b-b782-4609-86ee-ff462c2ec1ad/5c5c1b35-8adb-4bed-8f60-c08a0db2168d"
-					(reference "R26")
+					(reference "R24")
 					(unit 1)
 				)
@@
 		(on_board yes)
 		(dnp no)
-		(property "Reference" "R29"
+		(property "Reference" "R47"
 			(at 205.74 44.45 90)
 			(effects
@@
 			(project "EMBARCADOS - CURSO PCB"
 				(path "/d5268f1b-b782-4609-86ee-ff462c2ec1ad/5c5c1b35-8adb-4bed-8f60-c08a0db2168d"
-					(reference "R29")
+					(reference "R47")
 					(unit 1)
 				)
@@
 		(on_board yes)
 		(dnp no)
-		(property "Reference" "U5"
+		(property "Reference" "U4"
 			(at 93.98 53.34 0)
 			(effects
@@
 			(project ""
 				(path "/d5268f1b-b782-4609-86ee-ff462c2ec1ad/5c5c1b35-8adb-4bed-8f60-c08a0db2168d"
-					(reference "U5")
+					(reference "U4")
 					(unit 1)
 				)
@@
 		(on_board yes)
 		(dnp no)
-		(property "Reference" "R34"
+		(property "Reference" "R6"
 			(at 166.37 111.76 90)
 			(effects
@@
 			(project "EMBARCADOS - CURSO PCB"
 				(path "/d5268f1b-b782-4609-86ee-ff462c2ec1ad/5c5c1b35-8adb-4bed-8f60-c08a0db2168d"
-					(reference "R34")
+					(reference "R6")
 					(unit 1)
 				)
@@
 		(on_board yes)
 		(dnp no)
-		(property "Reference" "R30"
+		(property "Reference" "R48"
 			(at 203.2 44.45 90)
 			(effects
@@
 			(project "EMBARCADOS - CURSO PCB"
 				(path "/d5268f1b-b782-4609-86ee-ff462c2ec1ad/5c5c1b35-8adb-4bed-8f60-c08a0db2168d"
-					(reference "R30")
+					(reference "R48")
 					(unit 1)
 				)
@@
 		(on_board yes)
 		(dnp no)
-		(property "Reference" "FB4"
+		(property "Reference" "FB2"
 			(at 120.65 22.86 90)
 			(effects
@@
 			(project "EMBARCADOS - CURSO PCB"
 				(path "/d5268f1b-b782-4609-86ee-ff462c2ec1ad/5c5c1b35-8adb-4bed-8f60-c08a0db2168d"
-					(reference "FB4")
+					(reference "FB2")
 					(unit 1)
 				)
