File: HARDWARE/KICAD/IO.kicad_sch (KiCad schematic)
At the start: 25 parts, among them J1 Conn_02x20_Odd_Even, J3 USB, J5 Micro SD, J6 Conn_02x20_Odd_Even, U4 USBLC6-2SC6

Commit message: Refactoring after Class 08.07 Part 5.
Parts:
- renumbered U4 to D5, R8 to R10, R4 to R6, R5 to R7, R6 to R8, R7 to R9
Changed lines of the file:
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@@
 		(on_board yes)
 		(dnp no)
-		(property "Reference" "R5"
+		(property "Reference" "R7"
 			(at 166.37 114.3 90)
 			(effects
@@
 			(project "EMBARCADOS - CURSO PCB"
 				(path "/d5268f1b-b782-4609-86ee-ff462c2ec1ad/5c5c1b35-8adb-4bed-8f60-c08a0db2168d"
-					(reference "R5")
+					(reference "R7")
 					(unit 1)
 				)
@@
 		(on_board yes)
 		(dnp no)
-		(property "Reference" "R7"
+		(property "Reference" "R9"
 			(at 166.37 109.22 90)
 			(effects
@@
 			(project "EMBARCADOS - CURSO PCB"
 				(path "/d5268f1b-b782-4609-86ee-ff462c2ec1ad/5c5c1b35-8adb-4bed-8f60-c08a0db2168d"
-					(reference "R7")
+					(reference "R9")
 					(unit 1)
 				)
@@
 		(on_board yes)
 		(dnp no)
-		(property "Reference" "R4"
+		(property "Reference" "R6"
 			(at 166.37 119.38 90)
 			(effects
@@
 			(project "EMBARCADOS - CURSO PCB"
 				(path "/d5268f1b-b782-4609-86ee-ff462c2ec1ad/5c5c1b35-8adb-4bed-8f60-c08a0db2168d"
-					(reference "R4")
+					(reference "R6")
 					(unit 1)
 				)
@@
 		(on_board yes)
 		(dnp no)
-		(property "Reference" "R8"
+		(property "Reference" "R10"
 			(at 166.37 106.68 90)
 			(effects
@@
 			(project "EMBARCADOS - CURSO PCB"
 				(path "/d5268f1b-b782-4609-86ee-ff462c2ec1ad/5c5c1b35-8adb-4bed-8f60-c08a0db2168d"
-					(reference "R8")
+					(reference "R10")
 					(unit 1)
 				)
@@
 		(on_board yes)
 		(dnp no)
-		(property "Reference" "U4"
+		(property "Reference" "D5"
 			(at 93.98 53.34 0)
 			(effects
@@
 			(project ""
 				(path "/d5268f1b-b782-4609-86ee-ff462c2ec1ad/5c5c1b35-8adb-4bed-8f60-c08a0db2168d"
-					(reference "U4")
+					(reference "D5")
 					(unit 1)
 				)
@@
 		(on_board yes)
 		(dnp no)
-		(property "Reference" "R6"
+		(property "Reference" "R8"
 			(at 166.37 111.76 90)
 			(effects
@@
 			(project "EMBARCADOS - CURSO PCB"
 				(path "/d5268f1b-b782-4609-86ee-ff462c2ec1ad/5c5c1b35-8adb-4bed-8f60-c08a0db2168d"
-					(reference "R6")
+					(reference "R8")
 					(unit 1)
 				)

Commit message: Finished PCB Layout.
Parts:
- renumbered R6 to R10, R7 to R4, R8 to R5, R9 to R6, R10 to R7
Changed lines of the file:
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@@
 		(on_board yes)
 		(dnp no)
-		(property "Reference" "R7"
+		(property "Reference" "R4"
 			(at 166.37 114.3 90)
 			(effects
@@
 			(project "EMBARCADOS - CURSO PCB"
 				(path "/d5268f1b-b782-4609-86ee-ff462c2ec1ad/5c5c1b35-8adb-4bed-8f60-c08a0db2168d"
-					(reference "R7")
+					(reference "R4")
 					(unit 1)
 				)
@@
 		(on_board yes)
 		(dnp no)
-		(property "Reference" "R9"
+		(property "Reference" "R6"
 			(at 166.37 109.22 90)
 			(effects
@@
 			(project "EMBARCADOS - CURSO PCB"
 				(path "/d5268f1b-b782-4609-86ee-ff462c2ec1ad/5c5c1b35-8adb-4bed-8f60-c08a0db2168d"
-					(reference "R9")
+					(reference "R6")
 					(unit 1)
 				)
@@
 		(on_board yes)
 		(dnp no)
-		(property "Reference" "R6"
+		(property "Reference" "R10"
 			(at 166.37 119.38 90)
 			(effects
@@
 			(project "EMBARCADOS - CURSO PCB"
 				(path "/d5268f1b-b782-4609-86ee-ff462c2ec1ad/5c5c1b35-8adb-4bed-8f60-c08a0db2168d"
-					(reference "R6")
+					(reference "R10")
 					(unit 1)
 				)
@@
 		(on_board yes)
 		(dnp no)
-		(property "Reference" "R10"
+		(property "Reference" "R7"
 			(at 166.37 106.68 90)
 			(effects
@@
 			(project "EMBARCADOS - CURSO PCB"
 				(path "/d5268f1b-b782-4609-86ee-ff462c2ec1ad/5c5c1b35-8adb-4bed-8f60-c08a0db2168d"
-					(reference "R10")
+					(reference "R7")
 					(unit 1)
 				)
@@
 		(on_board yes)
 		(dnp no)
-		(property "Reference" "R8"
+		(property "Reference" "R5"
 			(at 166.37 111.76 90)
 			(effects
@@
 			(project "EMBARCADOS - CURSO PCB"
 				(path "/d5268f1b-b782-4609-86ee-ff462c2ec1ad/5c5c1b35-8adb-4bed-8f60-c08a0db2168d"
-					(reference "R8")
+					(reference "R5")
 					(unit 1)
 				)
