File: HARDWARE/KICAD/IO.kicad_sch (KiCad schematic)
At the start: 25 parts, among them J1 Conn_02x20_Odd_Even, J3 USB, J5 Micro SD, J6 Conn_02x20_Odd_Even

Commit message: Finished overall project review for PCB fabrication at JLCPCB.
Parts:
- C14, C35: LCSC Part # C15850 -> (none); LCSC Part #  (none) -> C15850
- C15: LCSC Part # C327005 -> (none); LCSC Part #  (none) -> C327005
- C25, C45: LCSC Part # C14663 -> (none); LCSC Part #  (none) -> C14663
- J1, J6: LCSC MANUFACTURER - -> (none); LCSC MANUFACTURER  (none) -> -; LCSC MPN - -> (none); LCSC MPN  (none) -> -
- J5: LCSC MANUFACTURER HANXIA -> (none); LCSC MANUFACTURER  (none) -> HANXIA
Changed lines of the file:
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@@
 			)
 		)
-		(property "LCSC Part #" "C14663 "
-			(at 240.284 38.1 0)
+		(property "LCSC MPN " "CC0603KRX7R9BB104 "
+			(at 235.966 37.592 0)
 			(effects
 				(font
@@
 			)
 		)
-		(property "LCSC MPN " "CC0603KRX7R9BB104 "
-			(at 235.966 37.592 0)
+		(property "LCSC MANUFACTURER " "YAGEO "
+			(at 238.252 37.846 0)
 			(effects
 				(font
@@
 			)
 		)
-		(property "LCSC MANUFACTURER " "YAGEO "
-			(at 238.252 37.846 0)
+		(property "LCSC Part # " "C14663 "
+			(at 240.284 38.1 0)
 			(effects
 				(font
@@
 			)
 		)
-		(property "LCSC MPN" "-"
+		(property "LCSC MPN " "-"
 			(at 71.882 165.862 0)
 			(effects
@@
 			)
 		)
-		(property "LCSC MANUFACTURER" "-"
+		(property "LCSC MANUFACTURER " "-"
 			(at 72.136 165.354 0)
 			(effects
@@
 			)
 		)
-		(property "LCSC MPN" "-"
+		(property "LCSC MPN " "-"
 			(at 207.518 165.862 0)
 			(effects
@@
 			)
 		)
-		(property "LCSC MANUFACTURER" "-"
+		(property "LCSC MANUFACTURER " "-"
 			(at 207.264 165.354 0)
 			(effects
@@
 			)
 		)
-		(property "LCSC MANUFACTURER" "HANXIA "
+		(property "LCSC MANUFACTURER " "HANXIA "
 			(at 245.11 89.916 0)
 			(effects
@@
 			)
 		)
-		(property "LCSC Part #" "C327005 "
-			(at 110.49 18.796 0)
+		(property "LCSC MPN " "CC0603KRX5R8BB684 "
+			(at 109.982 23.114 0)
 			(effects
 				(font
@@
 			)
 		)
-		(property "LCSC MPN " "CC0603KRX5R8BB684 "
-			(at 109.982 23.114 0)
+		(property "LCSC MANUFACTURER " "YAGEO "
+			(at 110.236 20.828 0)
 			(effects
 				(font
@@
 			)
 		)
-		(property "LCSC MANUFACTURER " "YAGEO "
-			(at 110.236 20.828 0)
+		(property "LCSC Part # " "C327005 "
+			(at 110.49 18.796 0)
 			(effects
 				(font
@@
 			)
 		)
-		(property "LCSC Part #" "C15850 "
-			(at 240.284 26.67 0)
+		(property "LCSC MPN " "CL21A106KAYNNNE "
+			(at 235.966 26.162 0)
 			(effects
 				(font
@@
 			)
 		)
-		(property "LCSC MPN " "CL21A106KAYNNNE "
-			(at 235.966 26.162 0)
+		(property "LCSC MANUFACTURER " "SAMSUNG "
+			(at 238.252 26.416 0)
 			(effects
 				(font
@@
 			)
 		)
-		(property "LCSC MANUFACTURER " "SAMSUNG "
-			(at 238.252 26.416 0)
+		(property "LCSC Part # " "C15850 "
+			(at 240.284 26.67 0)
 			(effects
 				(font
@@
 			)
 		)
-		(property "LCSC Part #" "C15850 "
-			(at 99.314 26.67 0)
+		(property "LCSC MPN " "CL21A106KAYNNNE "
+			(at 94.996 26.162 0)
 			(effects
 				(font
@@
 			)
 		)
-		(property "LCSC MPN " "CL21A106KAYNNNE "
-			(at 94.996 26.162 0)
+		(property "LCSC MANUFACTURER " "SAMSUNG "
+			(at 97.282 26.416 0)
 			(effects
 				(font
@@
 			)
 		)
-		(property "LCSC MANUFACTURER " "SAMSUNG "
-			(at 97.282 26.416 0)
+		(property "LCSC Part # " "C15850 "
+			(at 99.314 26.67 0)
 			(effects
 				(font
@@
 			)
 		)
-		(property "LCSC Part #" "C14663 "
-			(at 68.326 46.99 0)
+		(property "LCSC MPN " "CC0603KRX7R9BB104 "
+			(at 72.644 47.498 0)
 			(effects
 				(font
@@
 			)
 		)
-		(property "LCSC MPN " "CC0603KRX7R9BB104 "
-			(at 72.644 47.498 0)
+		(property "LCSC MANUFACTURER " "YAGEO "
+			(at 70.358 47.244 0)
 			(effects
 				(font
@@
 			)
 		)
-		(property "LCSC MANUFACTURER " "YAGEO "
-			(at 70.358 47.244 0)
+		(property "LCSC Part # " "C14663 "
+			(at 68.326 46.99 0)
 			(effects
 				(font
