File: HARDWARE/KICAD/ANALOG.kicad_sch (KiCad schematic)
At the start: 24 parts, among them J6 CONN 02x05 ODD EVEN, U6 LMV324, U7 ADS1115

Commit message: Refactoring.
Connections:
- net AA0: now reaches C29.1, R37.2, R38.1
- net AA0+: now reaches C30.2, R38.2, U6.3 (+)
- net AA2: now reaches C33.1, R41.2, R42.1
- net AA1+: now reaches C32.2, R40.2, U6.5 (+)
- net AA3: now reaches C35.1, R43.2, R44.1
- net AA3+: now reaches C36.2, R44.2, U6.12 (+)
- net AA2+: now reaches C34.2, R42.2, U6.10 (+)
- net AA1: now reaches C31.1, R39.2, R40.1
Other:
- moved on the sheet: C29, C30, C31, C32, C33, C34, C35, C36, C37, C38, C39, C40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

Commit message: Recorded Class 08.07 Part 5.
Parts:
- renumbered C31 to C19, C32 to C20, C38 to C21, C30 to C22, C29 to C23, C37 to C29, C39 to C30, C40 to C31, C33 to C36, C34 to C37, C36 to C38, C35 to C39, D4 to D5, J6 to J4, R39 to R27, R37 to R28, R40 to R29, R38 to R30, R42 to R38, R44 to R39, R41 to R43, R43 to R44, U6 to U5, U7 to U6
Changed lines of the file:
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@@
 		(on_board yes)
 		(dnp no)
-		(property "Reference" "C29"
+		(property "Reference" "C23"
 			(at 132.08 27.94 90)
 			(effects
@@
 			(project ""
 				(path "/d5268f1b-b782-4609-86ee-ff462c2ec1ad/9b5c5d79-aa85-43d6-bc66-deb2192346a3"
-					(reference "C29")
+					(reference "C23")
 					(unit 1)
 				)
@@
 		(on_board yes)
 		(dnp no)
-		(property "Reference" "U6"
+		(property "Reference" "U5"
 			(at 149.86 33.02 0)
 			(effects
@@
 			(project ""
 				(path "/d5268f1b-b782-4609-86ee-ff462c2ec1ad/9b5c5d79-aa85-43d6-bc66-deb2192346a3"
-					(reference "U6")
+					(reference "U5")
 					(unit 1)
 				)
@@
 		(on_board yes)
 		(dnp no)
-		(property "Reference" "R38"
+		(property "Reference" "R30"
 			(at 132.08 38.1 90)
 			(effects
@@
 			(project "EMBARCADOS - CURSO PCB"
 				(path "/d5268f1b-b782-4609-86ee-ff462c2ec1ad/9b5c5d79-aa85-43d6-bc66-deb2192346a3"
-					(reference "R38")
+					(reference "R30")
 					(unit 1)
 				)
@@
 		(on_board yes)
 		(dnp no)
-		(property "Reference" "R41"
+		(property "Reference" "R43"
 			(at 116.84 114.3 90)
 			(effects
@@
 			(project "EMBARCADOS - CURSO PCB"
 				(path "/d5268f1b-b782-4609-86ee-ff462c2ec1ad/9b5c5d79-aa85-43d6-bc66-deb2192346a3"
-					(reference "R41")
+					(reference "R43")
 					(unit 1)
 				)
@@
 		(on_board yes)
 		(dnp no)
-		(property "Reference" "C32"
+		(property "Reference" "C20"
 			(at 137.16 85.09 90)
 			(effects
@@
 			(project "EMBARCADOS - CURSO PCB"
 				(path "/d5268f1b-b782-4609-86ee-ff462c2ec1ad/9b5c5d79-aa85-43d6-bc66-deb2192346a3"
-					(reference "C32")
+					(reference "C20")
 					(unit 1)
 				)
@@
 		(on_board yes)
 		(dnp no)
-		(property "Reference" "C40"
+		(property "Reference" "C31"
 			(at 228.6 83.82 90)
 			(effects
@@
 			(project "EMBARCADOS - CURSO PCB"
 				(path "/d5268f1b-b782-4609-86ee-ff462c2ec1ad/9b5c5d79-aa85-43d6-bc66-deb2192346a3"
-					(reference "C40")
+					(reference "C31")
 					(unit 1)
 				)
@@
 		(on_board yes)
 		(dnp no)
-		(property "Reference" "R44"
+		(property "Reference" "R39"
 			(at 132.08 152.4 90)
 			(effects
@@
 			(project "EMBARCADOS - CURSO PCB"
 				(path "/d5268f1b-b782-4609-86ee-ff462c2ec1ad/9b5c5d79-aa85-43d6-bc66-deb2192346a3"
-					(reference "R44")
+					(reference "R39")
 					(unit 1)
 				)
@@
 		(on_board yes)
 		(dnp no)
-		(property "Reference" "C38"
+		(property "Reference" "C21"
 			(at 35.56 40.64 90)
 			(effects
@@
 			(project "EMBARCADOS - CURSO PCB"
 				(path "/d5268f1b-b782-4609-86ee-ff462c2ec1ad/9b5c5d79-aa85-43d6-bc66-deb2192346a3"
-					(reference "C38")
+					(reference "C21")
 					(unit 1)
 				)
@@
 		(on_board yes)
 		(dnp no)
-		(property "Reference" "R37"
+		(property "Reference" "R28"
 			(at 116.84 38.1 90)
 			(effects
@@
 			(project ""
 				(path "/d5268f1b-b782-4609-86ee-ff462c2ec1ad/9b5c5d79-aa85-43d6-bc66-deb2192346a3"
-					(reference "R37")
+					(reference "R28")
 					(unit 1)
 				)
@@
 		(on_board yes)
 		(dnp no)
-		(property "Reference" "C36"
+		(property "Reference" "C38"
 			(at 137.16 161.29 90)
 			(effects
@@
 			(project "EMBARCADOS - CURSO PCB"
 				(path "/d5268f1b-b782-4609-86ee-ff462c2ec1ad/9b5c5d79-aa85-43d6-bc66-deb2192346a3"
-					(reference "C36")
+					(reference "C38")
 					(unit 1)
 				)
@@
 		(on_board yes)
 		(dnp no)
-		(property "Reference" "C34"
+		(property "Reference" "C37"
 			(at 137.16 124.46 90)
 			(effects
@@
 			(project "EMBARCADOS - CURSO PCB"
 				(path "/d5268f1b-b782-4609-86ee-ff462c2ec1ad/9b5c5d79-aa85-43d6-bc66-deb2192346a3"
-					(reference "C34")
+					(reference "C37")
 					(unit 1)
 				)
@@
 		(on_board yes)
 		(dnp no)
-		(property "Reference" "U7"
+		(property "Reference" "U6"
 			(at 228.6 92.71 0)
 			(effects
@@
 			(project ""
 				(path "/d5268f1b-b782-4609-86ee-ff462c2ec1ad/9b5c5d79-aa85-43d6-bc66-deb2192346a3"
-					(reference "U7")
+					(reference "U6")
 					(unit 1)
 				)
@@
 		(on_board yes)
 		(dnp no)
-		(property "Reference" "U6"
+		(property "Reference" "U5"
 			(at 149.86 147.32 0)
 			(effects
@@
 			(project ""
 				(path "/d5268f1b-b782-4609-86ee-ff462c2ec1ad/9b5c5d79-aa85-43d6-bc66-deb2192346a3"
-					(reference "U6")
+					(reference "U5")
 					(unit 4)
 				)
@@
 		(on_board yes)
 		(dnp no)
-		(property "Reference" "C33"
+		(property "Reference" "C36"
 			(at 132.08 104.14 90)
 			(effects
@@
 			(project "EMBARCADOS - CURSO PCB"
 				(path "/d5268f1b-b782-4609-86ee-ff462c2ec1ad/9b5c5d79-aa85-43d6-bc66-deb2192346a3"
-					(reference "C33")
+					(reference "C36")
 					(unit 1)
 				)
@@
 		(on_board yes)
 		(dnp no)
-		(property "Reference" "R40"
+		(property "Reference" "R29"
 			(at 132.08 76.2 90)
 			(effects
@@
 			(project "EMBARCADOS - CURSO PCB"
 				(path "/d5268f1b-b782-4609-86ee-ff462c2ec1ad/9b5c5d79-aa85-43d6-bc66-deb2192346a3"
-					(reference "R40")
+					(reference "R29")
 					(unit 1)
 				)
@@
 		(dnp no)
 		(fields_autoplaced yes)
-		(property "Reference" "D4"
+		(property "Reference" "D5"
 			(at 63.5 113.0299 0)
 			(effects
@@
 			(project ""
 				(path "/d5268f1b-b782-4609-86ee-ff462c2ec1ad/9b5c5d79-aa85-43d6-bc66-deb2192346a3"
-					(reference "D4")
+					(reference "D5")
 					(unit 1)
 				)
@@
 		(on_board yes)
 		(dnp no)
-		(property "Reference" "C30"
+		(property "Reference" "C22"
 			(at 137.16 46.99 90)
 			(effects
@@
 			(project "EMBARCADOS - CURSO PCB"
 				(path "/d5268f1b-b782-4609-86ee-ff462c2ec1ad/9b5c5d79-aa85-43d6-bc66-deb2192346a3"
-					(reference "C30")
+					(reference "C22")
 					(unit 1)
 				)
@@
 		(on_board yes)
 		(dnp no)
-		(property "Reference" "R42"
+		(property "Reference" "R38"
 			(at 132.08 114.3 90)
 			(effects
@@
 			(project "EMBARCADOS - CURSO PCB"
 				(path "/d5268f1b-b782-4609-86ee-ff462c2ec1ad/9b5c5d79-aa85-43d6-bc66-deb2192346a3"
-					(reference "R42")
+					(reference "R38")
 					(unit 1)
 				)
@@
 		(dnp no)
 		(fields_autoplaced yes)
-		(property "Reference" "U6"
+		(property "Reference" "U5"
 			(at 48.26 39.3699 0)
 			(effects
@@
 			(project ""
 				(path "/d5268f1b-b782-4609-86ee-ff462c2ec1ad/9b5c5d79-aa85-43d6-bc66-deb2192346a3"
-					(reference "U6")
+					(reference "U5")
 					(unit 5)
 				)
@@
 		(on_board yes)
 		(dnp no)
-		(property "Reference" "U6"
+		(property "Reference" "U5"
 			(at 149.86 71.12 0)
 			(effects
@@
 			(project ""
 				(path "/d5268f1b-b782-4609-86ee-ff462c2ec1ad/9b5c5d79-aa85-43d6-bc66-deb2192346a3"
-					(reference "U6")
+					(reference "U5")
 					(unit 2)
 				)
@@
 		(on_board yes)
 		(dnp no)
-		(property "Reference" "J6"
+		(property "Reference" "J4"
 			(at 38.1 93.98 0)
 			(effects
@@
 			(project ""
 				(path "/d5268f1b-b782-4609-86ee-ff462c2ec1ad/9b5c5d79-aa85-43d6-bc66-deb2192346a3"
-					(reference "J6")
+					(reference "J4")
 					(unit 1)
 				)
@@
 		(on_board yes)
 		(dnp no)
-		(property "Reference" "C31"
+		(property "Reference" "C19"
 			(at 132.08 66.04 90)
 			(effects
@@
 			(project "EMBARCADOS - CURSO PCB"
 				(path "/d5268f1b-b782-4609-86ee-ff462c2ec1ad/9b5c5d79-aa85-43d6-bc66-deb2192346a3"
-					(reference "C31")
+					(reference "C19")
 					(unit 1)
 				)
@@
 		(on_board yes)
 		(dnp no)
-		(property "Reference" "R39"
+		(property "Reference" "R27"
 			(at 116.84 76.2 90)
 			(effects
@@
 			(project "EMBARCADOS - CURSO PCB"
 				(path "/d5268f1b-b782-4609-86ee-ff462c2ec1ad/9b5c5d79-aa85-43d6-bc66-deb2192346a3"
-					(reference "R39")
+					(reference "R27")
 					(unit 1)
 				)
@@
 		(on_board yes)
 		(dnp no)
-		(property "Reference" "C37"
+		(property "Reference" "C29"
 			(at 26.67 40.64 90)
 			(effects
@@
 			(project ""
 				(path "/d5268f1b-b782-4609-86ee-ff462c2ec1ad/9b5c5d79-aa85-43d6-bc66-deb2192346a3"
-					(reference "C37")
+					(reference "C29")
 					(unit 1)
 				)
@@
 		(on_board yes)
 		(dnp no)
-		(property "Reference" "C39"
+		(property "Reference" "C30"
 			(at 226.06 73.66 90)
 			(effects
@@
 			(project "EMBARCADOS - CURSO PCB"
 				(path "/d5268f1b-b782-4609-86ee-ff462c2ec1ad/9b5c5d79-aa85-43d6-bc66-deb2192346a3"
-					(reference "C39")
+					(reference "C30")
 					(unit 1)
 				)
@@
 		(on_board yes)
 		(dnp no)
-		(property "Reference" "R43"
+		(property "Reference" "R44"
 			(at 116.84 152.4 90)
 			(effects
@@
 			(project "EMBARCADOS - CURSO PCB"
 				(path "/d5268f1b-b782-4609-86ee-ff462c2ec1ad/9b5c5d79-aa85-43d6-bc66-deb2192346a3"
-					(reference "R43")
+					(reference "R44")
 					(unit 1)
 				)
@@
 		(on_board yes)
 		(dnp no)
-		(property "Reference" "C35"
+		(property "Reference" "C39"
 			(at 132.08 142.24 90)
 			(effects
@@
 			(project "EMBARCADOS - CURSO PCB"
 				(path "/d5268f1b-b782-4609-86ee-ff462c2ec1ad/9b5c5d79-aa85-43d6-bc66-deb2192346a3"
-					(reference "C35")
+					(reference "C39")
 					(unit 1)
 				)
@@
 		(on_board yes)
 		(dnp no)
-		(property "Reference" "U6"
+		(property "Reference" "U5"
 			(at 149.86 109.22 0)
 			(effects
@@
 			(project ""
 				(path "/d5268f1b-b782-4609-86ee-ff462c2ec1ad/9b5c5d79-aa85-43d6-bc66-deb2192346a3"
-					(reference "U6")
+					(reference "U5")
 					(unit 3)
 				)

Commit message: Refactoring.
Parts:
- J4: value CONN 02x05 ODD EVEN -> ANALOG
Changed lines of the file:
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@@
 			)
 		)
-		(property "Value" "CONN 02x05 ODD EVEN"
-			(at 38.1 92.71 0)
+		(property "Value" "ANALOG"
+			(at 38.1 109.22 0)
 			(effects
 				(font
 					(size 1.27 1.27)
 				)
-				(hide yes)
 			)
 		)

Commit message: Refactoring after Class 08.07 Part 5.
Parts:
- renumbered D5 to D6, U5 to U4, U6 to U5
Changed lines of the file:
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@@
 		(on_board yes)
 		(dnp no)
-		(property "Reference" "U5"
+		(property "Reference" "U4"
 			(at 149.86 33.02 0)
 			(effects
@@
 			(project ""
 				(path "/d5268f1b-b782-4609-86ee-ff462c2ec1ad/9b5c5d79-aa85-43d6-bc66-deb2192346a3"
-					(reference "U5")
+					(reference "U4")
 					(unit 1)
 				)
@@
 		(on_board yes)
 		(dnp no)
-		(property "Reference" "U6"
+		(property "Reference" "U5"
 			(at 228.6 92.71 0)
 			(effects
@@
 			(project ""
 				(path "/d5268f1b-b782-4609-86ee-ff462c2ec1ad/9b5c5d79-aa85-43d6-bc66-deb2192346a3"
-					(reference "U6")
+					(reference "U5")
 					(unit 1)
 				)
@@
 		(on_board yes)
 		(dnp no)
-		(property "Reference" "U5"
+		(property "Reference" "U4"
 			(at 149.86 147.32 0)
 			(effects
@@
 			(project ""
 				(path "/d5268f1b-b782-4609-86ee-ff462c2ec1ad/9b5c5d79-aa85-43d6-bc66-deb2192346a3"
-					(reference "U5")
+					(reference "U4")
 					(unit 4)
 				)
@@
 		(dnp no)
 		(fields_autoplaced yes)
-		(property "Reference" "D5"
+		(property "Reference" "D6"
 			(at 63.5 113.0299 0)
 			(effects
@@
 			(project ""
 				(path "/d5268f1b-b782-4609-86ee-ff462c2ec1ad/9b5c5d79-aa85-43d6-bc66-deb2192346a3"
-					(reference "D5")
+					(reference "D6")
 					(unit 1)
 				)
@@
 		(dnp no)
 		(fields_autoplaced yes)
-		(property "Reference" "U5"
+		(property "Reference" "U4"
 			(at 48.26 39.3699 0)
 			(effects
@@
 			(project ""
 				(path "/d5268f1b-b782-4609-86ee-ff462c2ec1ad/9b5c5d79-aa85-43d6-bc66-deb2192346a3"
-					(reference "U5")
+					(reference "U4")
 					(unit 5)
 				)
@@
 		(on_board yes)
 		(dnp no)
-		(property "Reference" "U5"
+		(property "Reference" "U4"
 			(at 149.86 71.12 0)
 			(effects
@@
 			(project ""
 				(path "/d5268f1b-b782-4609-86ee-ff462c2ec1ad/9b5c5d79-aa85-43d6-bc66-deb2192346a3"
-					(reference "U5")
+					(reference "U4")
 					(unit 2)
 				)
@@
 		(on_board yes)
 		(dnp no)
-		(property "Reference" "U5"
+		(property "Reference" "U4"
 			(at 149.86 109.22 0)
 			(effects
@@
 			(project ""
 				(path "/d5268f1b-b782-4609-86ee-ff462c2ec1ad/9b5c5d79-aa85-43d6-bc66-deb2192346a3"
-					(reference "U5")
+					(reference "U4")
 					(unit 3)
 				)
