File: HARDWARE/KICAD/ANALOG.kicad_sch (KiCad schematic)
At the start: 24 parts, among them J4 ANALOG, U4 LMV324, U5 ADS1115

Commit message: Finished overall project review for PCB fabrication at JLCPCB.
Parts:
- C19, C20, C21, C22, C23, C31, C36, C37, C38, C39: LCSC Part # C14663 -> (none); LCSC Part #  (none) -> C14663
- C29, C30: LCSC Part # C15850 -> (none); LCSC Part #  (none) -> C15850
Changed lines of the file:
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@@
 			)
 		)
-		(property "LCSC Part #" "C14663 "
-			(at 147.574 30.48 0)
+		(property "LCSC MPN " "CC0603KRX7R9BB104 "
+			(at 143.256 29.972 0)
 			(effects
 				(font
@@
 			)
 		)
-		(property "LCSC MPN " "CC0603KRX7R9BB104 "
-			(at 143.256 29.972 0)
+		(property "LCSC MANUFACTURER " "YAGEO "
+			(at 145.542 30.226 0)
 			(effects
 				(font
@@
 			)
 		)
-		(property "LCSC MANUFACTURER " "YAGEO "
-			(at 145.542 30.226 0)
+		(property "LCSC Part # " "C14663 "
+			(at 147.574 30.48 0)
 			(effects
 				(font
@@
 			)
 		)
-		(property "LCSC Part #" "C14663 "
-			(at 139.7 69.596 0)
+		(property "LCSC MPN " "CC0603KRX7R9BB104 "
+			(at 139.192 73.914 0)
 			(effects
 				(font
@@
 			)
 		)
-		(property "LCSC MPN " "CC0603KRX7R9BB104 "
-			(at 139.192 73.914 0)
+		(property "LCSC MANUFACTURER " "YAGEO "
+			(at 139.446 71.628 0)
 			(effects
 				(font
@@
 			)
 		)
-		(property "LCSC MANUFACTURER " "YAGEO "
-			(at 139.446 71.628 0)
+		(property "LCSC Part # " "C14663 "
+			(at 139.7 69.596 0)
 			(effects
 				(font
@@
 			)
 		)
-		(property "LCSC Part #" "C14663 "
-			(at 213.106 86.36 0)
+		(property "LCSC MPN " "CC0603KRX7R9BB104 "
+			(at 217.424 85.852 0)
 			(effects
 				(font
@@
 			)
 		)
-		(property "LCSC MPN " "CC0603KRX7R9BB104 "
-			(at 217.424 85.852 0)
+		(property "LCSC MANUFACTURER " "YAGEO "
+			(at 215.138 86.106 0)
 			(effects
 				(font
@@
 			)
 		)
-		(property "LCSC MANUFACTURER " "YAGEO "
-			(at 215.138 86.106 0)
+		(property "LCSC Part # " "C14663 "
+			(at 213.106 86.36 0)
 			(effects
 				(font
@@
 			)
 		)
-		(property "LCSC Part #" "C14663 "
-			(at 38.1 25.146 0)
+		(property "LCSC MPN " "CC0603KRX7R9BB104 "
+			(at 37.592 29.464 0)
 			(effects
 				(font
@@
 			)
 		)
-		(property "LCSC MPN " "CC0603KRX7R9BB104 "
-			(at 37.592 29.464 0)
+		(property "LCSC MANUFACTURER " "YAGEO "
+			(at 37.846 27.178 0)
 			(effects
 				(font
@@
 			)
 		)
-		(property "LCSC MANUFACTURER " "YAGEO "
-			(at 37.846 27.178 0)
+		(property "LCSC Part # " "C14663 "
+			(at 38.1 25.146 0)
 			(effects
 				(font
@@
 			)
 		)
-		(property "LCSC Part #" "C14663 "
-			(at 139.7 145.796 0)
+		(property "LCSC MPN " "CC0603KRX7R9BB104 "
+			(at 139.192 150.114 0)
 			(effects
 				(font
@@
 			)
 		)
-		(property "LCSC MPN " "CC0603KRX7R9BB104 "
-			(at 139.192 150.114 0)
+		(property "LCSC MANUFACTURER " "YAGEO "
+			(at 139.446 147.828 0)
 			(effects
 				(font
@@
 			)
 		)
-		(property "LCSC MANUFACTURER " "YAGEO "
-			(at 139.446 147.828 0)
+		(property "LCSC Part # " "C14663 "
+			(at 139.7 145.796 0)
 			(effects
 				(font
@@
 			)
 		)
-		(property "LCSC Part #" "C14663 "
-			(at 139.7 108.966 0)
+		(property "LCSC MPN " "CC0603KRX7R9BB104 "
+			(at 139.192 113.284 0)
 			(effects
 				(font
@@
 			)
 		)
-		(property "LCSC MPN " "CC0603KRX7R9BB104 "
-			(at 139.192 113.284 0)
+		(property "LCSC MANUFACTURER " "YAGEO "
+			(at 139.446 110.998 0)
 			(effects
 				(font
@@
 			)
 		)
-		(property "LCSC MANUFACTURER " "YAGEO "
-			(at 139.446 110.998 0)
+		(property "LCSC Part # " "C14663 "
+			(at 139.7 108.966 0)
 			(effects
 				(font
@@
 			)
 		)
-		(property "LCSC Part #" "C14663 "
-			(at 147.574 106.68 0)
+		(property "LCSC MPN " "CC0603KRX7R9BB104 "
+			(at 143.256 106.172 0)
 			(effects
 				(font
@@
 			)
 		)
-		(property "LCSC MPN " "CC0603KRX7R9BB104 "
-			(at 143.256 106.172 0)
+		(property "LCSC MANUFACTURER " "YAGEO "
+			(at 145.542 106.426 0)
 			(effects
 				(font
@@
 			)
 		)
-		(property "LCSC MANUFACTURER " "YAGEO "
-			(at 145.542 106.426 0)
+		(property "LCSC Part # " "C14663 "
+			(at 147.574 106.68 0)
 			(effects
 				(font
@@
 			)
 		)
-		(property "LCSC Part #" "C14663 "
-			(at 139.7 31.496 0)
+		(property "LCSC MPN " "CC0603KRX7R9BB104 "
+			(at 139.192 35.814 0)
 			(effects
 				(font
@@
 			)
 		)
-		(property "LCSC MPN " "CC0603KRX7R9BB104 "
-			(at 139.192 35.814 0)
+		(property "LCSC MANUFACTURER " "YAGEO "
+			(at 139.446 33.528 0)
 			(effects
 				(font
@@
 			)
 		)
-		(property "LCSC MANUFACTURER " "YAGEO "
-			(at 139.446 33.528 0)
+		(property "LCSC Part # " "C14663 "
+			(at 139.7 31.496 0)
 			(effects
 				(font
@@
 			)
 		)
-		(property "LCSC Part #" "C14663 "
-			(at 147.574 68.58 0)
+		(property "LCSC MPN " "CC0603KRX7R9BB104 "
+			(at 143.256 68.072 0)
 			(effects
 				(font
@@
 			)
 		)
-		(property "LCSC MPN " "CC0603KRX7R9BB104 "
-			(at 143.256 68.072 0)
+		(property "LCSC MANUFACTURER " "YAGEO "
+			(at 145.542 68.326 0)
 			(effects
 				(font
@@
 			)
 		)
-		(property "LCSC MANUFACTURER " "YAGEO "
-			(at 145.542 68.326 0)
+		(property "LCSC Part # " "C14663 "
+			(at 147.574 68.58 0)
 			(effects
 				(font
@@
 			)
 		)
-		(property "LCSC Part #" "C15850 "
-			(at 29.21 56.134 0)
+		(property "LCSC MPN " "CL21A106KAYNNNE "
+			(at 28.702 51.816 0)
 			(effects
 				(font
@@
 			)
 		)
-		(property "LCSC MPN " "CL21A106KAYNNNE "
-			(at 28.702 51.816 0)
+		(property "LCSC MANUFACTURER " "SAMSUNG "
+			(at 28.956 54.102 0)
 			(effects
 				(font
@@
 			)
 		)
-		(property "LCSC MANUFACTURER " "SAMSUNG "
-			(at 28.956 54.102 0)
+		(property "LCSC Part # " "C15850 "
+			(at 29.21 56.134 0)
 			(effects
 				(font
@@
 			)
 		)
-		(property "LCSC Part #" "C15850 "
-			(at 213.106 76.2 0)
+		(property "LCSC MPN " "CL21A106KAYNNNE "
+			(at 217.424 75.692 0)
 			(effects
 				(font
@@
 			)
 		)
-		(property "LCSC MPN " "CL21A106KAYNNNE "
-			(at 217.424 75.692 0)
+		(property "LCSC MANUFACTURER " "SAMSUNG "
+			(at 215.138 75.946 0)
 			(effects
 				(font
@@
 			)
 		)
-		(property "LCSC MANUFACTURER " "SAMSUNG "
-			(at 215.138 75.946 0)
+		(property "LCSC Part # " "C15850 "
+			(at 213.106 76.2 0)
 			(effects
 				(font
@@
 			)
 		)
-		(property "LCSC Part #" "C14663 "
-			(at 147.574 144.78 0)
+		(property "LCSC MPN " "CC0603KRX7R9BB104 "
+			(at 143.256 144.272 0)
 			(effects
 				(font
@@
 			)
 		)
-		(property "LCSC MPN " "CC0603KRX7R9BB104 "
-			(at 143.256 144.272 0)
+		(property "LCSC MANUFACTURER " "YAGEO "
+			(at 145.542 144.526 0)
 			(effects
 				(font
@@
 			)
 		)
-		(property "LCSC MANUFACTURER " "YAGEO "
-			(at 145.542 144.526 0)
+		(property "LCSC Part # " "C14663 "
+			(at 147.574 144.78 0)
 			(effects
 				(font
