File: HARDWARE/KICAD/POWER.kicad_sch (KiCad schematic)
At the start: 32 parts, among them J1 DC BARREL JACK, U1 LD1117S33TR, U2 AP3012, U3 LD1117S50TR

Commit message: Recorded IO sheet class.
Changed lines of the file:
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@@
 	)
 	(junction
+		(at 50.8 66.04)
+		(diameter 0)
+		(color 0 0 0 0)
+	)
+	(junction
 		(at 88.9 40.64)
 		(diameter 0)
@@
 	(wire
 		(pts
+			(xy 50.8 66.04) (xy 62.23 66.04)
+		)
+		(stroke
+			(width 0)
+			(type default)
+		)
+	)
+	(wire
+		(pts
 			(xy 97.79 29.21) (xy 97.79 25.4)
 		)
@@
 	(wire
 		(pts
+			(xy 62.23 63.5) (xy 62.23 66.04)
+		)
+		(stroke
+			(width 0)
+			(type default)
+		)
+	)
+	(wire
+		(pts
 			(xy 165.1 67.31) (xy 162.56 67.31)
 		)
@@
 					(unit 1)
 				)
+			)
+		)
+	)
+	(symbol
+		(lib_id "power:PWR_FLAG")
+		(at 62.23 63.5 0)
+		(unit 1)
+		(exclude_from_sim no)
+		(in_bom yes)
+		(on_board yes)
+		(dnp no)
+		(fields_autoplaced yes)
+		(property "Reference" "#FLG01"
+			(at 62.23 61.595 0)
+			(effects
+				(font
+					(size 1.27 1.27)
+				)
+				(hide yes)
+			)
+		)
+		(property "Value" "PWR_FLAG"
+			(at 62.23 58.42 0)
+			(effects
+				(font
+					(size 1.27 1.27)
+				)
+			)
+		)
+		(property "Footprint" ""
+			(at 62.23 63.5 0)
+			(effects
+				(font
+					(size 1.27 1.27)
+				)
+				(hide yes)
+			)
+		)
+		(property "Datasheet" "~"
+			(at 62.23 63.5 0)
+			(effects
+				(font
+					(size 1.27 1.27)
+				)
+				(hide yes)
+			)
+		)
+		(property "Description" "Special symbol for telling ERC where power comes from"
+			(at 62.23 63.5 0)
+			(effects
+				(font
+					(size 1.27 1.27)
+				)
+				(hide yes)
+			)
+		)
+		(pin "1"
+		)
+		(instances
+			(project ""
+				(path "/d5268f1b-b782-4609-86ee-ff462c2ec1ad/25e9c17a-dec3-4329-9bcf-5cd51d1774f7"
+					(reference "#FLG01")
+					(unit 1)
+				)

Commit message: Refactoring.
Other:
- company: (none) -> Mechatronix Lab
- title: (none) -> EMBARCADOS - CURSO PCB
Changed lines of the file:
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@@
 	(generator_version "8.0")
 	(paper "A4")
+	(title_block
+		(title "EMBARCADOS - CURSO PCB")
+		(date "2024-11-11")
+		(rev "00")
+		(company "Mechatronix Lab")
+		(comment 1 "Eng. André A. M. Araújo")
+	)
 	(junction
 		(at 228.6 116.84)
@@
 		(lib_id "EMBARCADOS - CURSO PCB:CAP 0805 10uH 16V AVX KGM21AR71C106K")
 		(at 228.6 121.92 0)
+		(mirror y)
 		(unit 1)
 		(exclude_from_sim no)
@@
 		(dnp no)
 		(property "Reference" "C5"
-			(at 231.14 120.6562 0)
+			(at 226.06 123.19 90)
 			(effects
 				(font
@@
 		)
 		(property "Value" "10µF 16V"
-			(at 231.14 123.1962 0)
+			(at 231.14 127 90)
 			(effects
 				(font
@@
 		)
 		(property "Manufacturer" "KYOCERA/AVX "
-			(at 228.854 139.192 0)
+			(at 228.346 139.192 0)
 			(effects
 				(font
@@
 		)
 		(property "3D Model" "KiCad"
-			(at 228.346 143.51 0)
+			(at 228.854 143.51 0)
 			(effects
 				(font
@@
 		)
 		(property "LCSC MPN " "CL21A106KAYNNNE "
-			(at 229.108 133.096 0)
+			(at 228.092 133.096 0)
 			(effects
 				(font
@@
 		)
 		(property "LCSC MANUFACTURER " "SAMSUNG "
-			(at 228.854 135.382 0)
+			(at 228.346 135.382 0)
 			(effects
 				(font
@@
 		(dnp no)
 		(property "Reference" "FB1"
-			(at 241.3 114.3 90)
+			(at 241.3 113.03 90)
 			(effects
 				(font
@@
 		)
 		(property "Value" "600R 800mA"
-			(at 241.3 119.38 90)
+			(at 241.3 120.65 90)
 			(effects
 				(font

Commit message: Added ANALOG and INTERFACE sheets.
Parts:
- C1, C2, C3, C4, C5, C6, C7: symbol EMBARCADOS - CURSO PCB:CAP 0805 10uH 16V AVX KGM21AR71C106K -> EMBARCADOS - CURSO PCB:CAP 0805 10uF 16V AVX KGM21AR71C106K
Changed lines of the file:
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@@
 	)
 	(symbol
-		(lib_id "EMBARCADOS - CURSO PCB:CAP 0805 10uH 16V AVX KGM21AR71C106K")
+		(lib_id "EMBARCADOS - CURSO PCB:CAP 0805 10uF 16V AVX KGM21AR71C106K")
 		(at 114.3 121.92 0)
 		(mirror y)
@@
 			)
 		)
-		(property "Description" "CAP 0805 10uH 16V AVX"
+		(property "Description" "CAP 0805 10uF 16V AVX"
 			(at 114.3 131.318 0)
 			(effects
@@
 	)
 	(symbol
-		(lib_id "EMBARCADOS - CURSO PCB:CAP 0805 10uH 16V AVX KGM21AR71C106K")
+		(lib_id "EMBARCADOS - CURSO PCB:CAP 0805 10uF 16V AVX KGM21AR71C106K")
 		(at 254 121.92 0)
 		(unit 1)
@@
 			)
 		)
-		(property "Description" "CAP 0805 10uH 16V AVX"
+		(property "Description" "CAP 0805 10uF 16V AVX"
 			(at 254 131.318 0)
 			(effects
@@
 	)
 	(symbol
-		(lib_id "EMBARCADOS - CURSO PCB:CAP 0805 10uH 16V AVX KGM21AR71C106K")
+		(lib_id "EMBARCADOS - CURSO PCB:CAP 0805 10uF 16V AVX KGM21AR71C106K")
 		(at 228.6 121.92 0)
 		(mirror y)
@@
 			)
 		)
-		(property "Description" "CAP 0805 10uH 16V AVX"
+		(property "Description" "CAP 0805 10uF 16V AVX"
 			(at 228.6 131.318 0)
 			(effects
@@
 	)
 	(symbol
-		(lib_id "EMBARCADOS - CURSO PCB:CAP 0805 10uH 16V AVX KGM21AR71C106K")
+		(lib_id "EMBARCADOS - CURSO PCB:CAP 0805 10uF 16V AVX KGM21AR71C106K")
 		(at 127 69.85 0)
 		(mirror y)
@@
 			)
 		)
-		(property "Description" "CAP 0805 10uH 16V AVX"
+		(property "Description" "CAP 0805 10uF 16V AVX"
 			(at 127 79.248 0)
 			(effects
@@
 	)
 	(symbol
-		(lib_id "EMBARCADOS - CURSO PCB:CAP 0805 10uH 16V AVX KGM21AR71C106K")
+		(lib_id "EMBARCADOS - CURSO PCB:CAP 0805 10uF 16V AVX KGM21AR71C106K")
 		(at 203.2 121.92 0)
 		(mirror y)
@@
 			)
 		)
-		(property "Description" "CAP 0805 10uH 16V AVX"
+		(property "Description" "CAP 0805 10uF 16V AVX"
 			(at 203.2 131.318 0)
 			(effects
@@
 	)
 	(symbol
-		(lib_id "EMBARCADOS - CURSO PCB:CAP 0805 10uH 16V AVX KGM21AR71C106K")
+		(lib_id "EMBARCADOS - CURSO PCB:CAP 0805 10uF 16V AVX KGM21AR71C106K")
 		(at 139.7 121.92 0)
 		(unit 1)
@@
 			)
 		)
-		(property "Description" "CAP 0805 10uH 16V AVX"
+		(property "Description" "CAP 0805 10uF 16V AVX"
 			(at 139.7 131.318 0)
 			(effects
@@
 	)
 	(symbol
-		(lib_id "EMBARCADOS - CURSO PCB:CAP 0805 10uH 16V AVX KGM21AR71C106K")
+		(lib_id "EMBARCADOS - CURSO PCB:CAP 0805 10uF 16V AVX KGM21AR71C106K")
 		(at 190.5 69.85 0)
 		(unit 1)
@@
 			)
 		)
-		(property "Description" "CAP 0805 10uH 16V AVX"
+		(property "Description" "CAP 0805 10uF 16V AVX"
 			(at 190.5 79.248 0)
 			(effects

Commit message: Refactoring.
Other:
- note added: "INCLUIR MPN E MANUF. INCLUIR RANGE DE ENTRADA"
- moved on the sheet: D1, D2
Changed lines of the file:
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@@
 	)
 	(junction
-		(at 88.9 40.64)
+		(at 190.5 57.15)
 		(diameter 0)
 		(color 0 0 0 0)
 	)
 	(junction
-		(at 190.5 57.15)
+		(at 88.9 50.8)
 		(diameter 0)
 		(color 0 0 0 0)
@@
 	(wire
 		(pts
-			(xy 97.79 29.21) (xy 97.79 25.4)
-		)
-		(stroke
-			(width 0)
-			(type default)
-		)
-	)
-	(wire
-		(pts
 			(xy 127 185.42) (xy 127 187.96)
 		)
@@
 	(wire
 		(pts
-			(xy 88.9 57.15) (xy 88.9 40.64)
+			(xy 88.9 57.15) (xy 88.9 50.8)
 		)
 		(stroke
@@
 	(wire
 		(pts
-			(xy 101.6 40.64) (xy 101.6 38.1)
+			(xy 101.6 50.8) (xy 101.6 48.26)
 		)
 		(stroke
@@
 	(wire
 		(pts
-			(xy 78.74 21.59) (xy 78.74 31.75)
-		)
-		(stroke
-			(width 0)
-			(type default)
-		)
-	)
-	(wire
-		(pts
 			(xy 76.2 185.42) (xy 76.2 187.96)
 		)
@@
 	(wire
 		(pts
-			(xy 101.6 29.21) (xy 101.6 30.48)
-		)
-		(stroke
-			(width 0)
-			(type default)
-		)
-	)
-	(wire
-		(pts
 			(xy 114.3 57.15) (xy 116.84 57.15)
 		)
@@
 	(wire
 		(pts
-			(xy 78.74 40.64) (xy 88.9 40.64)
+			(xy 76.2 50.8) (xy 88.9 50.8)
 		)
 		(stroke
@@
 	(wire
 		(pts
-			(xy 78.74 39.37) (xy 78.74 40.64)
+			(xy 76.2 48.26) (xy 76.2 50.8)
 		)
 		(stroke
@@
 	(wire
 		(pts
-			(xy 88.9 40.64) (xy 101.6 40.64)
+			(xy 88.9 50.8) (xy 101.6 50.8)
 		)
 		(stroke
@@
 	(wire
 		(pts
-			(xy 101.6 29.21) (xy 97.79 29.21)
+			(xy 127 172.72) (xy 127 177.8)
 		)
 		(stroke
@@
 	(wire
 		(pts
-			(xy 127 172.72) (xy 127 177.8)
+			(xy 165.1 57.15) (xy 165.1 64.77)
 		)
 		(stroke
@@
 	(wire
 		(pts
-			(xy 165.1 57.15) (xy 165.1 64.77)
+			(xy 156.21 57.15) (xy 165.1 57.15)
 		)
 		(stroke
@@
 	(wire
 		(pts
-			(xy 156.21 57.15) (xy 165.1 57.15)
+			(xy 127 127) (xy 139.7 127)
 		)
 		(stroke
@@
 	(wire
 		(pts
-			(xy 127 127) (xy 139.7 127)
+			(xy 76.2 40.64) (xy 76.2 38.1)
 		)
 		(stroke
@@
 		)
 	)
+	(text "INCLUIR MPN E MANUF.\nINCLUIR RANGE DE ENTRADA\n"
+		(exclude_from_sim no)
+		(at 41.91 83.82 0)
+		(effects
+			(font
+				(size 1.27 1.27)
+				(thickness 0.254)
+				(bold yes)
+				(color 255 0 0 1)
+			)
+		)
+	)
 	(label "BOOST IN"
 		(at 140.97 57.15 0)
@@
 	(symbol
 		(lib_id "EMBARCADOS - CURSO PCB:DIODE SCHOTTKY 1N5819WS SOD-123 DIODES INC")
-		(at 78.74 35.56 90)
+		(at 76.2 44.45 90)
 		(unit 1)
 		(exclude_from_sim no)
@@
 		(dnp no)
 		(property "Reference" "D1"
-			(at 81.28 35.56 0)
+			(at 78.74 44.45 0)
 			(effects
 				(font
@@
 		)
 		(property "Value" "1N5819HW"
-			(at 76.2 35.56 0)
+			(at 73.66 44.45 0)
 			(effects
 				(font
@@
 		)
 		(property "Footprint" "EMBARCADOS - CURSO PCB:D_SOD-123"
-			(at 83.185 35.56 0)
+			(at 80.645 44.45 0)
 			(effects
 				(font
@@
 		)
 		(property "Datasheet" "https://www.diodes.com/datasheet/download/1N5819HW.pdf"
-			(at 85.598 35.306 0)
+			(at 83.058 44.196 0)
 			(effects
 				(font
@@
 		)
 		(property "Description" "40V 600mV@1A 1A SOD-323 Schottky Barrier Diodes, SOD-323"
-			(at 85.598 35.306 0)
+			(at 83.058 44.196 0)
 			(effects
 				(font
@@
 		)
 		(property "MPN" "1N5819HW-7-F "
-			(at 83.82 35.56 0)
+			(at 81.28 44.45 0)
 			(effects
 				(font
@@
 		)
 		(property "Manufactrer" "DIODES INCORPORATED "
-			(at 85.598 35.306 0)
+			(at 83.058 44.196 0)
 			(effects
 				(font
@@
 		)
 		(property "3D Model" "KiCad"
-			(at 83.82 35.56 0)
+			(at 81.28 44.45 0)
 			(effects
 				(font
@@
 		)
 		(property "Notes" "-"
-			(at 87.122 35.56 0)
+			(at 84.582 44.45 0)
 			(effects
 				(font
@@
 		)
 		(property "LCSC Part # " "C82544 "
-			(at 83.82 35.56 0)
+			(at 81.28 44.45 0)
 			(effects
 				(font
@@
 		)
 		(property "LCSC MPN " "1N5819HW-7-F "
-			(at 83.82 35.56 0)
+			(at 81.28 44.45 0)
 			(effects
 				(font
@@
 		)
 		(property "LCSC MANUFACTURER " "DIODES INCORPORATED "
-			(at 85.598 35.306 0)
+			(at 83.058 44.196 0)
 			(effects
 				(font
@@
 	(symbol
 		(lib_id "EMBARCADOS - CURSO PCB:+5V")
-		(at 78.74 21.59 0)
+		(at 76.2 38.1 0)
 		(unit 1)
 		(exclude_from_sim no)
@@
 		(dnp no)
 		(property "Reference" "#PWR07"
-			(at 78.74 25.4 0)
+			(at 76.2 41.91 0)
 			(effects
 				(font
@@
 		)
 		(property "Value" "+VEXT"
-			(at 78.74 17.78 0)
+			(at 76.2 34.29 0)
 			(effects
 				(font
@@
 		)
 		(property "Footprint" ""
-			(at 78.74 21.59 0)
+			(at 76.2 38.1 0)
 			(effects
 				(font
@@
 		)
 		(property "Datasheet" ""
-			(at 78.74 21.59 0)
+			(at 76.2 38.1 0)
 			(effects
 				(font
@@
 		)
 		(property "Description" "Power symbol creates a global label with name \"+5V\""
-			(at 78.74 21.59 0)
+			(at 76.2 38.1 0)
 			(effects
 				(font
@@
 		)
 		(property "MPN" ""
-			(at 78.74 21.59 0)
+			(at 76.2 38.1 0)
 			(effects
 				(font
@@
 		)
 		(property "Manufacturer" ""
-			(at 78.74 21.59 0)
+			(at 76.2 38.1 0)
 			(effects
 				(font
@@
 		)
 		(property "3D Model" ""
-			(at 78.74 21.59 0)
+			(at 76.2 38.1 0)
 			(effects
 				(font
@@
 		)
 		(property "Notes" ""
-			(at 78.74 21.59 0)
+			(at 76.2 38.1 0)
 			(effects
 				(font
@@
 		)
 		(property "LCSC Part # " ""
-			(at 78.74 21.59 0)
+			(at 76.2 38.1 0)
 			(effects
 				(font
@@
 		)
 		(property "LCSC MPN " ""
-			(at 78.74 21.59 0)
+			(at 76.2 38.1 0)
 			(effects
 				(font
@@
 		)
 		(property "LCSC MANUFACTURER " ""
-			(at 78.74 21.59 0)
+			(at 76.2 38.1 0)
 			(effects
 				(font
@@
 	(symbol
 		(lib_id "EMBARCADOS - CURSO PCB:DIODE SCHOTTKY 1N5819WS SOD-123 DIODES INC")
-		(at 101.6 34.29 90)
+		(at 101.6 44.45 90)
 		(unit 1)
 		(exclude_from_sim no)
@@
 		(dnp no)
 		(property "Reference" "D2"
-			(at 99.06 34.29 0)
+			(at 99.06 44.45 0)
 			(effects
 				(font
@@
 		)
 		(property "Value" "1N5819HW"
-			(at 104.14 34.29 0)
+			(at 104.14 44.45 0)
 			(effects
 				(font
@@
 		)
 		(property "Footprint" "EMBARCADOS - CURSO PCB:D_SOD-123"
-			(at 106.045 34.29 0)
+			(at 106.045 44.45 0)
 			(effects
 				(font
@@
 		)
 		(property "Datasheet" "https://www.diodes.com/datasheet/download/1N5819HW.pdf"
-			(at 108.458 34.036 0)
+			(at 108.458 44.196 0)
 			(effects
 				(font
@@
 		)
 		(property "Description" "40V 600mV@1A 1A SOD-323 Schottky Barrier Diodes, SOD-323"
-			(at 108.458 34.036 0)
+			(at 108.458 44.196 0)
 			(effects
 				(font
@@
 		)
 		(property "MPN" "1N5819HW-7-F "
-			(at 106.68 34.29 0)
+			(at 106.68 44.45 0)
 			(effects
 				(font
@@
 		)
 		(property "Manufactrer" "DIODES INCORPORATED "
-			(at 108.458 34.036 0)
+			(at 108.458 44.196 0)
 			(effects
 				(font
@@
 		)
 		(property "3D Model" "KiCad"
-			(at 106.68 34.29 0)
+			(at 106.68 44.45 0)
 			(effects
 				(font
@@
 		)
 		(property "Notes" "-"
-			(at 109.982 34.29 0)
+			(at 109.982 44.45 0)
 			(effects
 				(font
@@
 		)
 		(property "LCSC Part # " "C82544 "
-			(at 106.68 34.29 0)
+			(at 106.68 44.45 0)
 			(effects
 				(font
@@
 		)
 		(property "LCSC MPN " "1N5819HW-7-F "
-			(at 106.68 34.29 0)
+			(at 106.68 44.45 0)
 			(effects
 				(font
@@
 		)
 		(property "LCSC MANUFACTURER " "DIODES INCORPORATED "
-			(at 108.458 34.036 0)
+			(at 108.458 44.196 0)
 			(effects
 				(font

Commit message: Finished schematic.
Parts:
- J1: value DC BARREL JACK -> 3V-7V
Connections:
- net +VBUSF: now reaches LED2.2 (A)
- net +VBUSF: now also D2.2 (A)
Other:
- note removed: "INCLUIR MPN E MANUF. INCLUIR RANGE DE ENTRADA"
- note removed: "INCLUIR TEST POINTS"
- moved on the sheet: D3

Commit message: Refactoring of schematic. PDF plotting.
Other:
- note added: "BOOST OUT = 1.25 * (1 + R7/R8) +VBOOST = 7.125V"
- note removed: "BOOST OUT = 1.25 * (1 + R1/R2)"
Changed lines of the file:
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@@
 	(wire
 		(pts
-			(xy 50.8 125.73) (xy 50.8 128.27)
+			(xy 50.8 125.73) (xy 50.8 129.54)
 		)
 		(stroke
@@
 		)
 	)
-	(text "BOOST OUT = 1.25 * (1 + R1/R2)"
+	(text "BOOST OUT = 1.25 * (1 + R7/R8)\n+VBOOST = 7.125V"
 		(exclude_from_sim no)
 		(at 176.53 88.9 0)
@@
 	(symbol
 		(lib_id "EMBARCADOS - CURSO PCB:POWER GND")
-		(at 50.8 128.27 0)
+		(at 50.8 129.54 0)
 		(unit 1)
 		(exclude_from_sim no)
@@
 		(fields_autoplaced yes)
 		(property "Reference" "#PWR04"
-			(at 50.8 134.62 0)
+			(at 50.8 135.89 0)
 			(effects
 				(font
@@
 		)
 		(property "Value" "GND"
-			(at 50.8 133.35 0)
+			(at 50.8 134.62 0)
 			(effects
 				(font
@@
 		)
 		(property "Footprint" ""
-			(at 50.8 128.27 0)
+			(at 50.8 129.54 0)
 			(effects
 				(font
@@
 		)
 		(property "Datasheet" ""
-			(at 50.8 128.27 0)
+			(at 50.8 129.54 0)
 			(effects
 				(font
@@
 		)
 		(property "Description" "Power symbol creates a global label with name \"GND\" , ground"
-			(at 50.8 128.27 0)
+			(at 50.8 129.54 0)
 			(effects
 				(font
@@
 					(size 1.27 1.27)
 				)
+				(hide yes)
 			)
 		)
