File: HARDWARE/KICAD/POWER.kicad_sch (KiCad schematic)
At the start: 32 parts, among them J1 3V-7V, U1 LD1117S33TR, U2 AP3012, U3 LD1117S50TR

Commit message: Recorded Class 08.07 Part 5.
Parts:
- renumbered C6 to C1, C1 to C10, C7 to C12, C2 to C4, C4 to C6, C3 to C9, D3 to D1, D2 to D3, D1 to D4, J1 to J2, JP2 to JP1, JP1 to JP2, LED3 to LED1, LED4 to LED2, LED5 to LED3, LED2 to LED4, LED1 to LED5, R3 to R1, R5 to R10, R6 to R13, R8 to R2, R2 to R20, R1 to R21, R7 to R3, R4 to R9, U2 to U1, U3 to U2, U1 to U3
Changed lines of the file:
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@@
 		(on_board yes)
 		(dnp no)
-		(property "Reference" "R5"
+		(property "Reference" "R10"
 			(at 149.86 181.61 90)
 			(effects
@@
 			(project "EMBARCADOS - CURSO PCB"
 				(path "/d5268f1b-b782-4609-86ee-ff462c2ec1ad/25e9c17a-dec3-4329-9bcf-5cd51d1774f7"
-					(reference "R5")
+					(reference "R10")
 					(unit 1)
 				)
@@
 		(dnp no)
 		(fields_autoplaced yes)
-		(property "Reference" "LED2"
+		(property "Reference" "LED4"
 			(at 80.01 169.2274 90)
 			(effects
@@
 			(project "EMBARCADOS - CURSO PCB"
 				(path "/d5268f1b-b782-4609-86ee-ff462c2ec1ad/25e9c17a-dec3-4329-9bcf-5cd51d1774f7"
-					(reference "LED2")
+					(reference "LED4")
 					(unit 1)
 				)
@@
 		(on_board yes)
 		(dnp no)
-		(property "Reference" "C1"
+		(property "Reference" "C10"
 			(at 111.76 120.6562 0)
 			(effects
@@
 			(project "EMBARCADOS - CURSO PCB"
 				(path "/d5268f1b-b782-4609-86ee-ff462c2ec1ad/25e9c17a-dec3-4329-9bcf-5cd51d1774f7"
-					(reference "C1")
+					(reference "C10")
 					(unit 1)
 				)
@@
 		(on_board yes)
 		(dnp no)
-		(property "Reference" "D1"
+		(property "Reference" "D4"
 			(at 73.66 44.45 0)
 			(effects
@@
 			(project "EMBARCADOS - CURSO PCB"
 				(path "/d5268f1b-b782-4609-86ee-ff462c2ec1ad/25e9c17a-dec3-4329-9bcf-5cd51d1774f7"
-					(reference "D1")
+					(reference "D4")
 					(unit 1)
 				)
@@
 		(on_board yes)
 		(dnp no)
-		(property "Reference" "R3"
+		(property "Reference" "R1"
 			(at 99.06 181.61 90)
 			(effects
@@
 			(project "EMBARCADOS - CURSO PCB"
 				(path "/d5268f1b-b782-4609-86ee-ff462c2ec1ad/25e9c17a-dec3-4329-9bcf-5cd51d1774f7"
-					(reference "R3")
+					(reference "R1")
 					(unit 1)
 				)
@@
 		(on_board yes)
 		(dnp no)
-		(property "Reference" "C7"
+		(property "Reference" "C12"
 			(at 256.54 120.6562 0)
 			(effects
@@
 			(project "EMBARCADOS - CURSO PCB"
 				(path "/d5268f1b-b782-4609-86ee-ff462c2ec1ad/25e9c17a-dec3-4329-9bcf-5cd51d1774f7"
-					(reference "C7")
+					(reference "C12")
 					(unit 1)
 				)
@@
 		(on_board yes)
 		(dnp no)
-		(property "Reference" "J1"
+		(property "Reference" "J2"
 			(at 40.64 63.5 0)
 			(effects
@@
 			(project "EMBARCADOS - CURSO PCB"
 				(path "/d5268f1b-b782-4609-86ee-ff462c2ec1ad/25e9c17a-dec3-4329-9bcf-5cd51d1774f7"
-					(reference "J1")
+					(reference "J2")
 					(unit 1)
 				)
@@
 		(dnp no)
 		(fields_autoplaced yes)
-		(property "Reference" "U1"
+		(property "Reference" "U3"
 			(at 127 110.49 0)
 			(effects
@@
 			(project "EMBARCADOS - CURSO PCB"
 				(path "/d5268f1b-b782-4609-86ee-ff462c2ec1ad/25e9c17a-dec3-4329-9bcf-5cd51d1774f7"
-					(reference "U1")
+					(reference "U3")
 					(unit 1)
 				)
@@
 		(dnp no)
 		(fields_autoplaced yes)
-		(property "Reference" "LED3"
+		(property "Reference" "LED1"
 			(at 105.41 169.2274 90)
 			(effects
@@
 			(project "EMBARCADOS - CURSO PCB"
 				(path "/d5268f1b-b782-4609-86ee-ff462c2ec1ad/25e9c17a-dec3-4329-9bcf-5cd51d1774f7"
-					(reference "LED3")
+					(reference "LED1")
 					(unit 1)
 				)
@@
 		(on_board yes)
 		(dnp no)
-		(property "Reference" "JP2"
+		(property "Reference" "JP1"
 			(at 196.85 54.61 0)
 			(effects
@@
 			(project "EMBARCADOS - CURSO PCB"
 				(path "/d5268f1b-b782-4609-86ee-ff462c2ec1ad/25e9c17a-dec3-4329-9bcf-5cd51d1774f7"
-					(reference "JP2")
+					(reference "JP1")
 					(unit 1)
 				)
@@
 		(on_board yes)
 		(dnp no)
-		(property "Reference" "D2"
+		(property "Reference" "D3"
 			(at 99.06 44.45 0)
 			(effects
@@
 			(project "EMBARCADOS - CURSO PCB"
 				(path "/d5268f1b-b782-4609-86ee-ff462c2ec1ad/25e9c17a-dec3-4329-9bcf-5cd51d1774f7"
-					(reference "D2")
+					(reference "D3")
 					(unit 1)
 				)
@@
 		(dnp no)
 		(fields_autoplaced yes)
-		(property "Reference" "LED1"
+		(property "Reference" "LED5"
 			(at 54.61 169.2274 90)
 			(effects
@@
 			(project "EMBARCADOS - CURSO PCB"
 				(path "/d5268f1b-b782-4609-86ee-ff462c2ec1ad/25e9c17a-dec3-4329-9bcf-5cd51d1774f7"
-					(reference "LED1")
+					(reference "LED5")
 					(unit 1)
 				)
@@
 		(on_board yes)
 		(dnp no)
-		(property "Reference" "R6"
+		(property "Reference" "R13"
 			(at 130.81 63.5 90)
 			(effects
@@
 			(project "EMBARCADOS - CURSO PCB"
 				(path "/d5268f1b-b782-4609-86ee-ff462c2ec1ad/25e9c17a-dec3-4329-9bcf-5cd51d1774f7"
-					(reference "R6")
+					(reference "R13")
 					(unit 1)
 				)
@@
 		(on_board yes)
 		(dnp no)
-		(property "Reference" "R1"
+		(property "Reference" "R21"
 			(at 48.26 181.61 90)
 			(effects
@@
 			(project "EMBARCADOS - CURSO PCB"
 				(path "/d5268f1b-b782-4609-86ee-ff462c2ec1ad/25e9c17a-dec3-4329-9bcf-5cd51d1774f7"
-					(reference "R1")
+					(reference "R21")
 					(unit 1)
 				)
@@
 		(on_board yes)
 		(dnp no)
-		(property "Reference" "D3"
+		(property "Reference" "D1"
 			(at 171.45 54.61 0)
 			(effects
@@
 			(project "EMBARCADOS - CURSO PCB"
 				(path "/d5268f1b-b782-4609-86ee-ff462c2ec1ad/25e9c17a-dec3-4329-9bcf-5cd51d1774f7"
-					(reference "D3")
+					(reference "D1")
 					(unit 1)
 				)
@@
 		(on_board yes)
 		(dnp no)
-		(property "Reference" "C2"
+		(property "Reference" "C4"
 			(at 124.46 68.5862 0)
 			(effects
@@
 			(project "EMBARCADOS - CURSO PCB"
 				(path "/d5268f1b-b782-4609-86ee-ff462c2ec1ad/25e9c17a-dec3-4329-9bcf-5cd51d1774f7"
-					(reference "C2")
+					(reference "C4")
 					(unit 1)
 				)
@@
 		(on_board yes)
 		(dnp no)
-		(property "Reference" "C4"
+		(property "Reference" "C6"
 			(at 200.66 120.6562 0)
 			(effects
@@
 			(project "EMBARCADOS - CURSO PCB"
 				(path "/d5268f1b-b782-4609-86ee-ff462c2ec1ad/25e9c17a-dec3-4329-9bcf-5cd51d1774f7"
-					(reference "C4")
+					(reference "C6")
 					(unit 1)
 				)
@@
 		(dnp no)
 		(fields_autoplaced yes)
-		(property "Reference" "LED4"
+		(property "Reference" "LED2"
 			(at 130.81 169.2274 90)
 			(effects
@@
 			(project "EMBARCADOS - CURSO PCB"
 				(path "/d5268f1b-b782-4609-86ee-ff462c2ec1ad/25e9c17a-dec3-4329-9bcf-5cd51d1774f7"
-					(reference "LED4")
+					(reference "LED2")
 					(unit 1)
 				)
@@
 		(on_board yes)
 		(dnp no)
-		(property "Reference" "C3"
+		(property "Reference" "C9"
 			(at 142.24 120.6562 0)
 			(effects
@@
 			(project "EMBARCADOS - CURSO PCB"
 				(path "/d5268f1b-b782-4609-86ee-ff462c2ec1ad/25e9c17a-dec3-4329-9bcf-5cd51d1774f7"
-					(reference "C3")
+					(reference "C9")
 					(unit 1)
 				)
@@
 		(dnp no)
 		(fields_autoplaced yes)
-		(property "Reference" "R8"
+		(property "Reference" "R2"
 			(at 180.34 74.9299 0)
 			(effects
@@
 			(project "EMBARCADOS - CURSO PCB"
 				(path "/d5268f1b-b782-4609-86ee-ff462c2ec1ad/25e9c17a-dec3-4329-9bcf-5cd51d1774f7"
-					(reference "R8")
+					(reference "R2")
 					(unit 1)
 				)
@@
 		(on_board yes)
 		(dnp no)
-		(property "Reference" "R4"
+		(property "Reference" "R9"
 			(at 124.46 181.61 90)
 			(effects
@@
 			(project "EMBARCADOS - CURSO PCB"
 				(path "/d5268f1b-b782-4609-86ee-ff462c2ec1ad/25e9c17a-dec3-4329-9bcf-5cd51d1774f7"
-					(reference "R4")
+					(reference "R9")
 					(unit 1)
 				)
@@
 		(dnp no)
 		(fields_autoplaced yes)
-		(property "Reference" "LED5"
+		(property "Reference" "LED3"
 			(at 156.21 169.2274 90)
 			(effects
@@
 			(project "EMBARCADOS - CURSO PCB"
 				(path "/d5268f1b-b782-4609-86ee-ff462c2ec1ad/25e9c17a-dec3-4329-9bcf-5cd51d1774f7"
-					(reference "LED5")
+					(reference "LED3")
 					(unit 1)
 				)
@@
 		(on_board yes)
 		(dnp no)
-		(property "Reference" "C6"
+		(property "Reference" "C1"
 			(at 193.04 68.5862 0)
 			(effects
@@
 			(project "EMBARCADOS - CURSO PCB"
 				(path "/d5268f1b-b782-4609-86ee-ff462c2ec1ad/25e9c17a-dec3-4329-9bcf-5cd51d1774f7"
-					(reference "C6")
+					(reference "C1")
 					(unit 1)
 				)
@@
 		(dnp no)
 		(fields_autoplaced yes)
-		(property "Reference" "R7"
+		(property "Reference" "R3"
 			(at 180.34 62.2299 0)
 			(effects
@@
 			(project "EMBARCADOS - CURSO PCB"
 				(path "/d5268f1b-b782-4609-86ee-ff462c2ec1ad/25e9c17a-dec3-4329-9bcf-5cd51d1774f7"
-					(reference "R7")
+					(reference "R3")
 					(unit 1)
 				)
@@
 		(on_board yes)
 		(dnp no)
-		(property "Reference" "R2"
+		(property "Reference" "R20"
 			(at 73.66 181.61 90)
 			(effects
@@
 			(project "EMBARCADOS - CURSO PCB"
 				(path "/d5268f1b-b782-4609-86ee-ff462c2ec1ad/25e9c17a-dec3-4329-9bcf-5cd51d1774f7"
-					(reference "R2")
+					(reference "R20")
 					(unit 1)
 				)
@@
 		(on_board yes)
 		(dnp no)
-		(property "Reference" "JP1"
+		(property "Reference" "JP2"
 			(at 120.65 54.61 0)
 			(effects
@@
 			(project "EMBARCADOS - CURSO PCB"
 				(path "/d5268f1b-b782-4609-86ee-ff462c2ec1ad/25e9c17a-dec3-4329-9bcf-5cd51d1774f7"
-					(reference "JP1")
+					(reference "JP2")
 					(unit 1)
 				)
@@
 		(on_board yes)
 		(dnp no)
-		(property "Reference" "U2"
+		(property "Reference" "U1"
 			(at 151.13 60.96 0)
 			(effects
@@
 			(project "EMBARCADOS - CURSO PCB"
 				(path "/d5268f1b-b782-4609-86ee-ff462c2ec1ad/25e9c17a-dec3-4329-9bcf-5cd51d1774f7"
-					(reference "U2")
+					(reference "U1")
 					(unit 1)
 				)
@@
 		(dnp no)
 		(fields_autoplaced yes)
-		(property "Reference" "U3"
+		(property "Reference" "U2"
 			(at 215.9 110.49 0)
 			(effects
@@
 			(project "EMBARCADOS - CURSO PCB"
 				(path "/d5268f1b-b782-4609-86ee-ff462c2ec1ad/25e9c17a-dec3-4329-9bcf-5cd51d1774f7"
-					(reference "U3")
+					(reference "U2")
 					(unit 1)
 				)

Commit message: Refactoring after Class 08.07 Part 5.
Parts:
- renumbered R9 to R4, R10 to R5
Changed lines of the file:
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@@
 		(on_board yes)
 		(dnp no)
-		(property "Reference" "R10"
+		(property "Reference" "R5"
 			(at 149.86 181.61 90)
 			(effects
@@
 			(project "EMBARCADOS - CURSO PCB"
 				(path "/d5268f1b-b782-4609-86ee-ff462c2ec1ad/25e9c17a-dec3-4329-9bcf-5cd51d1774f7"
-					(reference "R10")
+					(reference "R5")
 					(unit 1)
 				)
@@
 		(on_board yes)
 		(dnp no)
-		(property "Reference" "R9"
+		(property "Reference" "R4"
 			(at 124.46 181.61 90)
 			(effects
@@
 			(project "EMBARCADOS - CURSO PCB"
 				(path "/d5268f1b-b782-4609-86ee-ff462c2ec1ad/25e9c17a-dec3-4329-9bcf-5cd51d1774f7"
-					(reference "R9")
+					(reference "R4")
 					(unit 1)
 				)
