File: HARDWARE/KICAD/POWER.kicad_sch (KiCad schematic)
At the start: 32 parts, among them J2 3V-7V, U1 AP3012, U2 LD1117S50TR, U3 LD1117S33TR

Commit message: Finished PCB Layout.
Parts:
- renumbered R4 to R8, R5 to R9
Changed lines of the file:
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@@
 		(on_board yes)
 		(dnp no)
-		(property "Reference" "R5"
+		(property "Reference" "R9"
 			(at 149.86 181.61 90)
 			(effects
@@
 			(project "EMBARCADOS - CURSO PCB"
 				(path "/d5268f1b-b782-4609-86ee-ff462c2ec1ad/25e9c17a-dec3-4329-9bcf-5cd51d1774f7"
-					(reference "R5")
+					(reference "R9")
 					(unit 1)
 				)
@@
 		(on_board yes)
 		(dnp no)
-		(property "Reference" "R4"
+		(property "Reference" "R8"
 			(at 124.46 181.61 90)
 			(effects
@@
 			(project "EMBARCADOS - CURSO PCB"
 				(path "/d5268f1b-b782-4609-86ee-ff462c2ec1ad/25e9c17a-dec3-4329-9bcf-5cd51d1774f7"
-					(reference "R4")
+					(reference "R8")
 					(unit 1)
 				)

Commit message: Recorded Class 09.08. Generated PDFs for schematic and layout.
Other:
- note added: "BOOST OUT = 1.25 * (1 + R3/R2) +VBOOST = 7.125V"
- note removed: "BOOST OUT = 1.25 * (1 + R7/R8) +VBOOST = 7.125V"
Changed lines of the file:
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@@
 		)
 	)
-	(text "BOOST OUT = 1.25 * (1 + R7/R8)\n+VBOOST = 7.125V"
+	(text "BOOST OUT = 1.25 * (1 + R3/R2)\n+VBOOST = 7.125V"
 		(exclude_from_sim no)
 		(at 176.53 88.9 0)
@@
 				(thickness 0.254)
 				(bold yes)
-				(color 255 0 0 1)
+				(color 0 0 0 1)
 			)
 		)
