File: HARDWARE/KICAD/POWER.kicad_sch (KiCad schematic)
At the start: 32 parts, among them J2 3V-7V, U1 AP3012, U2 LD1117S50TR, U3 LD1117S33TR

Commit message: Finished overall project review for PCB fabrication at JLCPCB.
Parts:
- C1, C10, C12, C4, C5, C6, C9: LCSC Part # C15850 -> (none); LCSC Part #  (none) -> C15850
- D1, D3, D4: Manufactrer DIODES INCORPORATED -> (none); Manufacturer (none) -> DIODES INCORPORATED
- R3: LCSC MPN  0603WAF1002T5E -> 0603WAF4702T5E; LCSC Part #  C25804 -> C25819
Changed lines of the file:
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@@
 			)
 		)
-		(property "LCSC Part #" "C15850 "
-			(at 114.3 137.414 0)
+		(property "LCSC MPN " "CL21A106KAYNNNE "
+			(at 113.792 133.096 0)
 			(effects
 				(font
@@
 			)
 		)
-		(property "LCSC MPN " "CL21A106KAYNNNE "
-			(at 113.792 133.096 0)
+		(property "LCSC MANUFACTURER " "SAMSUNG "
+			(at 114.046 135.382 0)
 			(effects
 				(font
@@
 			)
 		)
-		(property "LCSC MANUFACTURER " "SAMSUNG "
-			(at 114.046 135.382 0)
+		(property "LCSC Part # " "C15850 "
+			(at 114.3 137.414 0)
 			(effects
 				(font
@@
 			)
 		)
-		(property "Manufactrer" "DIODES INCORPORATED "
-			(at 83.058 44.196 0)
-			(effects
-				(font
-					(size 1.27 1.27)
-				)
-				(hide yes)
-			)
-		)
 		(property "3D Model" "KiCad"
 			(at 81.28 44.45 0)
@@
 			)
 		)
+		(property "Manufacturer" "DIODES INCORPORATED "
+			(at 83.058 44.196 0)
+			(effects
+				(font
+					(size 1.27 1.27)
+				)
+				(hide yes)
+			)
+		)
 		(pin "2"
 		)
@@
 			)
 		)
-		(property "LCSC Part #" "C15850 "
-			(at 254 137.414 0)
+		(property "LCSC MPN " "CL21A106KAYNNNE "
+			(at 254.508 133.096 0)
 			(effects
 				(font
@@
 			)
 		)
-		(property "LCSC MPN " "CL21A106KAYNNNE "
-			(at 254.508 133.096 0)
+		(property "LCSC MANUFACTURER " "SAMSUNG "
+			(at 254.254 135.382 0)
 			(effects
 				(font
@@
 			)
 		)
-		(property "LCSC MANUFACTURER " "SAMSUNG "
-			(at 254.254 135.382 0)
+		(property "LCSC Part # " "C15850 "
+			(at 254 137.414 0)
 			(effects
 				(font
@@
 			)
 		)
-		(property "LCSC Part #" "C15850 "
-			(at 228.6 137.414 0)
+		(property "LCSC MPN " "CL21A106KAYNNNE "
+			(at 228.092 133.096 0)
 			(effects
 				(font
@@
 			)
 		)
-		(property "LCSC MPN " "CL21A106KAYNNNE "
-			(at 228.092 133.096 0)
+		(property "LCSC MANUFACTURER " "SAMSUNG "
+			(at 228.346 135.382 0)
 			(effects
 				(font
@@
 			)
 		)
-		(property "LCSC MANUFACTURER " "SAMSUNG "
-			(at 228.346 135.382 0)
+		(property "LCSC Part # " "C15850 "
+			(at 228.6 137.414 0)
 			(effects
 				(font
@@
 			)
 		)
-		(property "Manufactrer" "DIODES INCORPORATED "
-			(at 108.458 44.196 0)
-			(effects
-				(font
-					(size 1.27 1.27)
-				)
-				(hide yes)
-			)
-		)
 		(property "3D Model" "KiCad"
 			(at 106.68 44.45 0)
@@
 			)
 		)
+		(property "Manufacturer" "DIODES INCORPORATED "
+			(at 108.458 44.196 0)
+			(effects
+				(font
+					(size 1.27 1.27)
+				)
+				(hide yes)
+			)
+		)
 		(pin "2"
 		)
@@
 			)
 		)
-		(property "Manufactrer" "DIODES INCORPORATED "
-			(at 171.196 64.008 0)
-			(effects
-				(font
-					(size 1.27 1.27)
-				)
-				(hide yes)
-			)
-		)
 		(property "3D Model" "KiCad"
 			(at 171.45 62.23 0)
@@
 			)
 		)
+		(property "Manufacturer" "DIODES INCORPORATED "
+			(at 171.196 64.008 0)
+			(effects
+				(font
+					(size 1.27 1.27)
+				)
+				(hide yes)
+			)
+		)
 		(pin "1"
 		)
@@
 			)
 		)
-		(property "LCSC Part #" "C15850 "
-			(at 127 85.344 0)
+		(property "LCSC MPN " "CL21A106KAYNNNE "
+			(at 126.492 81.026 0)
 			(effects
 				(font
@@
 			)
 		)
-		(property "LCSC MPN " "CL21A106KAYNNNE "
-			(at 126.492 81.026 0)
+		(property "LCSC MANUFACTURER " "SAMSUNG "
+			(at 126.746 83.312 0)
 			(effects
 				(font
@@
 			)
 		)
-		(property "LCSC MANUFACTURER " "SAMSUNG "
-			(at 126.746 83.312 0)
+		(property "LCSC Part # " "C15850 "
+			(at 127 85.344 0)
 			(effects
 				(font
@@
 			)
 		)
-		(property "LCSC Part #" "C15850 "
-			(at 203.2 137.414 0)
+		(property "LCSC MPN " "CL21A106KAYNNNE "
+			(at 202.692 133.096 0)
 			(effects
 				(font
@@
 			)
 		)
-		(property "LCSC MPN " "CL21A106KAYNNNE "
-			(at 202.692 133.096 0)
+		(property "LCSC MANUFACTURER " "SAMSUNG "
+			(at 202.946 135.382 0)
 			(effects
 				(font
@@
 			)
 		)
-		(property "LCSC MANUFACTURER " "SAMSUNG "
-			(at 202.946 135.382 0)
+		(property "LCSC Part # " "C15850 "
+			(at 203.2 137.414 0)
 			(effects
 				(font
@@
 			)
 		)
-		(property "LCSC Part #" "C15850 "
-			(at 139.7 137.414 0)
+		(property "LCSC MPN " "CL21A106KAYNNNE "
+			(at 140.208 133.096 0)
 			(effects
 				(font
@@
 			)
 		)
-		(property "LCSC MPN " "CL21A106KAYNNNE "
-			(at 140.208 133.096 0)
+		(property "LCSC MANUFACTURER " "SAMSUNG "
+			(at 139.954 135.382 0)
 			(effects
 				(font
@@
 			)
 		)
-		(property "LCSC MANUFACTURER " "SAMSUNG "
-			(at 139.954 135.382 0)
+		(property "LCSC Part # " "C15850 "
+			(at 139.7 137.414 0)
 			(effects
 				(font
@@
 			)
 		)
-		(property "LCSC Part #" "C15850 "
-			(at 190.5 85.344 0)
+		(property "LCSC MPN " "CL21A106KAYNNNE "
+			(at 191.008 81.026 0)
 			(effects
 				(font
@@
 			)
 		)
-		(property "LCSC MPN " "CL21A106KAYNNNE "
-			(at 191.008 81.026 0)
+		(property "LCSC MANUFACTURER " "SAMSUNG "
+			(at 190.754 83.312 0)
 			(effects
 				(font
@@
 			)
 		)
-		(property "LCSC MANUFACTURER " "SAMSUNG "
-			(at 190.754 83.312 0)
+		(property "LCSC Part # " "C15850 "
+			(at 190.5 85.344 0)
 			(effects
 				(font
@@
 			)
 		)
-		(property "LCSC Part # " "C25804 "
+		(property "LCSC Part # " "C25819"
 			(at 178.054 88.392 0)
 			(effects
@@
 			)
 		)
-		(property "LCSC MPN " "0603WAF1002T5E "
+		(property "LCSC MPN " "0603WAF4702T5E"
 			(at 178.054 83.82 0)
 			(effects
