File: HARDWARE/KICAD/INTERFACE.kicad_sch (KiCad schematic)
At the start: 20 parts, among them Q3 2N7002K, SW1 UP, SW2 DOWN, SW3 LEFT, SW4 RIGHT, SW5 CENTER, U8 OLED 1.3" 128x64

Commit message: Refactoring.
Parts:
- added R52, R53: 10K 1%, EMBARCADOS - CURSO PCB:R_0603_1608Metric, symbol EMBARCADOS - CURSO PCB:RES 0603 10K 1% VISHAY CRCW060310K0FK
- added SW6: BUTTON 1, EMBARCADOS - CURSO PCB:C&K PTS526SM20SMTR21 LFS, symbol EMBARCADOS - CURSO PCB:SWITCH TACTILE C&K PTS526SM20SMTR21 LFS
- added SW7: BUTTON 2, EMBARCADOS - CURSO PCB:C&K PTS526SM20SMTR21 LFS, symbol EMBARCADOS - CURSO PCB:SWITCH TACTILE C&K PTS526SM20SMTR21 LFS
Connections:
- net +3.3V: now also R52.1, R53.1
- net BUTTON 1: now also R52.2, SW6.3 (B), SW6.4 (B)
- net BUTTON 2: now also R53.2, SW7.3 (B), SW7.4 (B)
- net BUTTON CENTER: now also R51.2, SW5.3 (B), SW5.4 (B)
- net BUTTON LEFT: now also R49.2, SW3.3 (B), SW3.4 (B)
- net BUTTON RIGHT: now also R50.2, SW4.3 (B), SW4.4 (B)
- net GND: now also SW6.1 (A), SW6.2 (A), SW7.1 (A), SW7.2 (A)
- net BUZZER DRAIN: now reaches LS1.2, Q3.3 (D), R45.2
Other:
- moved on the sheet: C41, C42, C43, D5, D6, LS1, Q3, R45, R46, R47, R48, R49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

Commit message: Finished schematic.
Parts:
- added C45: 100nF 50V, EMBARCADOS - CURSO PCB:C_0603_1608Metric, symbol EMBARCADOS - CURSO PCB:CAP 0603 100nF 50V AVX KGM15BR71H104K
- added R54, R55: 10K 1%, EMBARCADOS - CURSO PCB:R_0603_1608Metric, symbol EMBARCADOS - CURSO PCB:RES 0603 10K 1% VISHAY CRCW060310K0FK
- added SW8: ~{RST}, EMBARCADOS - CURSO PCB:C&K PTS526SM20SMTR21 LFS, symbol EMBARCADOS - CURSO PCB:SWITCH TACTILE C&K PTS526SM20SMTR21 LFS
- added SW9: BOOT, EMBARCADOS - CURSO PCB:C&K PTS526SM20SMTR21 LFS, symbol EMBARCADOS - CURSO PCB:SWITCH TACTILE C&K PTS526SM20SMTR21 LFS
Connections:
- net +3.3V: now also R54.1, SW9.3 (B), SW9.4 (B)
- net +5V: now also C45.2
- net BOOT0: now also R55.1, SW9.1 (A), SW9.2 (A)
- net GND: now also C45.1, R55.2, SW8.1 (A), SW8.2 (A)
- net NRST: now also R54.2, SW8.3 (B), SW8.4 (B)
Other:
- note removed: "BOTÃO BOOT0"

Commit message: Finished initial positioning.
Connections:
- net +3.3V: now also SW9.2 (B); no longer SW9.3 (B), SW9.4 (B)
- net BOOT0: no longer SW9.2 (A)
- net BUTTON 1: now also SW6.2 (B); no longer SW6.3 (B), SW6.4 (B)
- net BUTTON 2: now also SW7.2 (B); no longer SW7.3 (B), SW7.4 (B)
- net BUTTON CENTER: now also SW5.2 (B); no longer SW5.3 (B), SW5.4 (B)
- net BUTTON DOWN: now also SW2.2 (B); no longer SW2.3 (B), SW2.4 (B)
- net BUTTON LEFT: now also SW3.2 (B); no longer SW3.3 (B), SW3.4 (B)
- net BUTTON RIGHT: now also SW4.2 (B); no longer SW4.3 (B), SW4.4 (B)
- net BUTTON UP: now also SW1.2 (B); no longer SW1.3 (B), SW1.4 (B)
- net GND: no longer SW1.2 (A), SW2.2 (A), SW3.2 (A), SW4.2 (A), SW5.2 (A), SW6.2 (A), SW7.2 (A), SW8.2 (A)
- net NRST: now also SW8.2 (B); no longer SW8.3 (B), SW8.4 (B)
Changed lines of the file:
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@@
 		(pin "2"
 		)
-		(pin "3"
-		)
 		(pin "1"
 		)
-		(pin "4"
-		)
 		(instances
 			(project "EMBARCADOS - CURSO PCB"
@@
 		(pin "2"
 		)
-		(pin "3"
-		)
 		(pin "1"
 		)
-		(pin "4"
-		)
 		(instances
 			(project "EMBARCADOS - CURSO PCB"
@@
 		(pin "2"
 		)
-		(pin "3"
-		)
 		(pin "1"
 		)
-		(pin "4"
-		)
 		(instances
 			(project "EMBARCADOS - CURSO PCB"
@@
 		(pin "2"
 		)
-		(pin "3"
-		)
 		(pin "1"
 		)
-		(pin "4"
-		)
 		(instances
 			(project "EMBARCADOS - CURSO PCB"
@@
 		(pin "2"
 		)
-		(pin "3"
-		)
 		(pin "1"
 		)
-		(pin "4"
-		)
 		(instances
 			(project "EMBARCADOS - CURSO PCB"
@@
 		(pin "2"
 		)
-		(pin "3"
-		)
 		(pin "1"
 		)
-		(pin "4"
-		)
 		(instances
 			(project ""
@@
 		(pin "2"
 		)
-		(pin "3"
-		)
 		(pin "1"
 		)
-		(pin "4"
-		)
 		(instances
 			(project "EMBARCADOS - CURSO PCB"
@@
 		(pin "2"
 		)
-		(pin "3"
-		)
 		(pin "1"
 		)
-		(pin "4"
-		)
 		(instances
 			(project "EMBARCADOS - CURSO PCB"
@@
 		(pin "2"
 		)
-		(pin "3"
-		)
 		(pin "1"
 		)
-		(pin "4"
-		)
 		(instances

Commit message: Recorded Class 08.07 Part 5.
Parts:
- renumbered C42 to C11, C43 to C13, C45 to C2, C41 to C3, D5 to D2, Q3 to Q1, R45 to R11, R46 to R12, R54 to R15, R55 to R16, R47 to R49, R49 to R50, R50 to R51, R51 to R54, R48 to R55, SW8 to SW1, SW9 to SW2, SW1 to SW3, SW3 to SW4, SW4 to SW6, SW6 to SW7, SW7 to SW8, SW2 to SW9
Changed lines of the file:
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@@
 		(on_board yes)
 		(dnp no)
-		(property "Reference" "R45"
+		(property "Reference" "R11"
 			(at 226.06 40.64 0)
 			(effects
@@
 			(project ""
 				(path "/d5268f1b-b782-4609-86ee-ff462c2ec1ad/6145c3a7-bcf4-4534-931d-bf3c6674fe6b"
-					(reference "R45")
+					(reference "R11")
 					(unit 1)
 				)
@@
 		(dnp no)
 		(fields_autoplaced yes)
-		(property "Reference" "R49"
+		(property "Reference" "R50"
 			(at 104.14 106.6799 0)
 			(effects
@@
 			(project "EMBARCADOS - CURSO PCB"
 				(path "/d5268f1b-b782-4609-86ee-ff462c2ec1ad/6145c3a7-bcf4-4534-931d-bf3c6674fe6b"
-					(reference "R49")
+					(reference "R50")
 					(unit 1)
 				)
@@
 		(on_board yes)
 		(dnp no)
-		(property "Reference" "C43"
+		(property "Reference" "C13"
 			(at 142.24 40.64 90)
 			(effects
@@
 			(project ""
 				(path "/d5268f1b-b782-4609-86ee-ff462c2ec1ad/6145c3a7-bcf4-4534-931d-bf3c6674fe6b"
-					(reference "C43")
+					(reference "C13")
 					(unit 1)
 				)
@@
 		(dnp no)
 		(fields_autoplaced yes)
-		(property "Reference" "R55"
+		(property "Reference" "R16"
 			(at 154.94 171.4499 0)
 			(effects
@@
 			(project "EMBARCADOS - CURSO PCB"
 				(path "/d5268f1b-b782-4609-86ee-ff462c2ec1ad/6145c3a7-bcf4-4534-931d-bf3c6674fe6b"
-					(reference "R55")
+					(reference "R16")
 					(unit 1)
 				)
@@
 		(on_board yes)
 		(dnp no)
-		(property "Reference" "SW4"
+		(property "Reference" "SW6"
 			(at 128.27 120.6499 90)
 			(effects
@@
 			(project "EMBARCADOS - CURSO PCB"
 				(path "/d5268f1b-b782-4609-86ee-ff462c2ec1ad/6145c3a7-bcf4-4534-931d-bf3c6674fe6b"
-					(reference "SW4")
+					(reference "SW6")
 					(unit 1)
 				)
@@
 		(dnp no)
 		(fields_autoplaced yes)
-		(property "Reference" "R48"
+		(property "Reference" "R55"
 			(at 78.74 106.6799 0)
 			(effects
@@
 			(project "EMBARCADOS - CURSO PCB"
 				(path "/d5268f1b-b782-4609-86ee-ff462c2ec1ad/6145c3a7-bcf4-4534-931d-bf3c6674fe6b"
-					(reference "R48")
+					(reference "R55")
 					(unit 1)
 				)
@@
 		(on_board yes)
 		(dnp no)
-		(property "Reference" "C45"
+		(property "Reference" "C2"
 			(at 44.45 46.99 90)
 			(effects
@@
 			(project "EMBARCADOS - CURSO PCB"
 				(path "/d5268f1b-b782-4609-86ee-ff462c2ec1ad/6145c3a7-bcf4-4534-931d-bf3c6674fe6b"
-					(reference "C45")
+					(reference "C2")
 					(unit 1)
 				)
@@
 		(on_board yes)
 		(dnp no)
-		(property "Reference" "SW6"
+		(property "Reference" "SW7"
 			(at 204.47 120.6499 90)
 			(effects
@@
 			(project "EMBARCADOS - CURSO PCB"
 				(path "/d5268f1b-b782-4609-86ee-ff462c2ec1ad/6145c3a7-bcf4-4534-931d-bf3c6674fe6b"
-					(reference "SW6")
+					(reference "SW7")
 					(unit 1)
 				)
@@
 		(on_board yes)
 		(dnp no)
-		(property "Reference" "Q3"
+		(property "Reference" "Q1"
 			(at 232.41 57.15 0)
 			(effects
@@
 			(project ""
 				(path "/d5268f1b-b782-4609-86ee-ff462c2ec1ad/6145c3a7-bcf4-4534-931d-bf3c6674fe6b"
-					(reference "Q3")
+					(reference "Q1")
 					(unit 1)
 				)
@@
 		(on_board yes)
 		(dnp no)
-		(property "Reference" "SW7"
+		(property "Reference" "SW8"
 			(at 229.87 120.6499 90)
 			(effects
@@
 			(project "EMBARCADOS - CURSO PCB"
 				(path "/d5268f1b-b782-4609-86ee-ff462c2ec1ad/6145c3a7-bcf4-4534-931d-bf3c6674fe6b"
-					(reference "SW7")
+					(reference "SW8")
 					(unit 1)
 				)
@@
 		(on_board yes)
 		(dnp no)
-		(property "Reference" "C42"
+		(property "Reference" "C11"
 			(at 142.24 30.48 90)
 			(effects
@@
 			(project "EMBARCADOS - CURSO PCB"
 				(path "/d5268f1b-b782-4609-86ee-ff462c2ec1ad/6145c3a7-bcf4-4534-931d-bf3c6674fe6b"
-					(reference "C42")
+					(reference "C11")
 					(unit 1)
 				)
@@
 		(on_board yes)
 		(dnp no)
-		(property "Reference" "SW9"
+		(property "Reference" "SW2"
 			(at 153.67 156.2099 90)
 			(effects
@@
 			(project "EMBARCADOS - CURSO PCB"
 				(path "/d5268f1b-b782-4609-86ee-ff462c2ec1ad/6145c3a7-bcf4-4534-931d-bf3c6674fe6b"
-					(reference "SW9")
+					(reference "SW2")
 					(unit 1)
 				)
@@
 		(dnp no)
 		(fields_autoplaced yes)
-		(property "Reference" "R51"
+		(property "Reference" "R54"
 			(at 154.94 106.6799 0)
 			(effects
@@
 			(project "EMBARCADOS - CURSO PCB"
 				(path "/d5268f1b-b782-4609-86ee-ff462c2ec1ad/6145c3a7-bcf4-4534-931d-bf3c6674fe6b"
-					(reference "R51")
+					(reference "R54")
 					(unit 1)
 				)
@@
 		(dnp no)
 		(fields_autoplaced yes)
-		(property "Reference" "R50"
+		(property "Reference" "R51"
 			(at 129.54 106.6799 0)
 			(effects
@@
 			(project "EMBARCADOS - CURSO PCB"
 				(path "/d5268f1b-b782-4609-86ee-ff462c2ec1ad/6145c3a7-bcf4-4534-931d-bf3c6674fe6b"
-					(reference "R50")
+					(reference "R51")
 					(unit 1)
 				)
@@
 		(dnp no)
 		(fields_autoplaced yes)
-		(property "Reference" "R47"
+		(property "Reference" "R49"
 			(at 53.34 106.6799 0)
 			(effects
@@
 			(project "EMBARCADOS - CURSO PCB"
 				(path "/d5268f1b-b782-4609-86ee-ff462c2ec1ad/6145c3a7-bcf4-4534-931d-bf3c6674fe6b"
-					(reference "R47")
+					(reference "R49")
 					(unit 1)
 				)
@@
 		(on_board yes)
 		(dnp no)
-		(property "Reference" "D5"
+		(property "Reference" "D2"
 			(at 46.99 55.88 0)
 			(effects
@@
 			(project ""
 				(path "/d5268f1b-b782-4609-86ee-ff462c2ec1ad/6145c3a7-bcf4-4534-931d-bf3c6674fe6b"
-					(reference "D5")
+					(reference "D2")
 					(unit 1)
 				)
@@
 		(on_board yes)
 		(dnp no)
-		(property "Reference" "SW1"
+		(property "Reference" "SW3"
 			(at 52.07 120.6499 90)
 			(effects
@@
 			(project ""
 				(path "/d5268f1b-b782-4609-86ee-ff462c2ec1ad/6145c3a7-bcf4-4534-931d-bf3c6674fe6b"
-					(reference "SW1")
+					(reference "SW3")
 					(unit 1)
 				)
@@
 		(on_board yes)
 		(dnp no)
-		(property "Reference" "R46"
+		(property "Reference" "R12"
 			(at 214.63 63.5 0)
 			(effects
@@
 			(project ""
 				(path "/d5268f1b-b782-4609-86ee-ff462c2ec1ad/6145c3a7-bcf4-4534-931d-bf3c6674fe6b"
-					(reference "R46")
+					(reference "R12")
 					(unit 1)
 				)
@@
 		(on_board yes)
 		(dnp no)
-		(property "Reference" "SW2"
+		(property "Reference" "SW9"
 			(at 77.47 120.6499 90)
 			(effects
@@
 			(project "EMBARCADOS - CURSO PCB"
 				(path "/d5268f1b-b782-4609-86ee-ff462c2ec1ad/6145c3a7-bcf4-4534-931d-bf3c6674fe6b"
-					(reference "SW2")
+					(reference "SW9")
 					(unit 1)
 				)
@@
 		(on_board yes)
 		(dnp no)
-		(property "Reference" "SW8"
+		(property "Reference" "SW1"
 			(at 128.27 171.4499 90)
 			(effects
@@
 			(project "EMBARCADOS - CURSO PCB"
 				(path "/d5268f1b-b782-4609-86ee-ff462c2ec1ad/6145c3a7-bcf4-4534-931d-bf3c6674fe6b"
-					(reference "SW8")
+					(reference "SW1")
 					(unit 1)
 				)
@@
 		(on_board yes)
 		(dnp no)
-		(property "Reference" "SW3"
+		(property "Reference" "SW4"
 			(at 102.87 120.6499 90)
 			(effects
@@
 			(project "EMBARCADOS - CURSO PCB"
 				(path "/d5268f1b-b782-4609-86ee-ff462c2ec1ad/6145c3a7-bcf4-4534-931d-bf3c6674fe6b"
-					(reference "SW3")
+					(reference "SW4")
 					(unit 1)
 				)
@@
 		(dnp no)
 		(fields_autoplaced yes)
-		(property "Reference" "R54"
+		(property "Reference" "R15"
 			(at 129.54 156.2099 0)
 			(effects
@@
 			(project "EMBARCADOS - CURSO PCB"
 				(path "/d5268f1b-b782-4609-86ee-ff462c2ec1ad/6145c3a7-bcf4-4534-931d-bf3c6674fe6b"
-					(reference "R54")
+					(reference "R15")
 					(unit 1)
 				)
@@
 		(on_board yes)
 		(dnp no)
-		(property "Reference" "C41"
+		(property "Reference" "C3"
 			(at 222.25 30.48 90)
 			(effects
@@
 			(project ""
 				(path "/d5268f1b-b782-4609-86ee-ff462c2ec1ad/6145c3a7-bcf4-4534-931d-bf3c6674fe6b"
-					(reference "C41")
+					(reference "C3")
 					(unit 1)
 				)

Commit message: Refactoring after Class 08.07 Part 5.
Parts:
- renumbered D6 to D7, U8 to U6
Changed lines of the file:
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@@
 		(on_board yes)
 		(dnp no)
-		(property "Reference" "U8"
+		(property "Reference" "U6"
 			(at 140.97 53.34 0)
 			(effects
@@
 			(project ""
 				(path "/d5268f1b-b782-4609-86ee-ff462c2ec1ad/6145c3a7-bcf4-4534-931d-bf3c6674fe6b"
-					(reference "U8")
+					(reference "U6")
 					(unit 1)
 				)
@@
 		(on_board yes)
 		(dnp no)
-		(property "Reference" "D6"
+		(property "Reference" "D7"
 			(at 114.3 50.8 0)
 			(effects
@@
 			(project ""
 				(path "/d5268f1b-b782-4609-86ee-ff462c2ec1ad/6145c3a7-bcf4-4534-931d-bf3c6674fe6b"
-					(reference "D6")
+					(reference "D7")
 					(unit 1)
 				)

Commit message: Refactoring before Class 08.07 Part 6.
Changed lines of the file:
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@@
+	)
+	(symbol
+		(lib_id "EMBARCADOS - CURSO PCB:DISPLAY OLED 1.3{dblquote} 128x64")
+		(at 152.4 63.5 0)
+		(unit 1)
+		(exclude_from_sim no)
+		(in_bom yes)
+		(on_board yes)
+		(dnp no)
+		(fields_autoplaced yes)
+		(property "Reference" "U6"
+			(at 165.1 62.2299 0)
+			(effects
+				(font
+					(size 1.27 1.27)
+				)
+				(justify left)
+			)
+		)
+		(property "Value" "OLED 1.3\" 128x64"
+			(at 165.1 64.7699 0)
+			(effects
+				(font
+					(size 1.27 1.27)
+				)
+				(justify left)
+			)
+		)
+		(property "Footprint" "EMBARCADOS - CURSO PCB:OLED 128x64 1.3in"
+			(at 152.4 57.15 0)
+			(effects
+				(font
+					(size 1.27 1.27)
+				)
+				(hide yes)
+			)
+		)
+		(property "Datasheet" "https://www.we-online.com/components/products/datasheet/61300411821.pdf"
+			(at 152.146 82.042 0)
+			(effects
+				(font
+					(size 1.27 1.27)
+				)
+				(hide yes)
+			)
+		)
+		(property "Description" "OLED 1.3\" 128x64"
+			(at 152.4 85.344 0)
+			(effects
+				(font
+					(size 1.27 1.27)
+				)
+				(hide yes)
+			)
+		)
+		(property "MPN" "61300411821 "
+			(at 152.4 78.74 0)
+			(effects
+				(font
+					(size 1.27 1.27)
+				)
+				(hide yes)
+			)
+		)
+		(property "Manufacturer" "WÜRTH ELEKTRONIK "
+			(at 152.4 78.74 0)
+			(effects
+				(font
+					(size 1.27 1.27)
+				)
+				(hide yes)
+			)
+		)
+		(property "3D Model" "https://www.we-online.com/components/products/download/61300411821%20%28rev1%29.iges"
+			(at 153.416 76.2 0)
+			(effects
+				(font
+					(size 1.27 1.27)
+				)
+				(hide yes)
+			)
+		)
+		(property "Notes" "THRU HOLE"
+			(at 152.4 78.74 0)
+			(effects
+				(font
+					(size 1.27 1.27)
+				)
+				(hide yes)
+			)
+		)
+		(property "LCSC Part # " "-"
+			(at 152.4 78.74 0)
+			(effects
+				(font
+					(size 1.27 1.27)
+				)
+				(hide yes)
+			)
+		)
+		(property "LCSC MPN " "-"
+			(at 152.4 78.74 0)
+			(effects
+				(font
+					(size 1.27 1.27)
+				)
+				(hide yes)
+			)
+		)
+		(property "LCSC MANUFACTURER " "-"
+			(at 152.4 78.74 0)
+			(effects
+				(font
+					(size 1.27 1.27)
+				)
+				(hide yes)
+			)
+		)
+		(pin "4"
+		)
+		(pin "3"
+		)
+		(pin "2"
+		)
+		(pin "1"
+		)
+		(instances
+			(project ""
+				(path "/d5268f1b-b782-4609-86ee-ff462c2ec1ad/6145c3a7-bcf4-4534-931d-bf3c6674fe6b"
+					(reference "U6")
+					(unit 1)
+				)
+			)
+		)
 	)
 	(symbol
@@
 					(unit 1)
 				)
-			)
-		)
-	)
-	(symbol
-		(lib_id "EMBARCADOS - CURSO PCB:DISPLAY OLED 1.3{dblquote} 128x64")
-		(at 152.4 63.5 0)
-		(unit 1)
-		(exclude_from_sim no)
-		(in_bom yes)
-		(on_board yes)
-		(dnp no)
-		(property "Reference" "U6"
-			(at 140.97 53.34 0)
-			(effects
-				(font
-					(size 1.27 1.27)
-				)
-				(justify left)
-			)
-		)
-		(property "Value" "OLED 1.3\" 128x64"
-			(at 152.4 73.66 0)
-			(effects
-				(font
-					(size 1.27 1.27)
-				)
-			)
-		)
-		(property "Footprint" "EMBARCADOS - CURSO PCB:OLED 128x64 1.3in"
-			(at 152.4 57.15 0)
-			(effects
-				(font
-					(size 1.27 1.27)
-				)
-				(hide yes)
-			)
-		)
-		(property "Datasheet" "https://www.we-online.com/components/products/datasheet/61300411821.pdf"
-			(at 152.146 82.042 0)
-			(effects
-				(font
-					(size 1.27 1.27)
-				)
-				(hide yes)
-			)
-		)
-		(property "Description" "OLED 1.3\" 128x64"
-			(at 152.4 85.344 0)
-			(effects
-				(font
-					(size 1.27 1.27)
-				)
-				(hide yes)
-			)
-		)
-		(property "MPN" "61300411821 "
-			(at 152.4 78.74 0)
-			(effects
-				(font
-					(size 1.27 1.27)
-				)
-				(hide yes)
-			)
-		)
-		(property "Manufacturer" "WÜRTH ELEKTRONIK "
-			(at 152.4 78.74 0)
-			(effects
-				(font
-					(size 1.27 1.27)
-				)
-				(hide yes)
-			)
-		)
-		(property "3D Model" "https://www.we-online.com/components/products/download/61300411821%20%28rev1%29.iges"
-			(at 153.416 76.2 0)
-			(effects
-				(font
-					(size 1.27 1.27)
-				)
-				(hide yes)
-			)
-		)
-		(property "Notes" "THRU HOLE"
-			(at 152.4 78.74 0)
-			(effects
-				(font
-					(size 1.27 1.27)
-				)
-				(hide yes)
-			)
-		)
-		(property "LCSC Part # " "-"
-			(at 152.4 78.74 0)
-			(effects
-				(font
-					(size 1.27 1.27)
-				)
-				(hide yes)
-			)
-		)
-		(property "LCSC MPN " "-"
-			(at 152.4 78.74 0)
-			(effects
-				(font
-					(size 1.27 1.27)
-				)
-				(hide yes)
-			)
-		)
-		(property "LCSC MANUFACTURER " "-"
-			(at 152.4 78.74 0)
-			(effects
-				(font
-					(size 1.27 1.27)
-				)
-				(hide yes)
-			)
-		)
-		(pin "2"
-		)
-		(pin "4"
-		)
-		(pin "3"
-		)
-		(pin "1"
-		)
-		(instances
-			(project ""
-				(path "/d5268f1b-b782-4609-86ee-ff462c2ec1ad/6145c3a7-bcf4-4534-931d-bf3c6674fe6b"
-					(reference "U6")
-					(unit 1)
-				)

Commit message: Finished PCB Layout.
Parts:
- renumbered R15 to R17, R16 to R18
Changed lines of the file:
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@@
 		(dnp no)
 		(fields_autoplaced yes)
-		(property "Reference" "R16"
+		(property "Reference" "R18"
 			(at 154.94 171.4499 0)
 			(effects
@@
 			(project "EMBARCADOS - CURSO PCB"
 				(path "/d5268f1b-b782-4609-86ee-ff462c2ec1ad/6145c3a7-bcf4-4534-931d-bf3c6674fe6b"
-					(reference "R16")
+					(reference "R18")
 					(unit 1)
 				)
@@
 		(dnp no)
 		(fields_autoplaced yes)
-		(property "Reference" "R15"
+		(property "Reference" "R17"
 			(at 129.54 156.2099 0)
 			(effects
@@
 			(project "EMBARCADOS - CURSO PCB"
 				(path "/d5268f1b-b782-4609-86ee-ff462c2ec1ad/6145c3a7-bcf4-4534-931d-bf3c6674fe6b"
-					(reference "R15")
+					(reference "R17")
 					(unit 1)
 				)
