File: HARDWARE/KICAD/INTERFACE.kicad_sch (KiCad schematic)
At the start: 29 parts, among them Q1 2N7002K, SW1 ~{RST}, SW2 BOOT, SW3 UP, SW4 LEFT, SW5 CENTER, SW6 RIGHT, SW7 BUTTON 1, SW8 BUTTON 2, SW9 DOWN, U6 OLED 1.3" 128x64

Commit message: Finished overall project review for PCB fabrication at JLCPCB.
Parts:
- C11, C3: LCSC Part # C15850 -> (none); LCSC Part #  (none) -> C15850
- C13, C2: LCSC Part # C14663 -> (none); LCSC Part #  (none) -> C14663
- SW1, SW2, SW3, SW4, SW5, SW6, SW7, SW8, SW9: LCSC MANUFACTURER  - -> XKB Connection; LCSC MPN  - -> TS-1187A-B-A-B; LCSC Part #  - -> C318884
Changed lines of the file:
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@@
 			)
 		)
-		(property "LCSC Part #" "C14663 "
-			(at 157.734 43.18 0)
+		(property "LCSC MPN " "CC0603KRX7R9BB104 "
+			(at 153.416 42.672 0)
 			(effects
 				(font
@@
 			)
 		)
-		(property "LCSC MPN " "CC0603KRX7R9BB104 "
-			(at 153.416 42.672 0)
+		(property "LCSC MANUFACTURER " "YAGEO "
+			(at 155.702 42.926 0)
 			(effects
 				(font
@@
 			)
 		)
-		(property "LCSC MANUFACTURER " "YAGEO "
-			(at 155.702 42.926 0)
+		(property "LCSC Part # " "C14663 "
+			(at 157.734 43.18 0)
 			(effects
 				(font
@@
 			)
 		)
-		(property "LCSC Part # " "-"
+		(property "LCSC Part # " "C318884"
 			(at 139.192 121.92 0)
 			(effects
@@
 			)
 		)
-		(property "LCSC MPN " "-"
+		(property "LCSC MPN " "TS-1187A-B-A-B"
 			(at 139.192 121.92 0)
 			(effects
@@
 			)
 		)
-		(property "LCSC MANUFACTURER " "-"
+		(property "LCSC MANUFACTURER " "XKB Connection"
 			(at 139.192 121.92 0)
 			(effects
@@
 			)
 		)
-		(property "LCSC Part #" "C14663 "
-			(at 59.944 49.53 0)
+		(property "LCSC MPN " "CC0603KRX7R9BB104 "
+			(at 55.626 49.022 0)
 			(effects
 				(font
@@
 			)
 		)
-		(property "LCSC MPN " "CC0603KRX7R9BB104 "
-			(at 55.626 49.022 0)
+		(property "LCSC MANUFACTURER " "YAGEO "
+			(at 57.912 49.276 0)
 			(effects
 				(font
@@
 			)
 		)
-		(property "LCSC MANUFACTURER " "YAGEO "
-			(at 57.912 49.276 0)
+		(property "LCSC Part # " "C14663 "
+			(at 59.944 49.53 0)
 			(effects
 				(font
@@
 			)
 		)
-		(property "LCSC Part # " "-"
+		(property "LCSC Part # " "C318884"
 			(at 215.392 121.92 0)
 			(effects
@@
 			)
 		)
-		(property "LCSC MPN " "-"
+		(property "LCSC MPN " "TS-1187A-B-A-B"
 			(at 215.392 121.92 0)
 			(effects
@@
 			)
 		)
-		(property "LCSC MANUFACTURER " "-"
+		(property "LCSC MANUFACTURER " "XKB Connection"
 			(at 215.392 121.92 0)
 			(effects
@@
 			)
 		)
-		(property "LCSC Part # " "-"
+		(property "LCSC Part # " "C318884"
 			(at 240.792 121.92 0)
 			(effects
@@
 			)
 		)
-		(property "LCSC MPN " "-"
+		(property "LCSC MPN " "TS-1187A-B-A-B"
 			(at 240.792 121.92 0)
 			(effects
@@
 			)
 		)
-		(property "LCSC MANUFACTURER " "-"
+		(property "LCSC MANUFACTURER " "XKB Connection"
 			(at 240.792 121.92 0)
 			(effects
@@
 			)
 		)
-		(property "LCSC Part #" "C15850 "
-			(at 157.734 33.02 0)
+		(property "LCSC MPN " "CL21A106KAYNNNE "
+			(at 153.416 32.512 0)
 			(effects
 				(font
@@
 			)
 		)
-		(property "LCSC MPN " "CL21A106KAYNNNE "
-			(at 153.416 32.512 0)
+		(property "LCSC MANUFACTURER " "SAMSUNG "
+			(at 155.702 32.766 0)
 			(effects
 				(font
@@
 			)
 		)
-		(property "LCSC MANUFACTURER " "SAMSUNG "
-			(at 155.702 32.766 0)
+		(property "LCSC Part # " "C15850 "
+			(at 157.734 33.02 0)
 			(effects
 				(font
@@
 			)
 		)
-		(property "LCSC Part # " "-"
+		(property "LCSC Part # " "C318884"
 			(at 164.592 157.48 0)
 			(effects
@@
 			)
 		)
-		(property "LCSC MPN " "-"
+		(property "LCSC MPN " "TS-1187A-B-A-B"
 			(at 164.592 157.48 0)
 			(effects
@@
 			)
 		)
-		(property "LCSC MANUFACTURER " "-"
+		(property "LCSC MANUFACTURER " "XKB Connection"
 			(at 164.592 157.48 0)
 			(effects
@@
 			)
 		)
-		(property "LCSC Part # " "-"
+		(property "LCSC Part # " "C318884"
 			(at 164.592 121.92 0)
 			(effects
@@
 			)
 		)
-		(property "LCSC MPN " "-"
+		(property "LCSC MPN " "TS-1187A-B-A-B"
 			(at 164.592 121.92 0)
 			(effects
@@
 			)
 		)
-		(property "LCSC MANUFACTURER " "-"
+		(property "LCSC MANUFACTURER " "XKB Connection"
 			(at 164.592 121.92 0)
 			(effects
@@
 			)
 		)
-		(property "LCSC Part # " "-"
+		(property "LCSC Part # " "C318884"
 			(at 62.992 121.92 0)
 			(effects
@@
 			)
 		)
-		(property "LCSC MPN " "-"
+		(property "LCSC MPN " "TS-1187A-B-A-B"
 			(at 62.992 121.92 0)
 			(effects
@@
 			)
 		)
-		(property "LCSC MANUFACTURER " "-"
+		(property "LCSC MANUFACTURER " "XKB Connection"
 			(at 62.992 121.92 0)
 			(effects
@@
 			)
 		)
-		(property "LCSC Part # " "-"
+		(property "LCSC Part # " "C318884"
 			(at 88.392 121.92 0)
 			(effects
@@
 			)
 		)
-		(property "LCSC MPN " "-"
+		(property "LCSC MPN " "TS-1187A-B-A-B"
 			(at 88.392 121.92 0)
 			(effects
@@
 			)
 		)
-		(property "LCSC MANUFACTURER " "-"
+		(property "LCSC MANUFACTURER " "XKB Connection"
 			(at 88.392 121.92 0)
 			(effects
@@
 			)
 		)
-		(property "LCSC Part # " "-"
+		(property "LCSC Part # " "C318884"
 			(at 139.192 172.72 0)
 			(effects
@@
 			)
 		)
-		(property "LCSC MPN " "-"
+		(property "LCSC MPN " "TS-1187A-B-A-B"
 			(at 139.192 172.72 0)
 			(effects
@@
 			)
 		)
-		(property "LCSC MANUFACTURER " "-"
+		(property "LCSC MANUFACTURER " "XKB Connection"
 			(at 139.192 172.72 0)
 			(effects
@@
 			)
 		)
-		(property "LCSC Part # " "-"
+		(property "LCSC Part # " "C318884"
 			(at 113.792 121.92 0)
 			(effects
@@
 			)
 		)
-		(property "LCSC MPN " "-"
+		(property "LCSC MPN " "TS-1187A-B-A-B"
 			(at 113.792 121.92 0)
 			(effects
@@
 			)
 		)
-		(property "LCSC MANUFACTURER " "-"
+		(property "LCSC MANUFACTURER " "XKB Connection"
 			(at 113.792 121.92 0)
 			(effects
@@
 			)
 		)
-		(property "LCSC Part #" "C15850 "
-			(at 237.744 33.02 0)
+		(property "LCSC MPN " "CL21A106KAYNNNE "
+			(at 233.426 32.512 0)
 			(effects
 				(font
@@
 			)
 		)
-		(property "LCSC MPN " "CL21A106KAYNNNE "
-			(at 233.426 32.512 0)
+		(property "LCSC MANUFACTURER " "SAMSUNG "
+			(at 235.712 32.766 0)
 			(effects
 				(font
@@
 			)
 		)
-		(property "LCSC MANUFACTURER " "SAMSUNG "
-			(at 235.712 32.766 0)
+		(property "LCSC Part # " "C15850 "
+			(at 237.744 33.02 0)
 			(effects
 				(font

Commit message: Revision 02: fixed minor issues with D2 and U6 symbols/footprints. Generated new gerber and Drill files. Generated new PDF files of schematic and layout.
Connections:
- net +5V: now also D2.3 (VDD); no longer D2.1 (VDD)
- net GND: now also D2.1 (VSS); no longer D2.3 (VSS)
- net NEOPIXEL DIN: now also D2.2 (DIN); no longer D2.4 (DIN)
- net NEOPIXEL DOUT: now also D2.4 (DOUT); no longer D2.2 (DOUT)
Changed lines of the file:
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@@
 	(title_block
 		(title "EMBARCADOS - CURSO PCB")
-		(date "2025-01-05")
-		(rev "01")
+		(date "2025-02-09")
+		(rev "02")
 		(company "Mechatronix Lab")
 		(comment 1 "Eng. André A. M. Araújo")
